File: HW/EAGLE/b333.brd (EAGLE design)
At the start: 80.6 x 52.4 mm, 87 parts, among them Q5 NMOSD

Commit message: .
Parts:
- added 1C2: 220u/6V, resistor:E3,5-8
- added 2C1: 0.47n, resistor:C0805K
- added 2D2: SS12, diode:SMB
- added 2L2: 220uH, rcl:6000-XXXX-RC
- added 2R5: 180R, resistor:R0805
- added 2R6: 1R, resistor:R0805
- added 2R7: 18K, resistor:R0805
- added 2R8: 56K, resistor:R0805
- added C4: 50u, resistor:E2,5-6
- added C5, C6: 100n, resistor:C0805K
- added D7: MC34063AD, mc34063-2:SOIC8
Connections:
- new net N$13: 2D2.A, 2L2.2, D7.1
- new net N$14: 2L2.1, 2R5.1, 2R6.2, D7.7
- new net N$15: 2R5.2, D7.8
- new net N$16: 2R7.2, 2R8.1, D7.5
- new net N$8: 2C1.1, D7.3
- net +5V: now also 1C2.+, 2D2.C, 2R8.2, C5.1
- net GND: now also 1C2.-, 2C1.2, 2R7.1, C4.-, C5.2, C6.2, D7.2, D7.4
- net V+: now also 2R6.1, C4.+, C6.1, D7.6

Commit message: .
Parts:
- added 1C5: 220u/6V, resistor:E2-5
- added 2L3: 220uH, rcl:6000-XXXX-RC
- added C7: 100n, resistor:C0805K
- 1C2: device resistor:E3,5-8 -> resistor:E2-5
- moved 2R8 40.3 mm to (-42.5, -83.8), turned to 270 degrees
- moved 1C2 31.8 mm to (-44.5, -90.2), turned to 180 degrees
- moved S1 28.7 mm to (-54.3, -36.8)
- moved C5 27.9 mm to (-44.1, -87.6), turned to 180 degrees
- moved 2C1 27.0 mm to (-48.9, -90.2), turned to 180 degrees
- moved 2R5 23.6 mm to (-53.7, -78.1), turned to 180 degrees
- moved C4 23.2 mm to (-60.0, -81.3), turned to 270 degrees
- moved 2R6 22.6 mm to (-48.9, -78.1), turned to 180 degrees
- moved 2L2 21.7 mm to (-52.7, -83.2), turned to 270 degrees
- moved C6 21.4 mm to (-57.8, -81.6), turned to 270 degrees
- moved 2D2 19.9 mm to (-49.2, -93.7), turned to 180 degrees
- moved 2R7 18.0 mm to (-45.1, -83.2), turned to 90 degrees
- moved D7 13.5 mm to (-48.9, -84.5)
Connections:
- new net N$17: 1C2.+, 2D2.C, 2L3.1, 2R8.2, C5.1
- net +5V: now also 1C5.+, 2L3.2, C7.1; no longer 1C2.+, 2D2.C, 2R8.2, C5.1
- net GND: now also 1C5.-, C7.2
Routing:
- net GND: track 102.5 -> 130.7 mm
- net V+: track 0.00 -> 24.3 mm
- net N$17: track 0.00 -> 18.1 mm
- net N$14: track 0.00 -> 9.94 mm
- net N$13: track 0.00 -> 9.26 mm
- net N$15: track 0.00 -> 7.43 mm
- net N$8: track 0.00 -> 3.27 mm
- net N$16: track 0.00 -> 1.96 mm

Commit message: .
Parts:
- removed D7: MC34063AD, mc34063-2:SOIC8
- added 1Q1: NMOSD, DSS:DPACK_1
- added 2L4: 220uH, rcl:6000-XXXX-RC
- added 3C10, 3C7, C8: 100n, resistor:C0805K
- added 3C11: 47u, resistor:E2,5-6
- added 3C5: 1n, resistor:C0805K
- added 3C6, 3C9: 47u/50V, resistor:E2,5-6
- added 3C8: 100u, resistor:E2,5-6
- added 3D2: 1N5819, diode:SMB
- added 3L2: 180uH, rcl:6000-XXXX-RC
- added 3R1B1, 3R8: 1R, resistor:R0805
- added 3R5: 62K, resistor:R0805
- added 3R6: 2K, resistor:R0805
- added 3R7: 180R, resistor:R0805
- added 5MA: 10MA, jumper:JP2
- added B+OUT+, B-1, GND: B-, TP4056_18650:PAD-
- added C11, C12, C13: 100n, rcl:C0805
- added D10, D11, D9: LL4148, diode:SOD80C
- added DA1: TP4056, TP4056:SOP-8
- added DA2: DW01A, DW01:SOT23-6
- added DA3, DA5: MC34063AD, mc34063-2:SOIC8
- added DA4: 78L05, v-reg:SOT89R
- added DA4A: MCP1702, v-reg:SOT89R
- added GREEN, RED: (no value), led:CHIP-LED0805
- added Q1: BF423, transistor-pnp:TO92-BCE
- added R10, R24: 1k2, resistor:R0805
- added R11: 300, resistor:R0805
- added R12: 150, resistor:R0805
- added R13: 39k, resistor:R0805
- added R19: 0.5, resistor:R0805
- added R20, R22, R23: 1k, resistor:R0805
- added R21: 100, resistor:R0805
- added R8: 10k, resistor:R0805
- added R9: 100k, resistor:R0805
- added VT2: FS8205A, FS8205A:TSSOP-8
- added X2: USB MICRO, SmartPrj:CON2_USB_MICRO_B_AT
- added ZEN_A1, ZEN_K1: (no value), pinhead:1X01
- moved C4 80.4 mm to (19.4, -94.0), turned to 90 degrees
- moved C6 75.9 mm to (17.1, -93.7), turned to 90 degrees
- moved 2R5 69.3 mm to (13.0, -97.2), turned to 0 degrees
- moved 2L2 65.4 mm to (12.1, -92.1), turned to 90 degrees
- moved 2R6 60.2 mm to (8.26, -97.2), turned to 0 degrees
- moved 2D2 59.0 mm to (8.57, -81.6), turned to 0 degrees
- moved 2C1 57.4 mm to (8.26, -85.1), turned to 0 degrees
- moved 2R7 50.3 mm to (4.45, -92.1), turned to 270 degrees
- moved 1C2 48.5 mm to (3.81, -85.1), turned to 0 degrees
- moved C5 47.6 mm to (3.49, -87.6), turned to 0 degrees
- moved 2R8 45.1 mm to (1.91, -91.4), turned to 90 degrees
- moved 1C5 32.8 mm to (-2.86, -93.0)
- moved 2L3 28.2 mm to (-6.35, -85.7), turned to 180 degrees
- moved C7 24.9 mm to (-8.57, -91.4)
Connections:
- new net +3V7: B+OUT+.B-, C13.1, DA1.5, R21.2
- new net +7V: 1C5.+, 2L3.2, C7.1, DA4.1, DA4A.3, DA4A.4
- new net 1MA: 5MA.2, Q1.E, R10.2
- new net B-: B-1.B-, C11.1, DA2.6, VT2.2, VT2.3
- new net N$18: Q1.C, ZEN_K1.1
- new net N$23: 3C5.1, DA5.3
- new net N$26: 3D2.A, 3L2.2, DA5.1
- new net N$51: 3R5.1, 3R6.1, DA5.5
- new net N$52: 2L4.1, 3C6.+, 3C7.1, 3D2.C, 3R5.2
- new net N$53: 3R7.2, DA5.8
- new net N$54: 3L2.1, 3R1B1.2, 3R7.1, 3R8.2, DA5.7
- new net N$55: 5MA.3, R11.2
- new net N$56: 1Q1.G, R8.2, R9.1
- new net N$57: 2L4.2, 3C10.1, 3C9.+, D9.A, R10.1, R11.1, R12.1
- new net N$58: 1Q1.D, DA5.2, DA5.4
- new net N$59: 5MA.1, R12.2
- new net N$65: D10.A, D9.C
- new net N$66: D10.C, D11.A
- new net N$67: D11.C, Q1.B, R13.2
- new net N$75: VT2.1, VT2.8
- new net N$76: DA2.3, VT2.5
- new net N$77: DA2.1, VT2.4
- new net N$78: DA2.2, R20.2
- new net N$79: C11.2, DA2.5, R21.1
- new net N$80: DA1.7, RED.C
- new net N$81: DA1.6, GREEN.C
- new net N$82: R22.1, RED.A
- new net N$83: GREEN.A, R23.1
- new net N$84: C12.1, DA1.4, DA1.8, R19.2, R22.2, R23.2
- new net N$85: R19.1, X2.P1
- new net N$86: DA1.2, R24.2
- new net UGND: C12.2, C13.2, DA1.1, DA1.3, R20.1, R24.1, VT2.6, VT2.7, X2.P5, X2.S1, X2.S2, X2.S3, X2.S4, X2.S5, X2.S6
- new net ZENER_EN: R8.1
- net +5V: now also 3C11.+, C8.1, DA4.2, DA4A.1; no longer 1C5.+, 2L3.2, C7.1
- net GND: now also 1Q1.S, 3C10.2, 3C11.-, 3C5.2, 3C6.-, 3C7.2, 3C8.-, 3C9.-, 3R6.2, C8.2, DA3.2, DA3.4, DA4.3, DA4.4, DA4A.2, GND.B-, R13.1, R9.2, ZEN_A1.1; no longer D7.2, D7.4
- net N$13: now also DA3.1; no longer D7.1
- net N$14: now also DA3.7; no longer D7.7
- net N$15: now also DA3.8; no longer D7.8
- net N$16: now also DA3.5; no longer D7.5
- net N$8: now also DA3.3; no longer D7.3
- net V+: now also 3C8.+, 3R1B1.1, 3R8.1, DA3.6, DA5.6; no longer D7.6
Routing:
- net GND: track 130.7 -> 200.9 mm
- net UGND: track 0.00 -> 62.0 mm
- net +3V7: track 0.00 -> 32.0 mm
- net N$77: track 0.00 -> 29.9 mm
- net N$52: track 0.00 -> 29.6 mm
- net N$84: track 0.00 -> 29.2 mm, vias 0 -> 2
- net N$57: track 0.00 -> 24.7 mm
- net B-: track 0.00 -> 18.3 mm
- net N$76: track 0.00 -> 17.5 mm
- net N$54: track 0.00 -> 16.1 mm
- net +5V: track 20.6 -> 36.1 mm
- net N$58: track 0.00 -> 14.4 mm
- net N$18: track 0.00 -> 9.04 mm
- net V+: track 24.3 -> 32.6 mm
- net N$78: track 0.00 -> 8.25 mm
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
Commit message: .
Parts:
- removed X2: USB MICRO, SmartPrj:CON2_USB_MICRO_B_AT
- added 1C13, C10, C9: 100n, resistor:C0805
- added 1C6: 1n, resistor:C0805K
- added 1C7, 3C13, C17, C18: 100n, resistor:C0805K
- added 1C8, 1C9: 22p, resistor:C0805K
- added 1L2: 10mkhn, rcl:IRF24
- added 1R10, 1R9: 10K, resistor:R0805
- added 1R17: 3K3, resistor:R1206W
- added 1R18: 27K, resistor:R0805
- added 1R19, 1R21, 1R23: 680, resistor:0207/10
- added 1R20, 1R22, 1R24: 470K, resistor:0207/10
- added 1R25: 2K2, resistor:R0805
- added 1R26: 270, resistor:R1206W
- added 1RC2: 22K, resistor:R0805
- added 1RC2*1: 4K3, resistor:R1206W
- added 1Z2: 8MHz, crystal:HC49U70
- added 3C12: 47u, resistor:E2,5-6
- added 4R6, 4R7: 100, resistor:R0805
- added 4Y3, 4Y4: РЭС55А, relay_ussr:РЭС55А
- added D7: MEGA328P-AU, avr-6:TQFP32-08
- added D8: TL431, v-reg:TO92-CLP
- added DA6: 78L05, v-reg:SOT89R
- added H2: LCD, pinhead:1X16
- added ISP: (no value), con-lstb:MA03-2
- added J_NO_LI, J_ONE5V: (no value), jumper:SJ
- added R14: 180K, resistor:R0805
- added R15: 20.0k, resistor:R0805
- added R16: 180.0k, resistor:R0805
- added R4: 20K, resistor:R0805
- added T4, T5, T6: (no value), pinhead:1X01
- added TEST1: TT-P, transistor_tester:TT-P
- added X1: USB MICRO, SmartPrj:CON2_USB_MICRO_B_AT
- R24: device resistor:R0805 -> resistor:0204/7
- moved DIS1 244.1 mm to (216.5, 84.8)
- moved R23 228.8 mm to (279.7, 92.4), flipped to the bottom, turned to 180 degrees
- moved R22 225.2 mm to (279.7, 89.9), flipped to the bottom, turned to 180 degrees
- moved C13 221.4 mm to (272.1, 94.0), flipped to the bottom, turned to 90 degrees
- moved GREEN 219.8 mm to (275.3, 90.5), flipped to the bottom, turned to 270 degrees
- moved C12 219.1 mm to (279.4, 86.0), flipped to the bottom, turned to 270 degrees
- moved RED 217.1 mm to (275.3, 88.6), flipped to the bottom, turned to 270 degrees
- moved 2C1 214.5 mm to (219.4, -47.3)
- moved 2D2 214.5 mm to (219.7, -43.8)
- moved 2R6 214.5 mm to (219.4, -59.4)
- moved 2R7 214.5 mm to (215.6, -54.3)
- moved 3C11 214.5 mm to (189.5, -47.9)
- moved DA3 214.5 mm to (219.4, -53.0)
- moved 1C2 214.5 mm to (214.9, -47.3)
- moved 1C5 214.5 mm to (208.3, -55.2)
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Connections:
- net N$57 renamed +40V
- new net +5V/2: 1R26.2, 1RC2.1, 3C12.+, C18.1, DA6.2, H2.2, J_ONE5V.2
- new net E1: D7.9, H2.6
- new net N$60: 1RC2*1.2, 1RC2.2, H2.3
- new net N$61: 1R26.1, H2.15
- new net N$62: D7.1, H2.14
- new net N$63: R14.2
- new net N$64: 1C6.1, D7.20
- new net N$68: 1C8.2, 1Z2.2, D7.7
- new net N$69: 1C9.2, 1Z2.1, D7.8
- new net N$70: 1C13.1, 1L2.1, D7.18
- new net N$71: 4R6.2, 4Y3.P
- new net N$72: 4R7.2, 4Y4.P
- new net N$87: D7.30, H2.11
- new net N$88: D7.31, H2.12
- new net N$89: D7.32, H2.13
- new net PB3: 1R19.1, D7.12
- new net PB4: 1R20.1, D7.13
- new net PB5: 1R21.1, D7.14
- new net PC10: 1R21.2, 1R22.2, 4Y4.O, D7.24, T5.1, TEST1.P$2, TEST1.P$3, TEST1.P$4
- new net PC11: 1R23.2, 1R24.2, 4Y3.O, D7.25, T6.1, TEST1.P$5
- new net PC6: 1R10.2, 1R17.2, D7.28
- new net PC7: 1R25.2, D7.27, D8.C, D8.R
- new net PC8: C9.1, D7.26, R14.1, R4.2
- new net PC9: 1R19.2, 1R20.2, 4R6.1, 4R7.1, D7.23, T4.1, TEST1.P$1
- new net PD1: 1R18.2, C17.1, D7.11
- new net PD2: D7.10
- new net RS1: D7.2, H2.4
- new net V+1: 1R10.1, 1R9.2
- net +5V: now also 1C7.1, 1L2.2, 1R18.1, 1R25.1, C10.1, D7.4, D7.6, ISP.2, J_NO_LI.2, J_ONE5V.1
- net +7V: now also DA6.1, J_NO_LI.1
- net GND: now also 1C13.2, 1C6.2, 1C7.2, 1C8.1, 1C9.1, 1R17.1, 1RC2*1.1, 3C12.-, 3C13.2, C10.2, C17.2, C18.2, C9.2, D7.21, D7.3, D7.5, D8.A, DA6.3, DA6.4, H2.1, H2.10, H2.16, H2.5, H2.7, H2.8, H2.9, ISP.6, R15.1, R4.1
- net MISO: now also 1R23.1, D7.16, ISP.1
- net MOSI: now also 1R22.1, D7.15, ISP.4
- net N$18: now also R16.2
- net N$85: now also X1.P1; no longer X2.P1
- net PC3: now also 3C13.1, R15.2, R16.1
- net RESET: now also 1R9.1, D7.29, ISP.5
- net SCK: now also 1R24.1, D7.17, ISP.3
- net UGND: now also DA1.., X1.P5, X1.S1, X1.S2, X1.S3, X1.S4, X1.S5, X1.S6; no longer X2.P5, X2.S1, X2.S2, X2.S3, X2.S4, X2.S5, X2.S6
Routing:
- net PC3: track 0.00 -> 51.3 mm, vias 0 -> 2
- net +3V7: track 32.0 -> 6.60 mm
- net V+: track 32.6 -> 46.7 mm
- net +40V: track 24.7 -> 14.5 mm
- net B-: track 18.3 -> 26.7 mm
- net N$54: track 16.1 -> 10.8 mm
- net N$26: track 4.78 -> 8.12 mm
- net GND: track 200.9 -> 197.7 mm
- net N$67: track 5.72 -> 8.48 mm
- net N$77: track 29.9 -> 32.0 mm
- net N$78: track 8.25 -> 10.1 mm
- net N$56: track 6.90 -> 5.27 mm
- net N$52: track 29.6 -> 31.2 mm
- net N$84: track 29.2 -> 28.1 mm
- net N$76: track 17.5 -> 18.3 mm
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
Commit message: .
Parts:
- removed R9: 100k, resistor:R0805
- added R18, R25: 10k, resistor:R0805
- added VT4: МП15, transistor-pnp:TO92-BCE
- R8: value 10k -> 100k
- moved DIS1 179.1 mm to (37.5, 80.6)
- moved 2L3 80.1 mm to (234.0, 26.7)
- moved 3C11 80.1 mm to (218.8, 26.7)
- moved C18 80.1 mm to (279.4, 4.45)
- moved C6 80.1 mm to (257.5, 18.7)
- moved DA6 80.1 mm to (280.4, 17.8)
- moved 1C2 80.1 mm to (244.2, 27.3)
- moved 1C5 80.1 mm to (237.5, 19.4)
- moved 2C1 80.1 mm to (248.6, 27.3)
- moved 2D2 80.1 mm to (248.9, 30.8)
- moved 2L2 80.1 mm to (252.4, 20.3)
- moved 2R5 80.1 mm to (253.4, 15.2)
- moved 2R6 80.1 mm to (248.6, 15.2)
- moved 2R7 80.1 mm to (244.8, 20.3)
- moved 2R8 80.1 mm to (242.3, 21.0)
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- renumbered 1Q1 to VT5, Q1 to VT6
Connections:
- removed net ZENER_EN: R8.1
- new net !BUTTON: R18.1
- new net N$73: R25.2, R8.1, VT4.C
- new net N$74: R18.2, VT4.B
- net +5V/2: now also VT4.E
- net GND: now also R25.1; no longer 3R6.2, R9.2
- net N$56: no longer R9.1
- net N$58: now also 3R6.2
Routing:
- net GND: track 197.7 -> 188.2 mm
- net +40V: track 14.5 -> 8.30 mm
- net N$56: track 5.27 -> 0.00 mm
- net N$92: track 31.2 -> 26.1 mm

Commit message: 34063 links
Parts:
- removed 1C10: 220u/6V, resistor:E3,5-8
- removed 2C2: 0.47n, resistor:C0805K
- removed 2D1: SS12, diode:DO41-10
- removed 2L1: 220uH, inductor-neosid:SD12_1000
- removed 2R1: 1R, resistor:R0805
- removed 2R2: 180R, resistor:R0805
- removed 2R3: 18K, resistor:R0805
- removed 2R4: 56K, resistor:R0805
- removed C14, C15: 100n, resistor:C0805K
- removed C16: 50u, resistor:E2,5-6
- removed C9: 100n, resistor:C0805
- removed D3: MC34063AD, mc34063:SOIC8
- removed R14: 180K, resistor:R0805
- removed R4: 20K, resistor:R0805
- added T7: (no value), transistor:TO92-ECB
- moved DIS1 123.9 mm to (0.95, -37.8)
- moved C3 37.5 mm to (6.67, -38.1), flipped to the top
- moved S2 35.0 mm to (5.40, -50.2), flipped to the bottom
- moved 1RC1 30.2 mm to (2.86, -38.1), flipped to the top
- moved 1R1 22.2 mm to (-1.59, -59.7), flipped to the top
- moved 1Z2 19.1 mm to (128.9, 181.0), turned to 0 degrees
- moved T3 17.4 mm to (-18.1, -78.7), flipped to the bottom
- moved 1R2 16.9 mm to (-4.76, -61.6), flipped to the bottom
- moved 1R3 15.0 mm to (-6.03, -56.5), flipped to the top
- moved 1L1 13.8 mm to (-6.99, -44.5), flipped to the top
- moved 1C1 12.7 mm to (-7.94, -53.7), flipped to the bottom
- moved T1 12.7 mm to (-7.94, -78.7), flipped to the bottom
- moved 1R4 12.7 mm to (-7.94, -57.8), flipped to the bottom
- moved 1R5 12.1 mm to (-8.57, -54.0), flipped to the top
- moved D1 12.1 mm to (-8.57, -45.1), flipped to the bottom
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Connections:
- net PC6 renamed U_BAT
- net PC7 renamed +2V5
- removed net N$22: 2R2.2, D3.8
- removed net N$24: 2L1.1, 2R1.2, 2R2.1, D3.7
- removed net N$25: 2R3.2, 2R4.1, D3.5
- removed net N$56: R8.2, VT5.G
- removed net N$63: R14.2
- removed net N$73: R25.2, R8.1, VT4.C
- removed net N$74: R18.2, VT4.B
- removed net PC8: C9.1, D7.26, R14.1, R4.2
- removed net V+1: 1R10.1, 1R9.2
- net +5V: now also 1R9.2; no longer 1C10.+, 2D1.C, 2R4.2, C14.1
- net +5V/2: now also R25.2; no longer VT4.E
- net GND: now also R8.1, T7.E; no longer 1C10.-, 2C2.2, 2R3.1, C14.2, C15.2, C16.-, C9.2, D3.2, D3.4, R25.1, R4.1
- net N$19: now also R18.2, T7.B; no longer 2C2.1, D3.3
- net N$21: now also R25.1, R8.2, T7.C, VT5.G; no longer 2D1.A, 2L1.2, D3.1
- net PC3: now also D7.26
- net V+: now also 1R10.1; no longer 2R1.1, C15.1, C16.+, D3.6
Routing:
- net N$41: track 14.2 -> 39.7 mm
- net N$42: track 15.1 -> 37.5 mm, vias 2 -> 0
- net N$44: track 16.4 -> 36.0 mm, vias 2 -> 0
- net N$11: track 16.9 -> 0.00 mm
- net E: track 9.30 -> 26.0 mm, vias 0 -> 2
- net N$43: track 19.7 -> 28.2 mm, vias 2 -> 0
- net GND: track 188.2 -> 180.4 mm
- net RS: track 21.3 -> 26.5 mm

Commit message: add lnk
Parts:
- removed D7: MEGA328P-AU, avr-6:TQFP32-08
- added DD1: MEGA328P-AU, avr-6:TQFP32-08
- 1C5: value 220u/6V -> 1000u/6V
- 1R19, 1R20, 1R21, 1R22, 1R23, 1R24: device resistor:0207/10 -> resistor:M0805
- moved DIS1 313.1 mm to (155.3, 234.6)
- moved 1R20 134.0 mm to (151.1, 183.8), flipped to the bottom, turned to 270 degrees
- moved TEST1 125.8 mm to (147.6, 173.7)
- moved 3C13 119.6 mm to (232.1, 166.7)
- moved 3D2 119.6 mm to (244.5, 188.0)
- moved 3L2 119.6 mm to (244.5, 195.9)
- moved B+OUT+ 119.6 mm to (204.5, 180.7)
- moved B-1 119.6 mm to (204.5, 172.1)
- moved C11 119.6 mm to (204.8, 176.5)
- moved D11 119.6 mm to (232.4, 154.3)
- moved DA1 119.6 mm to (205.1, 190.2)
- moved R10 119.6 mm to (243.8, 160.0)
- moved R11 119.6 mm to (243.8, 162.6)
- moved R21 119.6 mm to (208.9, 178.4)
- moved R25 119.6 mm to (247.7, 163.2)
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Connections:
- removed net PC10: 1R21.2, 1R22.2, 4Y4.O, D7.24, T5.1, TEST1.P$2, TEST1.P$3, TEST1.P$4
- removed net PC11: 1R23.2, 1R24.2, 4Y3.O, D7.25, T6.1, TEST1.P$5
- removed net PC9: 1R19.2, 1R20.2, 4R6.1, 4R7.1, D7.23, T4.1, TEST1.P$1
- new net T1: 1R19.2, 1R20.2, 4R6.1, 4R7.1, DD1.23, T4.1, TEST1.P$5
- new net T2: 1R21.2, 1R22.2, 4Y4.O, DD1.24, T5.1, TEST1.P$2, TEST1.P$3, TEST1.P$4
- new net T3: 1R23.2, 1R24.2, 4Y3.O, DD1.25, T6.1, TEST1.P$1
- net +2V5: now also DD1.27; no longer D7.27
- net +5V: now also DD1.4, DD1.6; no longer D7.4, D7.6
- net E1: now also DD1.9; no longer D7.9
- net GND: now also DD1.21, DD1.3, DD1.5; no longer D7.21, D7.3, D7.5
- net MISO: now also DD1.16; no longer D7.16
- net MOSI: now also DD1.15; no longer D7.15
- net N$62: now also DD1.1; no longer D7.1
- net N$64: now also DD1.20; no longer D7.20
- net N$68: now also DD1.7; no longer D7.7
- net N$69: now also DD1.8; no longer D7.8
- net N$70: now also DD1.18; no longer D7.18
- net N$87: now also DD1.30; no longer D7.30
- net N$88: now also DD1.31; no longer D7.31
- net N$89: now also DD1.32; no longer D7.32
- net PB3: now also DD1.12; no longer D7.12
- net PB4: now also DD1.13; no longer D7.13
- net PB5: now also DD1.14; no longer D7.14
- net PC3: now also DD1.26; no longer D7.26
- net PD1: now also DD1.11; no longer D7.11
- net PD2: now also DD1.10; no longer D7.10
- net RESET: now also DD1.29; no longer D7.29
- net RS1: now also DD1.2; no longer D7.2
- net SCK: now also DD1.17; no longer D7.17
- net U_BAT: now also DD1.28; no longer D7.28
Routing:
- net E1: track 0.00 -> 46.0 mm, vias 0 -> 2
- net RS1: track 0.00 -> 43.1 mm, vias 0 -> 2
- net T3: track 0.00 -> 26.4 mm, vias 0 -> 2
- net T1: track 0.00 -> 26.1 mm, vias 0 -> 2
- net T2: track 0.00 -> 24.8 mm, vias 0 -> 2
- net N$87: track 0.00 -> 16.6 mm
- net N$88: track 0.00 -> 16.6 mm
- net N$62: track 0.00 -> 16.1 mm
- net N$89: track 0.00 -> 14.8 mm
- net PB3: track 0.00 -> 6.88 mm
- net SCK: track 18.7 -> 24.3 mm
- net PB4: track 0.00 -> 5.22 mm
- net PB5: track 0.00 -> 4.37 mm
- net MISO: track 14.2 -> 18.5 mm
- net MOSI: track 33.1 -> 37.3 mm

Commit message: .
Parts:
- added 3R1B2: 2R, resistor:R0805
- 1C13: device resistor:C0805 -> resistor:C0805K
- 3C6: value 47u/50V -> 22u/100V
- 3D2: value 1N5819 -> RK19(1N5819)
- 3L2: value 180uH -> 230uH
- 3R1B1: value 1R -> 2R
- moved 1C7 95.0 mm to (154.9, 195.3), flipped to the bottom, turned to 270 degrees
- moved 1C13 94.3 mm to (141.0, 189.9), flipped to the bottom
- moved 1C6 72.1 mm to (141.0, 191.8), flipped to the bottom
- moved 1C9 34.0 mm to (160.0, 193.4), flipped to the bottom
- moved 1Z2 30.6 mm to (158.1, 190.2), turned to 180 degrees
- moved 1C8 26.3 mm to (157.5, 193.4), flipped to the bottom
- moved D8 6.48 mm to (144.8, 200.7)
- moved C17 5.26 mm to (69.2, 195.3)
- moved DIS1 3.43 mm to (158.1, 232.7)
- moved B+OUT+ 0.45 mm to (204.8, 181.0)
Connections:
- net N$54: now also 3R1B2.2
- net V+: now also 3R1B2.1
Routing:
- net GND: track 180.4 -> 212.6 mm
- net +3V7: track 6.60 -> 24.1 mm, vias 0 -> 2
- net E1: track 46.0 -> 62.1 mm
- net N$69: track 0.00 -> 12.6 mm
- net +5V: track 36.1 -> 44.3 mm
- net N$68: track 0.00 -> 7.32 mm
- net RS1: track 43.1 -> 48.5 mm
- net N$62: track 16.1 -> 18.5 mm
- net N$70: track 0.00 -> 2.24 mm
- net N$64: track 0.00 -> 1.88 mm
- net N$88: track 16.6 -> 14.9 mm
- net T3: track 26.4 -> 27.7 mm
- net T2: track 24.8 -> 26.1 mm
- net T1: track 26.1 -> 26.9 mm
