File: HW/EAGLE/b333.brd (EAGLE design)
At the start: 80.6 x 52.4 mm, 188 parts, among them Q5 NMOSD, X1 USB MICRO

Commit message: .
Parts:
- removed 1C1: 1n, resistor:C0805K
- removed 1C11, 1C12: 22p, resistor:C0805K
- removed 1C3, C3: 100n, resistor:C0805
- removed 1C4: 100n, resistor:C0805K
- removed 1L1: 10mkhn, rcl:IRF24
- removed 1R1, 1R3, 1R5: 680, resistor:0207/10
- removed 1R11, 1R13: 10K, resistor:R0805
- removed 1R12: 3K3, resistor:R1206W
- removed 1R16: 2K2, resistor:R0805
- removed 1R2, 1R4: 470K, resistor:0207/10
- removed 1Z1: 8MHz, crystal:HC49U70
- removed D1: MEGA328P-AU, avr-6:TQFP32-08
- removed D2: TL431, v-reg:TO92-CLP
- removed H1: LCD, pinhead:1X16
- removed S2: ISP, con-lstb:MA03-2
- removed TEST: TT-P, transistor_tester:TT-P
- added 3C14: 1n, resistor:C0805K
- added 3C15, 3C16: 22u/100V, resistor:E2,5-6
- added 3C17: 100u, resistor:E2,5-6
- added 3D3, 3D4: RK19(1N5819), diode:SMB
- added 3L3, 3L4: 230uH, rcl:6000-XXXX-RC
- added 3R10: 2K, resistor:R0805
- added 3R11: 180R, resistor:R0805
- added 3R12: 1R, resistor:R0805
- added 3R1B3, 3R1B4: 2R, resistor:R0805
- added 3R9: 62K, resistor:R0805
- added C14: 33, rcl:C0805K
- added C15: 2n2, rcl:C0805K
- added C16: 47m, rcl:E2-4
- added C19: 1n, rcl:C0805K
- added C9: 56, rcl:C0805K
- added D12, D3, D7: 1N4148DO35-7, diode:DO35-7
- added DA7: MC34063AD, mc34063-2:SOIC8
- added JP1, JP2: (no value), pinhead:1X01
- added Q1, Q2: 2N4126, transistor-pnp:TO92-CBE
- added R14: 100, rcl:M0805
- added R17: 470, rcl:M0805
- added R26, R28, R32, R33: 1k, rcl:M0805
- added R27: 8k2, rcl:M0805
- added R29, R30: 10k, resistor:R0805
- added R31: 300, rcl:M0805
- added R34, R9: 15k, rcl:M0805
- added R35: (no value), rcl:RTRIM3296W
- added R4: 100k, resistor:R0805
- added T8: (no value), transistor:TO92-ECB
- added T9: (no value), transistor:TO92-EBC
- added VT1: NMOSD, DSS:DPACK_1
- moved 1R18 392.4 mm to (400.4, 94.6)
- moved 1R9 392.4 mm to (442.9, 94.6)
- moved 4R6 392.4 mm to (448.0, 94.6)
- moved 4Y4 392.4 mm to (448.0, 126.7)
- moved C17 392.4 mm to (447.7, 91.8)
- moved T5 392.4 mm to (420.1, 88.3)
- moved T6 392.4 mm to (423.5, 88.3)
- moved 1L2 392.4 mm to (406.4, 87.9)
- moved 1R25 392.4 mm to (406.7, 94.6)
- moved 4Y3 392.4 mm to (413.4, 126.7)
- moved C10 392.4 mm to (437.2, 94.6)
- moved ISP 392.4 mm to (402.6, 67.6)
- moved T4 392.4 mm to (416.6, 88.3)
- moved 4R7 392.4 mm to (463.2, 95.9)
- moved DIS1 113.4 mm to (61.3, 291.8)
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Connections:
- removed net E: D1.9, H1.6
- removed net N$12: 1C12.2, 1Z1.1, D1.8
- removed net N$4: 1C1.1, D1.20
- removed net N$41: D1.30, H1.11
- removed net N$42: D1.31, H1.12
- removed net N$43: D1.1, H1.14
- removed net N$44: D1.32, H1.13
- removed net N$45: 1C3.1, 1L1.1, D1.18
- removed net PB0: 1R1.1, D1.12
- removed net PB1: 1R2.1, D1.13
- removed net PB2: 1R3.1, D1.14
- removed net PC0: 1R1.2, 1R2.2, 4R1.1, 4R2.1, D1.23, T1.1, TEST.P$1
- removed net PC5: 1R11.2, 1R12.2, D1.28
- removed net RS: D1.2, H1.4
- removed net RS1: DD1.2, H2.4
- new net !BUTTON1: R29.1
- new net N$100: D3.A, D7.A, Q2.C, R31.2
- new net N$101: C14.2, C15.1, C16.-, R33.1
- new net N$102: D7.C, R32.2, T9.B
- new net N$103: C15.2, C16.+, JP1.1
- new net N$110: 4R1.1, 4R2.1
- new net N$114: 1R6.1
- new net N$115: 1R6.2
- new net N$22: 3C14.1, DA7.3
- new net N$24: 3D3.A, 3L3.2, 3L4.1, DA7.1
- new net N$25: 3R10.1, 3R9.1, DA7.5
- new net N$52: 3R11.2, DA7.8
- new net N$56: 3L3.1, 3R11.1, 3R12.2, 3R1B3.2, 3R1B4.2, DA7.7
- new net N$57: 3R10.2, DA7.2, DA7.4, VT1.D
- new net N$63: 3C16.+, 3D4.C
- new net N$73: 3D4.A, 3L4.2
- new net N$90: Q1.E, Q2.E, R14.1
- new net N$91: C14.1, D12.A, Q1.B, R33.2, R34.2, R9.1
- new net N$93: C9.1, Q2.B, R17.1, R26.2, R27.1
- new net N$94: 3C15.+, 3D3.C, 3R9.2
- new net N$95: R29.2, T8.B
- new net N$96: R30.1, R4.2, T8.C, VT1.G
- new net N$97: C19.1, D12.C, JP2.1, R14.2, R17.2, R28.2, R9.2
- new net PD4: D3.C, DD1.2, H2.4, R27.2, R28.1, T9.C
- net +5V: no longer 1C4.1, 1L1.2, 1R16.1, C3.1, D1.4, D1.6, H1.2, S2.2
- net +5V/2: now also R30.2
- net GND: now also 3C14.2, 3C15.-, 3C16.-, 3C17.-, C19.2, C9.2, Q1.C, R26.1, R31.1, R32.1, R35.1, R35.2, R4.1, T8.E, T9.E, VT1.S; no longer 1C1.2, 1C11.1, 1C12.1, 1C3.2, 1C4.2, 1R12.1, C3.2, D1.21, D1.3, D1.5, D2.A, H1.1, H1.10, H1.16, H1.5, H1.7, H1.8, H1.9, S2.6
- net MISO: no longer 1R5.1, D1.16, S2.1
- net MOSI: no longer 1R4.1, D1.15, S2.4
- net N$11: no longer H1.15
- net N$3: now also R34.1, R35.3; no longer 1C11.2, 1Z1.2, D1.7
- net N$6: no longer H1.3
- net PC1: no longer 1R3.2, 1R4.2, D1.24, T2.1, TEST.P$2, TEST.P$3, TEST.P$4
- net PC2: no longer 1R5.2, 1R6.2, D1.25, T3.1, TEST.P$5
- net PC3: no longer D1.26
- net PC4: no longer 1R16.2, D1.27, D2.C, D2.R
- net PD6: no longer D1.10
- net PD7: no longer D1.11
- net RESET: no longer 1R13.1, D1.29, S2.5
- net SCK: no longer 1R6.1, D1.17, S2.3
- net V+: now also 3C17.+, 3R12.1, 3R1B3.1, 3R1B4.1, DA7.6; no longer 1R11.1, 1R13.2
Routing:
- net PD4: track 0.00 -> 75.4 mm, vias 0 -> 2
- net RS1: track 48.5 -> 0.00 mm, vias 2 -> 0
- net N$41: track 39.7 -> 0.00 mm
- net N$42: track 37.5 -> 0.00 mm
- net N$44: track 36.0 -> 0.00 mm
- net MOSI: track 37.3 -> 4.14 mm
- net N$43: track 28.2 -> 0.00 mm
- net RS: track 26.5 -> 0.00 mm, vias 2 -> 0
- net E: track 26.0 -> 0.00 mm, vias 2 -> 0
- net GND: track 212.6 -> 189.0 mm, vias 0 -> 3
- net N$97: track 0.00 -> 21.7 mm
- net +5V: track 44.3 -> 23.8 mm
- net PB0: track 19.4 -> 0.00 mm
- net PB1: track 19.2 -> 0.00 mm
- net SCK: track 24.3 -> 5.55 mm
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
Commit message: .
Parts:
- added J_PD4: (no value), jumper:SJ
- 3R9: value 62K -> 120k
- moved 1R9 405.9 mm to (66.4, 246.1), flipped to the bottom, turned to 180 degrees
- moved T6 397.8 mm to (50.2, 225.4)
- moved 1R25 394.1 mm to (48.9, 259.7), flipped to the bottom, turned to 90 degrees
- moved T5 387.5 mm to (57.5, 225.1)
- moved 1L2 387.1 mm to (55.6, 251.5), turned to 20 degrees
- moved T4 380.2 mm to (61.9, 225.4)
- moved ISP 377.4 mm to (67.3, 241.0), turned to 270 degrees
- moved 1R10 14.4 mm to (45.1, 269.2)
- moved 1RC2 4.96 mm to (31.1, 284.5)
- moved 1R17 3.42 mm to (30.2, 280.7), turned to 0 degrees
- moved 1RC2*1 2.73 mm to (30.5, 287.0)
- moved D8 1.62 mm to (52.7, 262.6), turned to 90 degrees
Connections:
- net N$64 renamed AREF
- net N$70 renamed AVCC
- removed net N$63: 3C16.+, 3D4.C
- new net N$12: 3C15.+, 3D3.C
- new net N$4: DD1.2, J_PD4.1
- net N$94: now also 3C16.+, 3D4.C; no longer 3C15.+, 3D3.C
- net PD4: now also J_PD4.2; no longer DD1.2
Routing:
- net GND: track 189.0 -> 225.5 mm
- net RESET: track 0.00 -> 29.9 mm, vias 0 -> 2
- net +5V: track 23.8 -> 46.5 mm
- net MOSI: track 4.14 -> 20.6 mm
- net SCK: track 5.55 -> 21.8 mm
- net MISO: track 4.35 -> 17.5 mm
- net +2V5: track 0.00 -> 6.26 mm
- net PD4: track 75.4 -> 71.0 mm
- net N$4: track 0.00 -> 3.70 mm

Commit message: .
Connections:
- new net N$45: 3D3.A
- net N$24: no longer 3D3.A
Changed lines of the file:
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@@
 <signal name="N$24">
 <contactref element="DA7" pad="1"/>
-<contactref element="3D3" pad="A"/>
 <contactref element="3L3" pad="2"/>
 <contactref element="3L4" pad="1"/>
-<wire x1="-58.7375" y1="-104.835" x2="-58.76" y2="-110.1725" width="0" layer="19" extent="1-1"/>
 <wire x1="-63.2225" y1="-99.3775" x2="-58.7375" y2="-104.835" width="0" layer="19" extent="1-1"/>
 <wire x1="28.9325" y1="-79.375" x2="-58.7375" y2="-104.835" width="0" layer="19" extent="1-1"/>
@@
 <wire x1="37.7825" y1="-83.185" x2="-63.16" y2="-110.1725" width="0" layer="19" extent="1-1"/>
 </signal>
+<signal name="N$45">
+<contactref element="3D3" pad="A"/>
+</signal>
 </signals>

Commit message: .
Parts:
- moved DIS1 4.18 mm to (61.9, 295.9)
Changed lines of the file:
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@@
 <dimension x1="36.195" y1="261.9375" x2="35.56" y2="240.665" x3="2.2225" y3="251.30125" layer="21" dtype="vertical"/>
 <dimension x1="6.6675" y1="239.0775" x2="32.385" y2="233.9975" x3="19.52625" y3="265.7475" layer="21" dtype="horizontal"/>
+<dimension x1="21.2725" y1="221.2975" x2="44.7675" y2="209.2325" x3="33.02" y3="326.39" layer="21" dtype="horizontal"/>
+<dimension x1="135.5725" y1="273.05" x2="195.2625" y2="239.7125" x3="-29.845" y3="256.38125" layer="21" dtype="vertical"/>
+<dimension x1="71.755" y1="214.9475" x2="102.235" y2="209.2325" x3="86.995" y3="323.5325" layer="21" dtype="horizontal"/>
+<dimension x1="150.8125" y1="302.26" x2="178.1175" y2="218.7575" x3="-40.005" y3="260.50875" layer="21" dtype="vertical"/>
 </plain>
 <attributes>
@@
 <element name="T5" library="pinhead" package="1X01" value="" x="57.4675" y="225.1075"/>
 <element name="T6" library="pinhead" package="1X01" value="" x="50.165" y="225.425"/>
-<element name="DIS1" library="display-lcd" package="TUXGR_16X2_R2" value="TUXGR_16X2_R2" x="61.2775" y="291.7825">
-<attribute name="OC_NEWARK" value="unknown" x="51.435" y="156.21" size="1.778" layer="27" display="off"/>
-<attribute name="MPN" value="" x="51.435" y="156.21" size="1.778" layer="27" display="off"/>
-<attribute name="MF" value="" x="51.435" y="156.21" size="1.778" layer="27" display="off"/>
-<attribute name="OC_FARNELL" value="unknown" x="51.435" y="156.21" size="1.778" layer="27" display="off"/>
+<element name="DIS1" library="display-lcd" package="TUXGR_16X2_R2" value="TUXGR_16X2_R2" x="61.9125" y="295.91">
+<attribute name="OC_NEWARK" value="unknown" x="52.07" y="160.3375" size="1.778" layer="27" display="off"/>
+<attribute name="MPN" value="" x="52.07" y="160.3375" size="1.778" layer="27" display="off"/>
+<attribute name="MF" value="" x="52.07" y="160.3375" size="1.778" layer="27" display="off"/>
+<attribute name="OC_FARNELL" value="unknown" x="52.07" y="160.3375" size="1.778" layer="27" display="off"/>
 </element>
 <element name="D8" library="v-reg" package="TO92-CLP" value="TL431" x="52.705" y="262.5725" rot="R90"/>
@@
 <wire x1="28.981" y1="287.02" x2="28.6635" y2="280.67" width="0" layer="19" extent="1-1"/>
 <wire x1="66.675" y1="273.05" x2="51.435" y2="273.05" width="0" layer="19" extent="1-1"/>
-<wire x1="29.2775" y1="307.2825" x2="28.981" y2="287.02" width="0" layer="19" extent="1-1"/>
+<wire x1="29.9125" y1="311.41" x2="28.981" y2="287.02" width="0" layer="19" extent="1-1"/>
 <wire x1="121.92" y1="257.175" x2="72.0725" y2="254.3175" width="0" layer="19" extent="1-16"/>
 <wire x1="130.4925" y1="260.35" x2="121.92" y2="257.175" width="0" layer="19" extent="16-16"/>
@@
 <contactref element="J_PD4" pad="1"/>
 <contactref element="DD1" pad="2"/>
-<wire x1="59.442590625" y1="256.397515625" x2="60.6425" y2="256.8575" width="0.3048" layer="16"/>
-<wire x1="60.6425" y1="256.8575" x2="60.6425" y2="259.2705" width="0.3048" layer="16"/>
+<wire x1="59.442590625" y1="256.397515625" x2="60.6425" y2="256.54" width="0.3048" layer="16"/>
+<wire x1="60.6425" y1="256.54" x2="60.6425" y2="259.2705" width="0.3048" layer="16"/>
 </signal>
 <signal name="N$12">

Commit message: sch
Parts:
- removed 3C15: 22u/100V, resistor:E2,5-6
- removed 3D3, 3D4: RK19(1N5819), diode:SMB
- added D1: UF4007, diode:DO41-10
- 3L1A: value 230uH -> 100uH
- 3L1B: value 230uH -> 6800uH
- moved 3R10 26.6 mm to (-78.1, -153.0)
- renumbered 3L3 to 3L1A, 3L4 to 3L1B
Connections:
- net N$24 renamed Z_GREEN
- net N$56 renamed Z_BLUE
- removed net N$45: 3D3.A
- removed net N$57: 3R10.2, DA7.2, DA7.4, VT1.D
- removed net N$73: 3D4.A, 3L1B.2
- new net Z_YELLOW: 3L1B.2, D1.A
- net GND: no longer 3C15.-
- net N$12: now also 3R10.1, DA7.2, DA7.4, VT1.D; no longer 3C15.+, 3D3.C
- net N$25: now also 3R10.2; no longer 3R10.1
- net N$94: now also D1.C; no longer 3D4.C
Changed lines of the file:
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@@
 <element name="3R1B2" library="resistor" package="R0805" value="2R" x="-78.105" y="-90.17"/>
 <element name="DA7" library="mc34063-2" package="SOIC8" value="MC34063AD" x="-56.8325" y="-102.235"/>
-<element name="3L3" library="rcl" package="6000-XXXX-RC" value="230uH" x="-65.7225" y="-99.3775"/>
-<element name="3D3" library="diode" package="SMB" value="RK19(1N5819)" x="-60.96" y="-110.1725"/>
+<element name="3L1A" library="rcl" package="6000-XXXX-RC" value="100uH" x="-65.7225" y="-99.3775"/>
 <element name="3C14" library="resistor" package="C0805K" value="1n" x="-61.9125" y="-140.97"/>
 <element name="3R9" library="resistor" package="R0805" value="120k" x="38.4175" y="-72.39"/>
-<element name="3R10" library="resistor" package="R0805" value="2K" x="-64.4525" y="-130.175"/>
 <element name="3R11" library="resistor" package="R0805" value="180R" x="-58.1025" y="-130.175"/>
 <element name="3R12" library="resistor" package="R0805" value="1R" x="-51.7525" y="-130.175"/>
@@
 <element name="T8" library="transistor" package="TO92-ECB" value="" x="-46.6725" y="-111.125"/>
 <element name="3R1B4" library="resistor" package="R0805" value="2R" x="-47.625" y="-124.46"/>
-<element name="3C15" library="resistor" package="E2,5-6" value="22u/100V" x="39.0525" y="-83.185"/>
-<element name="3L4" library="rcl" package="6000-XXXX-RC" value="230uH" x="31.4325" y="-79.375"/>
-<element name="3D4" library="diode" package="SMB" value="RK19(1N5819)" x="30.1625" y="-90.4875"/>
+<element name="3L1B" library="rcl" package="6000-XXXX-RC" value="6800uH" x="31.4325" y="-79.375"/>
 <element name="3C16" library="resistor" package="E2,5-6" value="22u/100V" x="29.5275" y="-97.79"/>
 <element name="Q1" library="transistor-pnp" package="TO92-CBE" value="2N4126" x="13.335" y="254.3175" rot="R270"/>
@@
 <element name="R35" library="rcl" package="RTRIM3296W" value="" x="15.24" y="241.935" rot="R90"/>
 <element name="J_PD4" library="jumper" package="SJ" value="" x="60.6425" y="260.0325" rot="MR90"/>
+<element name="D1" library="diode" package="DO41-10" value="UF4007" x="-73.9775" y="-147.0025"/>
+<element name="3R10" library="resistor" package="R0805" value="2K" x="-78.105" y="-153.035"/>
 </elements>
 <signals>
@@
 <contactref element="T8" pad="E"/>
 <contactref element="R4" pad="1"/>
-<contactref element="3C15" pad="-"/>
 <contactref element="3C16" pad="-"/>
 <contactref element="R26" pad="1"/>
@@
 <wire x1="-60.9125" y1="-140.97" x2="-46.2525" y2="-130.175" width="0" layer="19" extent="1-1"/>
 <wire x1="30.7975" y1="-97.79" x2="-44.3925" y2="-103.5425" width="0" layer="19" extent="1-1"/>
-<wire x1="40.3225" y1="-83.185" x2="30.7975" y2="-97.79" width="0" layer="19" extent="1-1"/>
 <wire x1="1.27" y1="224.155" x2="-37.83" y2="100.33" width="0" layer="19" extent="1-16"/>
 <wire x1="17.78" y1="241.935" x2="17.78" y2="243.5225" width="0" layer="19" extent="16-16"/>
@@
 <wire x1="-56.1975" y1="-104.835" x2="-62.9125" y2="-140.97" width="0" layer="19" extent="1-1"/>
 </signal>
-<signal name="N$24">
+<signal name="Z_GREEN">
 <contactref element="DA7" pad="1"/>
-<contactref element="3L3" pad="2"/>
-<contactref element="3L4" pad="1"/>
+<contactref element="3L1A" pad="2"/>
+<contactref element="3L1B" pad="1"/>
 <wire x1="-63.2225" y1="-99.3775" x2="-58.7375" y2="-104.835" width="0" layer="19" extent="1-1"/>
 <wire x1="28.9325" y1="-79.375" x2="-58.7375" y2="-104.835" width="0" layer="19" extent="1-1"/>
 </signal>
 <signal name="N$25">
+<contactref element="DA7" pad="5"/>
 <contactref element="3R9" pad="1"/>
-<contactref element="DA7" pad="5"/>
-<contactref element="3R10" pad="1"/>
-<wire x1="-54.9275" y1="-99.635" x2="-65.3025" y2="-130.175" width="0" layer="19" extent="1-1"/>
+<contactref element="3R10" pad="2"/>
+<wire x1="-54.9275" y1="-99.635" x2="-77.255" y2="-153.035" width="0" layer="19" extent="1-1"/>
 <wire x1="37.5675" y1="-72.39" x2="-54.9275" y2="-99.635" width="0" layer="19" extent="1-1"/>
 </signal>
@@
 <wire x1="-58.7375" y1="-99.635" x2="-57.2525" y2="-130.175" width="0" layer="19" extent="1-1"/>
 </signal>
-<signal name="N$56">
+<signal name="Z_BLUE">
 <contactref element="DA7" pad="7"/>
 <contactref element="3R11" pad="1"/>
 <contactref element="3R12" pad="2"/>
 <contactref element="3R1B3" pad="2"/>
-<contactref element="3L3" pad="1"/>
+<contactref element="3L1A" pad="1"/>
 <contactref element="3R1B4" pad="2"/>
 <wire x1="-54.395" y1="-124.46" x2="-58.9525" y2="-130.175" width="0" layer="19" extent="1-1"/>
@@
 <wire x1="-68.2225" y1="-99.3775" x2="-57.4675" y2="-99.635" width="0" layer="19" extent="1-1"/>
 </signal>
-<signal name="N$57">
-<contactref element="DA7" pad="4"/>
-<contactref element="DA7" pad="2"/>
-<contactref element="VT1" pad="D"/>
-<contactref element="3R10" pad="2"/>
-<wire x1="-57.4675" y1="-104.835" x2="-63.6025" y2="-130.175" width="0" layer="19" extent="1-1"/>
-<wire x1="-54.9275" y1="-104.835" x2="-57.4675" y2="-104.835" width="0" layer="19" extent="1-1"/>
-<wire x1="-46.6725" y1="-96.2425" x2="-54.9275" y2="-104.835" width="0" layer="19" extent="1-1"/>
-</signal>
 <signal name="!BUTTON1">
 <contactref element="R29" pad="1"/>
 </signal>
 <signal name="N$94">
+<contactref element="3C16" pad="+"/>
+<contactref element="D1" pad="C"/>
 <contactref element="3R9" pad="2"/>
-<contactref element="3D4" pad="C"/>
-<contactref element="3C16" pad="+"/>
-<wire x1="27.9625" y1="-90.4875" x2="28.2575" y2="-97.79" width="0" layer="19" extent="1-1"/>
-<wire x1="39.2675" y1="-72.39" x2="27.9625" y2="-90.4875" width="0" layer="19" extent="1-1"/>
+<wire x1="28.2575" y1="-97.79" x2="-79.0575" y2="-147.0025" width="0" layer="19" extent="1-1"/>
+<wire x1="39.2675" y1="-72.39" x2="28.2575" y2="-97.79" width="0" layer="19" extent="1-1"/>
 </signal>
 <signal name="N$95">
@@
 <wire x1="-48.9525" y1="-103.5425" x2="-46.6725" y2="-111.125" width="0" layer="19" extent="1-1"/>
 </signal>
-<signal name="N$73">
-<contactref element="3D4" pad="A"/>
-<contactref element="3L4" pad="2"/>
-<wire x1="33.9325" y1="-79.375" x2="32.3625" y2="-90.4875" width="0" layer="19" extent="1-1"/>
+<signal name="Z_YELLOW">
+<contactref element="3L1B" pad="2"/>
+<contactref element="D1" pad="A"/>
+<wire x1="33.9325" y1="-79.375" x2="-68.8975" y2="-147.0025" width="0" layer="19" extent="1-1"/>
 </signal>
 <signal name="N$90">
@@
 </signal>
 <signal name="N$12">
-<contactref element="3D3" pad="C"/>
-<contactref element="3C15" pad="+"/>
-<wire x1="37.7825" y1="-83.185" x2="-63.16" y2="-110.1725" width="0" layer="19" extent="1-1"/>
-</signal>
-<signal name="N$45">
-<contactref element="3D3" pad="A"/>
+<contactref element="3R10" pad="1"/>
+<contactref element="DA7" pad="4"/>
+<contactref element="DA7" pad="2"/>
+<contactref element="VT1" pad="D"/>
+<wire x1="-57.4675" y1="-104.835" x2="-78.955" y2="-153.035" width="0" layer="19" extent="1-1"/>
+<wire x1="-54.9275" y1="-104.835" x2="-57.4675" y2="-104.835" width="0" layer="19" extent="1-1"/>
+<wire x1="-46.6725" y1="-96.2425" x2="-54.9275" y2="-104.835" width="0" layer="19" extent="1-1"/>
 </signal>
 </signals>

Commit message: .
Parts:
- removed 3D2: RK19(1N5819), diode:SMB
- removed 3L1B: 6800uH, rcl:6000-XXXX-RC
- removed 3L2: 230uH, rcl:6000-XXXX-RC
- added 3C15: 100n, resistor:C025-025X050
- added 3L2B: (no value), pinhead:1X01
- 3C16: device resistor:E2,5-6 -> resistor:E5-8,5
- 3R9: value 120k -> 130k
- moved 3R10 483.1 mm to (178.1, 256.5)
- moved D1 483.1 mm to (182.2, 262.6)
- moved 3R1B2 468.7 mm to (218.4, 272.7)
- moved T7 468.7 mm to (220.0, 277.8)
- moved 3R11 468.1 mm to (207.0, 255.6), flipped to the bottom, turned to 180 degrees
- moved 3C17 451.9 mm to (202.2, 256.2), turned to 180 degrees
- moved 3L1A 448.9 mm to (209.9, 255.0), turned to 270 degrees
- moved 3C14 442.3 mm to (227.3, 193.7), flipped to the bottom
- moved 3R12 442.3 mm to (237.5, 204.5), flipped to the bottom
- moved 3R1B3 442.3 mm to (234.0, 210.2), flipped to the bottom
- moved 3R1B4 442.3 mm to (241.6, 210.2), flipped to the bottom
- moved R29 442.3 mm to (231.5, 198.8), flipped to the bottom
- moved R30 442.3 mm to (236.5, 198.8), flipped to the bottom
- moved R4 442.3 mm to (243.8, 204.5), flipped to the bottom
- moved T8 442.3 mm to (242.6, 223.5)
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Connections:
- removed net N$26: 3D2.A, 3L2.2, DA5.1
- removed net N$92: 2L4.1, 3C6.+, 3C7.1, 3D2.C, 3R5.2
- removed net N$94: 3C16.+, 3R9.2, D1.C
- new net N$24: 3C15.2, 3C16.+, 3R9.2, D1.C
- new net N$45: 2L4.1, 3C6.+, 3C7.1
- net GND: now also 3C15.1
- net N$51: no longer 3R5.1, 3R6.1
- net N$54: no longer 3L2.1
- net N$58: no longer 3R6.2
- net Z_GREEN: no longer 3L1B.1
- net Z_YELLOW: now also 3L2B.1; no longer 3L1B.2
Routing:
- net N$92: track 26.1 -> 0.00 mm
- net N$26: track 8.12 -> 0.00 mm
- net N$51: track 4.83 -> 1.74 mm
- net N$54: track 10.8 -> 8.55 mm

Commit message: .
Parts:
- removed 3C6: 22u/100V, resistor:E2,5-6
- removed 3C7: 100n, resistor:C0805K
- removed 3L1A: 100uH, rcl:6000-XXXX-RC
- added 3L2G, 3L2Y: (no value), b333:1X01
- added L: L, b333:L
- 3C16: device resistor:E5-8,5 -> resistor:TT5D9L
- 3L2B: device pinhead:1X01 -> b333:1X01
- moved 3R9 323.8 mm to (170.5, 223.2), turned to 180 degrees
- moved DIS1 119.2 mm to (169.9, 245.4)
- moved 3R1B4 59.8 mm to (205.1, 257.5), turned to 180 degrees
- moved 3C14 59.1 mm to (200.7, 246.4), turned to 270 degrees
- moved 3R12 58.4 mm to (205.1, 253.0), turned to 180 degrees
- moved 3R1B3 53.5 mm to (205.1, 255.3), turned to 180 degrees
- moved R29 44.7 mm to (216.9, 241.0), turned to 180 degrees
- moved VT1 41.0 mm to (201.6, 237.2)
- moved R4 39.5 mm to (218.8, 234.9), turned to 270 degrees
- moved R30 36.5 mm to (218.4, 230.5), turned to 270 degrees
- moved 3C15 32.7 mm to (208.0, 238.8), turned to 270 degrees
- moved T8 30.0 mm to (214.3, 233.7), turned to 270 degrees
- moved 3R10 10.3 mm to (183.8, 248.0), turned to 90 degrees
- moved 3C16 9.92 mm to (206.1, 238.8), turned to 90 degrees
- moved 3C17 8.39 mm to (198.1, 248.9), turned to 270 degrees
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Connections:
- removed net N$45: 2L4.1, 3C6.+, 3C7.1
- net +40V: now also 3C10.2; no longer 3C10.1
- net GND: now also 3C10.1; no longer 3C10.2, 3C6.-, 3C7.2
- net N$24: now also 2L4.1
- net Z_BLUE: now also 3L2B.1; no longer 3L1A.1
- net Z_GREEN: now also 3L2G.1; no longer 3L1A.2
- net Z_YELLOW: now also 3L2Y.1; no longer 3L2B.1
Routing:
- net GND: track 225.5 -> 223.2 mm
