File: HW/EAGLE/b333.brd (EAGLE design)
At the start: 80.6 x 52.4 mm, 208 parts, among them Q1 2N4126, Q2 2N4126, Q5 NMOSD, X1 USB MICRO

Commit message: .
Parts:
- removed 3C5: 1n, resistor:C0805K
- removed 3C8: 100u, resistor:E2,5-6
- removed 3R1B1, 3R1B2: 2R, resistor:R0805
- removed 3R5: 62K, resistor:R0805
- removed 3R6: 2K, resistor:R0805
- removed 3R7: 180R, resistor:R0805
- removed 3R8: 1R, resistor:R0805
- removed DA5: MC34063AD, mc34063-2:SOIC8
- removed R18, R25, R30: 10k, resistor:R0805
- removed T7, T8: (no value), transistor:TO92-ECB
- removed VT5: NMOSD, DSS:DPACK_1
- added SL1, SL2: (no value), b333:1X01
- 3R12, 3R1B3, 3R1B4: device resistor:R0805 -> resistor:R1206
- R8: value 100k -> 10k
- moved R8 383.7 mm to (-78.1, -82.9), flipped to the top, turned to 0 degrees
- moved D11 63.0 mm to (202.9, 218.1), turned to 90 degrees
- moved D10 58.2 mm to (202.9, 223.5), turned to 90 degrees
- moved R13 56.4 mm to (193.7, 215.9), turned to 180 degrees
- moved VT6 56.2 mm to (197.2, 219.1), turned to 270 degrees
- moved D9 54.0 mm to (202.9, 228.9), turned to 90 degrees
- moved R16 52.6 mm to (193.4, 219.1), turned to 180 degrees
- moved 3C13 51.6 mm to (190.5, 217.8), turned to 270 degrees
- moved 5MA 50.4 mm to (197.2, 225.1), turned to 0 degrees
- moved R12 49.7 mm to (199.7, 229.6), turned to 270 degrees
- moved ZEN_K1 47.9 mm to (191.1, 221.6), turned to 270 degrees
- moved R10 46.6 mm to (197.2, 229.6), turned to 270 degrees
- moved R15 45.0 mm to (185.7, 220.3), turned to 90 degrees
- moved R11 43.7 mm to (194.6, 229.6), turned to 270 degrees
- moved ZEN_A1 40.3 mm to (190.5, 228.3), turned to 270 degrees
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Connections:
- removed net !BUTTON: R18.1
- removed net N$19: R18.2, T7.B
- removed net N$23: 3C5.1, DA5.3
- removed net N$51: DA5.5
- removed net N$53: 3R7.2, DA5.8
- removed net N$54: 3R1B1.2, 3R1B2.2, 3R7.1, 3R8.2, DA5.7
- removed net N$58: DA5.2, DA5.4, VT5.D
- net +5V/2: no longer R25.2, R30.2
- net GND: now also SL1.1; no longer 3C5.2, 3C8.-, R4.1, T7.E, T8.E, VT5.S
- net N$21: now also R4.1, VT4.C; no longer R25.1, T7.C, VT5.G
- net N$95: now also VT4.B; no longer T8.B
- net N$96: no longer R30.1, T8.C
- net V+: now also VT4.E; no longer 3C8.+, 3R1B1.1, 3R1B2.1, 3R8.1, DA5.6
Routing:
- net GND: track 223.2 -> 193.7 mm
- net Z_BLUE: track 0.00 -> 16.3 mm
- net N$12: track 0.00 -> 15.9 mm
- net N$58: track 14.4 -> 0.00 mm
- net N$24: track 0.00 -> 14.4 mm
- net V+: track 46.7 -> 32.7 mm
- net PC3: track 51.3 -> 37.9 mm
- net N$25: track 0.00 -> 8.76 mm
- net N$54: track 8.55 -> 0.00 mm
- net N$23: track 7.51 -> 0.00 mm
- net N$22: track 0.00 -> 6.62 mm
- net N$53: track 4.51 -> 0.00 mm
- net Z_GREEN: track 0.00 -> 2.97 mm
- net Z_YELLOW: track 0.00 -> 2.54 mm
- net N$52: track 0.00 -> 2.06 mm
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