File: HW/EAGLE/b333.brd (EAGLE design)
At the start: 80.6 x 52.4 mm, 195 parts, among them Q1 2N4126, Q2 2N4126, Q5 NMOSD, X1 USB MICRO

Commit message: .
Parts:
- DIS1: device display-lcd:TUXGR_16X2_R2 -> b333:TUXGR_16X2_R2
- moved R8 525.3 mm to (301.6, 280.0), turned to 270 degrees
- moved 3C9 163.4 mm to (344.8, 253.0), turned to 270 degrees
- moved 2L4 160.3 mm to (333.4, 267.7), turned to 180 degrees
- moved 3C17 158.8 mm to (346.4, 247.0), turned to 180 degrees
- moved D1 131.9 mm to (318.5, 267.7)
- moved 3C15 131.5 mm to (322.3, 256.2), turned to 270 degrees
- moved SL1 129.7 mm to (324.8, 275.6)
- moved 3L2Y 129.3 mm to (318.1, 275.9)
- moved 3R9 121.6 mm to (312.7, 269.2), turned to 180 degrees
- moved R29 118.6 mm to (294.6, 278.1), flipped to the top, turned to 0 degrees
- moved VT4 118.2 mm to (298.4, 280.7)
- moved SL2 116.2 mm to (314.0, 261.6), turned to 180 degrees
- moved 3C14 116.0 mm to (309.9, 276.2), turned to 180 degrees
- moved R4 115.9 mm to (302.9, 277.2), flipped to the top, turned to 0 degrees
- moved VT1 114.8 mm to (309.2, 280.7)
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Connections:
- new net GND1: DIS1.1
- net GND: no longer DIS1.1, SL1.1
Routing:
- net GND: track 193.7 -> 178.5 mm, vias 3 -> 4
- net N$24: track 14.4 -> 0.00 mm
- net N$25: track 8.76 -> 1.66 mm
- net N$21: track 0.00 -> 5.64 mm
- net N$96: track 0.00 -> 4.60 mm, vias 0 -> 1
- net N$95: track 0.00 -> 2.96 mm
- net Z_GREEN: track 2.97 -> 5.84 mm
- net N$22: track 6.62 -> 3.76 mm
- net Z_BLUE: track 16.3 -> 14.0 mm
- net N$12: track 15.9 -> 18.0 mm
- net N$52: track 2.06 -> 3.88 mm
- net Z_YELLOW: track 2.54 -> 3.19 mm

Commit message: .
Parts:
- 3C16: device resistor:TT5D9L -> ct-pack:TT5D9L
- moved 3C15 133.3 mm to (190.5, 235.9), turned to 0 degrees
- moved SL1 132.6 mm to (195.6, 246.1)
- moved 2L4 120.9 mm to (215.9, 239.1), turned to 270 degrees
- moved 3C14 119.5 mm to (192.1, 255.9), turned to 0 degrees
- moved 3L2Y 115.2 mm to (204.8, 255.3)
- moved 3C9 113.6 mm to (232.1, 239.1), turned to 90 degrees
- moved R4 112.5 mm to (192.4, 256.2)
- moved VT4 112.2 mm to (188.3, 259.4), turned to 90 degrees
- moved R8 112.1 mm to (191.5, 259.1)
- moved VT1 112.1 mm to (199.1, 259.7)
- moved 3C10 112.1 mm to (190.5, 215.9)
- moved 3C13 112.1 mm to (193.7, 203.2)
- moved D10 112.1 mm to (206.1, 208.9)
- moved D11 112.1 mm to (206.1, 203.5)
- moved D9 112.1 mm to (206.1, 214.3)
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Routing:
- net GND: track 178.5 -> 208.6 mm
- net V+: track 32.4 -> 58.4 mm
- net Z_BLUE: track 14.0 -> 26.4 mm
- net Z_GREEN: track 5.84 -> 1.91 mm
- net N$25: track 1.66 -> 4.93 mm
- net N$22: track 3.76 -> 5.30 mm
- net N$52: track 3.88 -> 5.18 mm
- net N$12: track 18.0 -> 17.3 mm

Commit message: .sh
Parts:
- removed 0S1: TEST, switch-omron:B3F-10XX
- removed 1Q3, 1Q4, Q5: NMOSD, DSS:DPACK_1
- removed 1R14: 270, resistor:R1206W
- removed 1R15: 27K, resistor:R0805
- removed 1R6: 470K, resistor:0207/10
- removed 1R7, R1: 1M, resistor:R0805
- removed 1R8: 300, resistor:R0805
- removed 1RC1: 22K, resistor:R0805
- removed 1RC2*: 4K3, resistor:R1206W
- removed 3C1: 100u, resistor:E2,5-6
- removed 3C2: 1n, resistor:C0805K
- removed 3C3: 47u/50V, resistor:E2,5-6
- removed 3C4, C2: 100n, resistor:C0805K
- removed 3D1: 1N5819, diode:DO41-10
- removed 3L1: 180uH, inductor-neosid:SD12_1000
- removed 3R1, 3R1B: 1R, resistor:R0805
- removed 3R2: 180R, resistor:R0805
- removed 3R3, R2, R3: 2K, resistor:R0805
- removed 3R4: 62K, resistor:R0805
- removed 4R1, 4R2: 100, resistor:R0805
- removed 4R3: 270, resistor:R0805
- removed 4R4: 47K, resistor:R1206W
- removed 4R5: 47K, resistor:R0805
- removed 4Y1, 4Y2: РЭС55А, relay_ussr:РЭС55А
- removed C1: 100n, resistor:C0805
- removed D4: MC34063AD, mc34063:SOIC8
- removed D5, D6: (no value), diode:SOD80C
- removed J1, J2, J3, J4: (no value), jumper:SJ
- removed OK1: PC817, optocoupler:DIL04
- removed R5: 20K, resistor:R0805
- removed R6: 180K, resistor:R0805
- removed R7: 10K, resistor:R1206W
- removed S1: 9077-2, switch-misc:9077-2
- removed T1, T2, T3, ZEN_A, ZEN_K: (no value), pinhead:1X01
- removed VD2: LL4148, diode:DO35-7
- added 3R5: 20K, resistor:R0805
- added R18: 10.0k, resistor:R0805
- added TEST2: TT-P, transistor_tester:TT-P
- added U$8: (no value), b333:F18650
- added VT3: FS8205A, FS8205A:TSSOP-8
- added X2: USB MICRO, SmartPrj:CON2_USB_MICRO_B_AT
- 3C10, 3C13: device resistor:C0805K -> resistor:C025-025X050
- 3C15: device resistor:C025-025X050 -> resistor:C050-025X075
- 3C9: value 47u/50V -> 10u/100V
- 3R9: value 130k -> 120k
- R16: value 180.0k -> 330.0k
- VT6: value BF423 -> КТ502
- moved 1RC2 183.9 mm to (76.8, 106.4), flipped to the bottom, turned to 180 degrees
- moved 1R17 170.6 mm to (72.1, 115.3)
- moved D12 169.1 mm to (53.0, 93.7)
- moved J_PD4 169.1 mm to (105.1, 96.8)
- moved R14 169.1 mm to (57.1, 96.8)
- moved R17 169.1 mm to (62.9, 96.8)
- moved R28 169.1 mm to (67.6, 96.8)
- moved R9 169.1 mm to (54.6, 93.7)
- moved T4 169.1 mm to (106.4, 62.2)
- moved T6 169.1 mm to (94.6, 62.2)
- moved 1C13 169.1 mm to (93.0, 87.0)
- moved 1C6 169.1 mm to (93.0, 88.9)
- moved 1C7 169.1 mm to (107.0, 92.4)
- moved 1C8 169.1 mm to (109.5, 90.5)
- moved 1C9 169.1 mm to (112.1, 90.5)
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Connections:
- net +40V renamed +90.5V
- removed net KEY: 0S1.1, 0S1.2, D6.A, R2.1, S1.1, S1.4
- removed net N$1: 4R4.1, 4R5.1, Q5.G
- removed net N$10: 1Q4.D, 3C2.2, 3R3.1, D4.4, J1.1, J2.1, ZEN_A.1
- removed net N$11: 1R14.1
- removed net N$110: 4R1.1, 4R2.1
- removed net N$114: 1R6.1
- removed net N$115: 1R6.2
- removed net N$18: R16.2, VT6.C, ZEN_K1.1
- removed net N$2: D5.A
- removed net N$20: 1R7.1, D6.C, OK1.3
- removed net N$27: 3C2.1, D4.3
- removed net N$28: 3D1.A, 3L1.2, D4.1, J3.1
- removed net N$29: 3R3.2, 3R4.1, D4.5, J2.2
- removed net N$30: 3C3.+, 3C4.1, 3D1.C, 3R4.2, J3.2, J4.2, R7.2
- removed net N$31: 4R3.2, 4Y1.2, 4Y2.2
- removed net N$32: 3R2.2, D4.8
- removed net N$33: 3L1.1, 3R1.2, 3R1B.2, 3R2.1, D4.7
- removed net N$34: 1R8.2, OK1.1
- removed net N$46: 4R1.2, 4Y1.P
- removed net N$47: 4R2.2, 4Y2.P
- removed net N$48: 1Q3.G, 1R7.2, R1.1
- removed net N$49: D4.2, J1.2, VD2.A
- removed net N$5: D5.C
- removed net N$50: 1Q4.G, R2.2, R3.1
- removed net N$6: 1RC1.2, 1RC2*.2
- removed net N$7: 4Y1.1, 4Y2.1, Q5.D
- removed net N$9: J4.1, R6.2, R7.1, ZEN_K.1
- removed net PC1: 4Y2.O
- removed net PC2: 4Y1.O
- removed net PC4: 4R4.2
- removed net PD6: 1R8.1
- removed net PD7: 1R15.2, C2.1, VD2.C
- removed net V-: 1Q3.S, R1.2
- new net N$19: 2L4.1, 3C15.2, 3C16.+, 3R5.2, D1.C
- new net N$23: 3R5.1, 3R9.2
- new net VBUS: X2.P1
- new net ZENER_A: DD1.26, R18.2, VT6.C, ZEN_K1.1
- net +5V: no longer 0S1.3, 0S1.4, 1R14.2, 1R15.1, 1RC1.1, 4R3.1
- net GND: no longer 1Q3.D, 1Q4.S, 1RC2*.1, 3C1.-, 3C3.-, 3C4.2, 4R5.2, 4Y1.G, 4Y2.G, C1.2, C2.2, OK1.2, Q5.S, R3.2, R5.1
- net N$24: now also R16.2, R18.1; no longer 2L4.1, 3C15.2, 3C16.+, 3R9.2, D1.C
- net PC3: no longer C1.1, DD1.26, R5.2, R6.1
- net V+: no longer 3C1.+, 3R1.1, 3R1B.1, D4.6, OK1.4, S1.2, S1.5
Routing:
- net N$40: track 100.3 -> 0.00 mm
- net N$38: track 100.3 -> 0.00 mm
- net N$36: track 99.7 -> 0.00 mm
- net GND: track 208.6 -> 268.5 mm
- net PC3: track 37.9 -> 0.00 mm, vias 2 -> 0
- net ZENER_A: track 0.00 -> 33.2 mm, vias 0 -> 1
- net N$39: track 29.2 -> 0.00 mm
- net N$37: track 29.2 -> 0.00 mm
- net N$35: track 29.2 -> 0.00 mm
- net N$19: track 0.00 -> 19.8 mm
- net N$18: track 9.56 -> 0.00 mm
- net Z_BLUE: track 26.4 -> 20.1 mm
- net V+: track 58.4 -> 55.4 mm
- net N$22: track 5.30 -> 7.87 mm
- net N$52: track 5.18 -> 2.70 mm
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Other:
- board outline removed

Commit message: .
Parts:
- renumbered 3C10 to 6C6, 3C13 to 6C7, 3C14 to 6C2, 3C15 to 6C4, 3C16 to 6C3, 3C17 to 6C1, 3C9 to 6C5, 3R10 to 6R5, 3R11 to 6R2, 3R12 to 6R1C, 3R1B3 to 6R1B, 3R1B4 to 6R1A, 3R5 to 6R3, 3R9 to 6R4, D1 to 6VD1, D10 to 6VD3, D11 to 6VD4, D9 to 6VD2, R10 to 6R7, R11 to 6R8, R12 to 6R6, R13 to 6R9, R15 to 6R12, R16 to 6R11, R18 to 6R10, R29 to 6R13, R4 to 6R15, R8 to 6R14, VT1 to 6VT2, VT4 to 6VT3

Commit message: -rcllbr
Parts:
- 2L2: value 220uH -> 100uH; device rcl:6000-XXXX-RC -> ct-pack:LH7X10MM
- moved 2L2 8.99 mm to (258.4, 27.0)
- moved 2L3 1.27 mm to (234.0, 27.9)
Routing:
- net N$14: track 9.94 -> 36.7 mm
- net N$13: track 9.26 -> 21.7 mm
Changed lines of the file:
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@@
 <wire x1="254.635" y1="103.505" x2="254.635" y2="131.445" width="0.3048" layer="47"/>
 <wire x1="254.635" y1="131.445" x2="237.1725" y2="131.445" width="0.3048" layer="47"/>
+<dimension x1="237.49" y1="84.7725" x2="237.49" y2="93.6625" x3="248.92" y3="89.2175" layer="21" dtype="vertical"/>
+<dimension x1="254" y1="24.765" x2="259.08" y2="31.75" x3="269.875" y3="28.2575" layer="21" dtype="vertical"/>
 </plain>
 <attributes>
@@
 <elements>
 <element name="DA3" library="mc34063-2" package="SOIC8" value="MC34063AD" x="248.6025" y="21.59" rot="R180"/>
-<element name="2L2" library="rcl" package="6000-XXXX-RC" value="220uH" x="252.4125" y="20.32" smashed="yes" rot="R90">
-<attribute name="NAME" x="250.3199" y="18.9894" size="1.27" layer="25" rot="R90"/>
-<attribute name="VALUE" x="258.8231" y="15.8144" size="1.27" layer="27" rot="R90"/>
+<element name="2L2" library="ct-pack" package="LH7X10MM" value="100uH" x="258.445" y="26.9875" smashed="yes" rot="R90">
+<attribute name="NAME" x="256.3524" y="25.6569" size="1.27" layer="25" rot="R90"/>
+<attribute name="VALUE" x="264.8556" y="22.4819" size="1.27" layer="27" rot="R90"/>
 </element>
 <element name="2C1" library="resistor" package="C0805K" value="0.47n" x="248.6025" y="27.305"/>
@@
 <element name="C5" library="resistor" package="C0805K" value="100n" x="243.84" y="24.765"/>
 <element name="C6" library="resistor" package="C0805K" value="100n" x="257.4925" y="18.7325" rot="R90"/>
-<element name="2L3" library="rcl" package="6000-XXXX-RC" value="220uH" x="233.9975" y="26.67" rot="R180"/>
+<element name="2L3" library="rcl" package="6000-XXXX-RC" value="220uH" x="233.9975" y="27.94" rot="R180"/>
 <element name="1C5" library="resistor" package="E2-5" value="1000u/6V" x="237.49" y="19.3675" rot="R270"/>
 <element name="C7" library="resistor" package="C0805K" value="100n" x="231.775" y="20.955" rot="R270"/>
@@
 <wire x1="251.12" y1="30.7975" x2="251.7775" y2="27.305" width="0.4064" layer="1"/>
 <wire x1="251.7775" y1="27.305" x2="250.5075" y2="24.19" width="0.4064" layer="1"/>
-<wire x1="250.5075" y1="24.19" x2="252.4125" y2="22.82" width="0.4064" layer="1"/>
+<wire x1="250.5075" y1="24.19" x2="264.445" y2="28.9875" width="0.4064" layer="1"/>
 </signal>
 <signal name="N$14">
@@
 <contactref element="2R6" pad="2"/>
 <contactref element="2L2" pad="1"/>
-<wire x1="252.515" y1="15.24" x2="252.4125" y2="17.82" width="0.4064" layer="1"/>
-<wire x1="252.4125" y1="17.82" x2="251.46" y2="16.8275" width="0.4064" layer="1"/>
+<wire x1="252.515" y1="15.24" x2="264.445" y2="24.9875" width="0.4064" layer="1"/>
+<wire x1="264.445" y1="24.9875" x2="251.46" y2="16.8275" width="0.4064" layer="1"/>
 <wire x1="251.46" y1="16.8275" x2="249.2375" y2="16.8275" width="0.4064" layer="1"/>
 <wire x1="249.2375" y1="16.8275" x2="249.2375" y2="18.99" width="0.4064" layer="1"/>
@@
 <wire x1="243.1415" y1="27.305" x2="242.84" y2="24.765" width="0.4064" layer="1"/>
 <wire x1="242.84" y1="24.765" x2="242.2525" y2="21.805" width="0.4064" layer="1"/>
-<wire x1="242.84" y1="24.765" x2="236.4975" y2="26.67" width="0.4064" layer="1"/>
+<wire x1="242.84" y1="24.765" x2="236.4975" y2="27.94" width="0.4064" layer="1"/>
 </signal>
 <signal name="+90.5V">
@@
 <contactref element="J_NO_LI" pad="1"/>
 <contactref element="DA6" pad="1"/>
-<wire x1="231.4975" y1="26.67" x2="231.775" y2="21.955" width="0" layer="19" extent="1-1"/>
+<wire x1="231.4975" y1="27.94" x2="231.775" y2="21.955" width="0" layer="19" extent="1-1"/>
 <wire x1="237.49" y1="20.3835" x2="231.775" y2="21.955" width="0" layer="19" extent="1-1"/>
-<wire x1="215.9875" y1="24.61" x2="231.4975" y2="26.67" width="0" layer="19" extent="1-1"/>
+<wire x1="215.9875" y1="24.61" x2="231.4975" y2="27.94" width="0" layer="19" extent="1-1"/>
 <wire x1="211.0105" y1="28.575" x2="211.19" y2="24.765" width="0" layer="19" extent="1-1"/>
 <wire x1="281.8525" y1="16.03" x2="237.49" y2="20.3835" width="0" layer="19" extent="1-1"/>

Commit message: .
Parts:
- added 2R1: 1R, resistor:R0805
- 2R7: value 18K -> 3.9k
- 2R8: value 56K -> 18k
- moved 2R5 4.77 mm to (253.0, 20.0), turned to 90 degrees
- moved 1C5 4.13 mm to (239.1, 15.6), turned to 90 degrees
- moved C4 2.93 mm to (262.6, 17.8)
- moved 2L3 2.42 mm to (234.9, 30.2)
- moved 2L2 1.42 mm to (257.2, 27.6)
Connections:
- net N$14: now also 2R1.2
- net V+: now also 2R1.1
Routing:
- net N$14: track 36.7 -> 21.6 mm
- net V+: track 55.4 -> 59.7 mm
- net N$15: track 7.43 -> 3.30 mm
- net N$13: track 21.7 -> 20.7 mm
- net N$17: track 18.6 -> 19.1 mm

Commit message: .
Parts:
- 2C1: value 0.47n -> 150
- 6R1A, 6R1B: value 2R -> 1R
- 6R1C: value 1R -> (none)
Connections:
- net N$25 renamed 5
Changed lines of the file:
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@@
 <attribute name="VALUE" x="263.5856" y="23.1169" size="1.27" layer="27" rot="R90"/>
 </element>
-<element name="2C1" library="resistor" package="C0805K" value="0.47n" x="248.6025" y="27.305"/>
+<element name="2C1" library="resistor" package="C0805K" value="150" x="248.6025" y="27.305"/>
 <element name="2R5" library="resistor" package="R0805" value="180R" x="253.0475" y="20.0025" rot="R90"/>
 <element name="2R6" library="resistor" package="R0805" value="1R" x="248.6025" y="15.24"/>
@@
 <element name="6R4" library="resistor" package="R0805" value="120k" x="228.6" y="100.33" rot="MR180"/>
 <element name="6R2" library="resistor" package="R0805" value="180R" x="225.7425" y="95.885" rot="MR90"/>
-<element name="6R1C" library="resistor" package="R1206" value="1R" x="221.9325" y="94.615" rot="MR180"/>
+<element name="6R1C" library="resistor" package="R1206" value="" x="221.9325" y="94.615" rot="MR180"/>
 <element name="6C1" library="resistor" package="E2,5-6" value="100u" x="212.4075" y="80.9625" rot="R270"/>
 <element name="6VT2" library="DSS" package="DPACK_1" value="NMOSD" x="220.98" y="108.9025" rot="MR90"/>
 <element name="6R15" library="resistor" package="R0805" value="100k" x="214.63" y="105.0925"/>
-<element name="6R1B" library="resistor" package="R1206" value="2R" x="221.9325" y="96.8375" rot="MR180"/>
+<element name="6R1B" library="resistor" package="R1206" value="1R" x="221.9325" y="96.8375" rot="MR180"/>
 <element name="6R13" library="resistor" package="R0805" value="10k" x="206.0575" y="110.1725"/>
-<element name="6R1A" library="resistor" package="R1206" value="2R" x="221.9325" y="92.3925" rot="MR180"/>
+<element name="6R1A" library="resistor" package="R1206" value="1R" x="221.9325" y="92.3925" rot="MR180"/>
 <element name="6C3" library="ct-pack" package="TT5D9L" value="22u/100V" x="212.09" y="87.3125"/>
 <element name="Q1" library="transistor-pnp" package="TO92-CBE" value="2N4126" x="57.785" y="91.1225" rot="R270"/>
@@
 <wire x1="217.17" y1="99.695" x2="219.9675" y2="99.3775" width="0.3048" layer="16"/>
 </signal>
-<signal name="N$25">
+<signal name="5">
 <contactref element="DA7" pad="5"/>
 <contactref element="6R4" pad="1"/>
