File: HW/EAGLE/b333.brd (EAGLE design)
At the start: 150 parts, among them Q1 2N4126, Q2 2N4126, X1 USB MICRO, X2 USB MICRO

Commit message: relbr
Parts:
- 2L3: device rcl:6000-XXXX-RC -> ct-pack:LV7X10MM
- DA4, DA4A, DA6: device v-reg:SOT89R -> ct-pack:SOT89R
- moved 4Y4 289.7 mm to (166.1, 60.0)
- moved 4Y3 253.7 mm to (166.1, 70.2)
- moved TEST2 3.84 mm to (191.5, 69.2)
- moved C4 3.42 mm to (261.3, 14.6)
Routing:
- net V+: track 59.7 -> 57.7 mm
- net N$17: track 19.1 -> 19.7 mm
Changed lines of the file:
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@@
 <dimension x1="51.1175" y1="75.8825" x2="76.835" y2="70.8025" x3="63.97625" y3="102.5525" layer="21" dtype="horizontal"/>
 <dimension x1="65.7225" y1="58.1025" x2="89.2175" y2="46.0375" x3="77.47" y3="163.195" layer="21" dtype="horizontal"/>
-<dimension x1="139.3825" y1="147.6375" x2="145.0975" y2="53.0225" x3="14.605" y3="100.33" layer="21" dtype="vertical"/>
-<dimension x1="231.4575" y1="47.625" x2="152.0825" y2="53.975" x3="191.77" y3="137.4775" layer="21" dtype="horizontal"/>
+<dimension x1="124.1425" y1="131.445" x2="127.635" y2="63.5" x3="295.5925" y3="97.4725" layer="21" dtype="vertical"/>
+<dimension x1="231.4575" y1="47.625" x2="152.0825" y2="53.975" x3="191.77" y3="144.4625" layer="21" dtype="horizontal"/>
 <dimension x1="68.58" y1="75.2475" x2="141.605" y2="131.7625" x3="269.24" y3="103.505" layer="21" dtype="vertical"/>
 <circle x="229.235" y="79.121" radius="1.5" width="0.4064" layer="1"/>
@@
 <dimension x1="237.49" y1="84.7725" x2="237.49" y2="93.6625" x3="248.92" y3="89.2175" layer="21" dtype="vertical"/>
 <dimension x1="254" y1="24.765" x2="259.08" y2="31.75" x3="269.875" y3="28.2575" layer="21" dtype="vertical"/>
+<wire x1="173.6725" y1="55.88" x2="173.6725" y2="83.82" width="0.3048" layer="47"/>
+<wire x1="173.6725" y1="83.82" x2="156.21" y2="83.82" width="0.3048" layer="47"/>
+<wire x1="156.21" y1="83.82" x2="156.21" y2="55.88" width="0.3048" layer="47"/>
+<wire x1="156.21" y1="55.88" x2="173.6725" y2="55.88" width="0.3048" layer="47"/>
 </plain>
 <attributes>
@@
 <element name="2R5" library="resistor" package="R0805" value="180R" x="253.0475" y="20.0025" rot="R90"/>
 <element name="2R6" library="resistor" package="R0805" value="1R" x="248.6025" y="15.24"/>
-<element name="C4" library="resistor" package="E2,5-6" value="50u" x="262.5725" y="17.78" rot="R90"/>
+<element name="C4" library="resistor" package="E2,5-6" value="50u" x="261.3025" y="14.605" rot="R90"/>
 <element name="2R7" library="resistor" package="R0805" value="3.9k" x="244.7925" y="20.32" rot="R270"/>
 <element name="2R8" library="resistor" package="R0805" value="18k" x="242.2525" y="20.955" rot="R90"/>
@@
 <element name="C5" library="resistor" package="C0805K" value="100n" x="243.84" y="24.765"/>
 <element name="C6" library="resistor" package="C0805K" value="100n" x="257.4925" y="18.7325" rot="R90"/>
-<element name="2L3" library="rcl" package="6000-XXXX-RC" value="220uH" x="234.95" y="30.1625" rot="R180"/>
+<element name="2L3" library="ct-pack" package="LV7X10MM" value="220uH" x="234.95" y="30.1625" rot="R180"/>
 <element name="1C5" library="resistor" package="E2-5" value="1000u/6V" x="239.0775" y="15.5575" rot="R90"/>
 <element name="C7" library="resistor" package="C0805K" value="100n" x="231.775" y="20.955" rot="R270"/>
@@
 <element name="C13" library="rcl" package="C0805" value="100n" x="130.4925" y="102.5525" rot="MR90"/>
 <element name="GND" library="TP4056_18650" package="PAD-" value="B-" x="136.8425" y="104.4575" rot="MR90"/>
-<element name="DA4" library="v-reg" package="SOT89R" value="78L05" x="217.4875" y="22.86" rot="R180"/>
+<element name="DA4" library="ct-pack" package="SOT89R" value="78L05" x="217.4875" y="22.86" rot="R180"/>
 <element name="3C11" library="resistor" package="E2,5-6" value="47u" x="218.7575" y="26.67" rot="R180"/>
 <element name="C8" library="resistor" package="C0805K" value="100n" x="215.5825" y="28.575"/>
-<element name="DA4A" library="v-reg" package="SOT89R" value="MCP1702" x="212.09" y="24.765" rot="R90"/>
+<element name="DA4A" library="ct-pack" package="SOT89R" value="MCP1702" x="212.09" y="24.765" rot="R90"/>
 <element name="J_NO_LI" library="jumper" package="SJ" value="" x="211.7725" y="28.575"/>
 <element name="DD1" library="avr-6" package="TQFP32-08" value="MEGA328P-AU" x="100.0125" y="90.4875" rot="MR350"/>
@@
 <element name="1L2" library="rcl" package="IRF24" value="10mkhn" x="100.0125" y="88.265" rot="R20"/>
 <element name="1C13" library="resistor" package="C0805K" value="100n" x="93.0275" y="86.995" rot="MR0"/>
-<element name="4Y3" library="relay_ussr" package="РЭС55А" value="РЭС55А" x="413.385" y="126.6825"/>
-<element name="4Y4" library="relay_ussr" package="РЭС55А" value="РЭС55А" x="447.9925" y="126.6825"/>
+<element name="4Y3" library="relay_ussr" package="РЭС55А" value="РЭС55А" x="166.0525" y="70.1675"/>
+<element name="4Y4" library="relay_ussr" package="РЭС55А" value="РЭС55А" x="166.0525" y="60.0075"/>
 <element name="4R6" library="resistor" package="R0805" value="100" x="447.9925" y="94.615"/>
 <element name="4R7" library="resistor" package="R0805" value="100" x="463.2325" y="95.885"/>
@@
 <element name="TEST1" library="transistor_tester" package="TT-P" value="TT-P" x="99.695" y="70.8025"/>
 <element name="ISP" library="con-lstb" package="MA03-2" value="" x="111.76" y="77.7875" rot="R270"/>
-<element name="DA6" library="v-reg" package="SOT89R" value="78L05" x="280.3525" y="17.78"/>
+<element name="DA6" library="ct-pack" package="SOT89R" value="78L05" x="280.3525" y="17.78"/>
 <element name="3C12" library="resistor" package="E2,5-6" value="47u" x="280.67" y="10.16"/>
 <element name="C18" library="resistor" package="C0805K" value="100n" x="279.4" y="4.445"/>
@@
 <element name="X2" library="SmartPrj" package="CON2_USB_MICRO_B_AT" value="USB MICRO" x="226.06" y="128.27" rot="R180"/>
 <element name="VT3" library="FS8205A" package="TSSOP-8" value="FS8205A" x="226.06" y="118.11" rot="R270"/>
-<element name="TEST2" library="transistor_tester" package="TT-P" value="TT-P" x="187.96" y="70.8025"/>
+<element name="TEST2" library="transistor_tester" package="TT-P" value="TT-P" x="191.4525" y="69.215"/>
 <element name="6R3" library="resistor" package="R0805" value="20K" x="228.6" y="98.1075" rot="MR0"/>
 <element name="6R10" library="resistor" package="R0805" value="10.0k" x="216.535" y="60.6425" rot="MR180"/>
@@
 <wire x1="246.6975" y1="21.59" x2="244.7925" y2="21.17" width="0" layer="19" extent="1-1"/>
 <wire x1="257.4925" y1="19.7325" x2="249.5075" y2="21.32" width="0" layer="19" extent="1-1"/>
-<wire x1="262.5725" y1="19.05" x2="257.4925" y2="19.7325" width="0" layer="19" extent="1-1"/>
+<wire x1="261.3025" y1="15.875" x2="257.4925" y2="19.7325" width="0" layer="19" extent="1-1"/>
 <wire x1="217.4875" y1="21.96" x2="231.775" y2="19.955" width="0" layer="19" extent="1-1"/>
-<wire x1="280.3525" y1="18.68" x2="262.5725" y2="19.05" width="0" layer="19" extent="1-1"/>
+<wire x1="280.3525" y1="18.68" x2="261.3025" y2="15.875" width="0" layer="19" extent="1-1"/>
 <wire x1="280.3525" y1="16.38" x2="280.3525" y2="18.68" width="0" layer="19" extent="1-1"/>
 <wire x1="281.94" y1="10.16" x2="280.3525" y2="16.38" width="0" layer="19" extent="1-1"/>
@@
 <wire x1="247.9675" y1="18.99" x2="247.9675" y2="17.145" width="0.4064" layer="1"/>
 <wire x1="247.9675" y1="17.145" x2="247.7525" y2="15.24" width="0.4064" layer="1"/>
-<wire x1="262.5725" y1="16.51" x2="256.8575" y2="12.065" width="0.4064" layer="1"/>
+<wire x1="261.3025" y1="13.335" x2="256.8575" y2="12.065" width="0.4064" layer="1"/>
 <wire x1="256.8575" y1="12.065" x2="247.9675" y2="11.7475" width="0.4064" layer="1"/>
 <wire x1="247.9675" y1="11.7475" x2="247.7525" y2="15.24" width="0.4064" layer="1"/>
-<wire x1="257.4925" y1="17.7325" x2="262.5725" y2="16.51" width="0.4064" layer="1"/>
+<wire x1="257.4925" y1="17.7325" x2="261.3025" y2="13.335" width="0.4064" layer="1"/>
 <contactref element="1R10" pad="1"/>
 <contactref element="6C1" pad="+"/>
@@
 <wire x1="243.1415" y1="27.305" x2="242.84" y2="24.765" width="0.4064" layer="1"/>
 <wire x1="242.84" y1="24.765" x2="242.2525" y2="21.805" width="0.4064" layer="1"/>
-<wire x1="242.84" y1="24.765" x2="237.45" y2="30.1625" width="0.4064" layer="1"/>
+<wire x1="242.84" y1="24.765" x2="236.7" y2="30.1625" width="0.4064" layer="1"/>
 </signal>
 <signal name="+90.5V">
@@
 <contactref element="J_NO_LI" pad="1"/>
 <contactref element="DA6" pad="1"/>
-<wire x1="232.45" y1="30.1625" x2="231.775" y2="21.955" width="0" layer="19" extent="1-1"/>
+<wire x1="233.2" y1="30.1625" x2="231.775" y2="21.955" width="0" layer="19" extent="1-1"/>
 <wire x1="239.0775" y1="14.5415" x2="231.775" y2="21.955" width="0" layer="19" extent="1-1"/>
 <wire x1="215.9875" y1="24.61" x2="231.775" y2="21.955" width="0" layer="19" extent="1-1"/>
@@
 <wire x1="97.155" y1="75.8825" x2="99.695" y2="75.8825" width="0" layer="19" extent="1-1"/>
 <wire x1="101.9175" y1="61.9125" x2="102.235" y2="75.8825" width="0" layer="19" extent="1-1"/>
-<wire x1="435.9275" y1="124.7775" x2="102.235" y2="75.8825" width="0" layer="19" extent="1-1"/>
+<wire x1="153.9875" y1="58.1025" x2="102.235" y2="75.8825" width="0" layer="19" extent="1-1"/>
 </signal>
 <signal name="T3">
@@
 <wire x1="90.4875" y1="89.2175" x2="90.805" y2="93.345" width="0.3048" layer="1"/>
 <wire x1="94.615" y1="62.23" x2="94.615" y2="75.8825" width="0" layer="19" extent="1-1"/>
-<wire x1="401.32" y1="124.7775" x2="96.5096375" y2="94.22866875" width="0" layer="19" extent="16-16"/>
+<wire x1="153.9875" y1="68.2625" x2="96.5096375" y2="94.22866875" width="0" layer="19" extent="16-16"/>
 </signal>
 <signal name="AVCC">
@@
 <contactref element="4R6" pad="2"/>
 <contactref element="4Y3" pad="P"/>
-<wire x1="401.32" y1="129.8575" x2="448.8425" y2="94.615" width="0" layer="19" extent="1-1"/>
+<wire x1="153.9875" y1="73.3425" x2="448.8425" y2="94.615" width="0" layer="19" extent="1-1"/>
 </signal>
 <signal name="N$72">
 <contactref element="4Y4" pad="P"/>
 <contactref element="4R7" pad="2"/>
-<wire x1="464.0825" y1="95.885" x2="435.9275" y2="129.8575" width="0" layer="19" extent="1-1"/>
+<wire x1="464.0825" y1="95.885" x2="153.9875" y2="63.1825" width="0" layer="19" extent="1-1"/>
 </signal>
 <signal name="PD1">
