File: HW/EAGLE/b333.sch (EAGLE design)
At the start: 87 parts, among them Q5 NMOSD

Commit message: .
Parts:
- added 1C2: 220u/6V, resistor:CPOL-EUE3.5-8
- added 2C1: 0.47n, resistor:C-EUC0805K
- added 2D2: SS12, diode:SCHOTTKY-DIODESMD
- added 2L2: 220uH, rcl:L-US6000-XXX-RC
- added 2R5: 180R, resistor:R-EU_R0805
- added 2R6: 1R, resistor:R-EU_R0805
- added 2R7: 18K, resistor:R-EU_R0805
- added 2R8: 56K, resistor:R-EU_R0805
- added C4: 50u, resistor:CPOL-EUE2.5-6
- added C5, C6: 100n, resistor:C-EUC0805K
- added D7: MC34063AD, mc34063-2:MC34063AD
Connections:
- new net N$13: 2D2.A, 2L2.2, D7.SWC
- new net N$14: 2L2.1, 2R5.1, 2R6.2, D7.IS
- new net N$15: 2R5.2, D7.DC
- new net N$16: 2R7.2, 2R8.1, D7.FB
- new net N$8: 2C1.1, D7.TC
- net +5V: now also 1C2.+, 2D2.C, 2R8.2, C5.1
- net GND: now also 1C2.-, 2C1.2, 2R7.1, C4.-, C5.2, C6.2, D7.GND, D7.SWE
- net V+: now also 2R6.1, C4.+, C6.1, D7.VCC

Commit message: .
Parts:
- added 1C5: 220u/6V, resistor:CPOL-EUE2-5
- added 2L3: 220uH, rcl:L-US6000-XXX-RC
- added C7: 100n, resistor:C-EUC0805K
- 1C2: device resistor:CPOL-EUE3.5-8 -> resistor:CPOL-EUE2-5
Connections:
- new net N$17: 1C2.+, 2D2.C, 2L3.1, 2R8.2, C5.1
- net +5V: now also 1C5.+, 2L3.2, C7.1; no longer 1C2.+, 2D2.C, 2R8.2, C5.1
- net GND: now also 1C5.-, C7.2
Other:
- moved on the sheet: 1C2, C5

Commit message: .
Parts:
- removed D7: MC34063AD, mc34063-2:MC34063AD
- added 1Q1: NMOSD, DSS:NMOSD
- added 2L4: 220uH, rcl:L-US6000-XXX-RC
- added 3C10, 3C7, C8: 100n, resistor:C-EUC0805K
- added 3C11: 47u, resistor:CPOL-EUE2.5-6
- added 3C5: 1n, resistor:C-EUC0805K
- added 3C6, 3C9: 47u/50V, resistor:CPOL-EUE2.5-6
- added 3C8: 100u, resistor:CPOL-EUE2.5-6
- added 3D2: 1N5819, diode:SCHOTTKY-DIODESMD
- added 3L2: 180uH, rcl:L-US6000-XXX-RC
- added 3R1B1, 3R8: 1R, resistor:R-EU_R0805
- added 3R5: 62K, resistor:R-EU_R0805
- added 3R6: 2K, resistor:R-EU_R0805
- added 3R7: 180R, resistor:R-EU_R0805
- added 5MA: 10MA, jumper:JP2N
- added B+OUT+, B-1, GND: B-, TP4056_18650:B-
- added C11, C12, C13: 100n, rcl:C-EUC0805
- added D10, D11, D9: LL4148, diode:DIODE-SOD80C
- added DA1: TP4056, TP4056:TP4056
- added DA2: DW01A, DW01:DW01
- added DA3, DA5: MC34063AD, mc34063-2:MC34063AD
- added DA4: 78L05, v-reg:78LXX
- added DA4A: MCP1702, v-reg:MCP1702
- added GREEN, RED: (no value), led:LEDCHIP-LED0805
- added Q1: BF423, transistor-pnp:BF423
- added R10, R24: 1k2, resistor:R-EU_R0805
- added R11: 300, resistor:R-EU_R0805
- added R12: 150, resistor:R-EU_R0805
- added R13: 39k, resistor:R-EU_R0805
- added R19: 0.5, resistor:R-EU_R0805
- added R20, R22, R23: 1k, resistor:R-EU_R0805
- added R21: 100, resistor:R-EU_R0805
- added R8: 10k, resistor:R-EU_R0805
- added R9: 100k, resistor:R-EU_R0805
- added VT2: FS8205A, FS8205A:DMN3024LSD
- added X2: USB MICRO, SmartPrj:MYCON2_USB-MINI-B
- added ZEN_A1, ZEN_K1: (no value), pinhead:PINHD-1X1
Connections:
- new net +3V7: B+OUT+.B-, C13.1, DA1.BAT, R21.2
- new net +7V: 1C5.+, 2L3.2, C7.1, DA4.IN, DA4A.IN
- new net 1MA: 5MA.2, Q1.E, R10.2
- new net B-: B-1.B-, C11.1, DA2.GND, VT2A.S
- new net N$18: Q1.C, ZEN_K1.1
- new net N$23: 3C5.1, DA5.TC
- new net N$26: 3D2.A, 3L2.2, DA5.SWC
- new net N$51: 3R5.1, 3R6.1, DA5.FB
- new net N$52: 2L4.1, 3C6.+, 3C7.1, 3D2.C, 3R5.2
- new net N$53: 3R7.2, DA5.DC
- new net N$54: 3L2.1, 3R1B1.2, 3R7.1, 3R8.2, DA5.IS
- new net N$55: 5MA.3, R11.2
- new net N$56: 1Q1.G, R8.2, R9.1
- new net N$57: 2L4.2, 3C10.1, 3C9.+, D9.A, R10.1, R11.1, R12.1
- new net N$58: 1Q1.D, DA5.GND, DA5.SWE
- new net N$59: 5MA.1, R12.2
- new net N$65: D10.A, D9.C
- new net N$66: D10.C, D11.A
- new net N$67: D11.C, Q1.B, R13.2
- new net N$75: VT2A.D, VT2B.D
- new net N$76: DA2.0C, VT2B.G
- new net N$77: DA2.0D, VT2A.G
- new net N$78: DA2.CS, R20.2
- new net N$79: C11.2, DA2.VCC, R21.1
- new net N$80: DA1.CHRG, RED.C
- new net N$81: DA1.STDBY, GREEN.C
- new net N$82: R22.1, RED.A
- new net N$83: GREEN.A, R23.1
- new net N$84: C12.1, DA1.CE, DA1.VCC, R19.2, R22.2, R23.2
- new net N$85: R19.1, X2.VBUS
- new net N$86: DA1.PROG, R24.2
- new net UGND: C12.2, C13.2, DA1.GND, DA1.TEMP, R20.1, R24.1, VT2B.S, X2.GND, X2.SH1, X2.SH2, X2.SH3, X2.SH4, X2.SH5, X2.SH6
- new net ZENER_EN: R8.1
- net +5V: now also 3C11.+, C8.1, DA4.OUT, DA4A.OUT; no longer 1C5.+, 2L3.2, C7.1
- net GND: now also 1Q1.S, 3C10.2, 3C11.-, 3C5.2, 3C6.-, 3C7.2, 3C8.-, 3C9.-, 3R6.2, C8.2, DA3.GND, DA3.SWE, DA4.GND, DA4A.GND, GND.B-, R13.1, R9.2, ZEN_A1.1; no longer D7.GND, D7.SWE
- net N$13: now also DA3.SWC; no longer D7.SWC
- net N$14: now also DA3.IS; no longer D7.IS
- net N$15: now also DA3.DC; no longer D7.DC
- net N$16: now also DA3.FB; no longer D7.FB
- net N$8: now also DA3.TC; no longer D7.TC
- net V+: now also 3C8.+, 3R1B1.1, 3R8.1, DA3.VCC, DA5.VCC; no longer D7.VCC
Other:
- note added: "B+"
- note added: "B-"
- note added: "OUT+"
- note added: "OUT-"
- moved on the sheet: 1C2, 1C5, 1R15, 2C1, 2D2, 2L2, 2L3, 2R5, 2R6, 2R7, 2R8, C2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

Commit message: .
Parts:
- added 1C13, C10, C9: 100n, resistor:C-EUC0805
- added 1C6: 1n, resistor:C-EUC0805K
- added 1C7, 3C13, C17, C18: 100n, resistor:C-EUC0805K
- added 1C8, 1C9: 22p, resistor:C-EUC0805K
- added 1L2: 10mkhn, rcl:L-USIRF-24
- added 1R10, 1R9: 10K, resistor:R-EU_R0805
- added 1R17: 3K3, resistor:R-EU_R1206W
- added 1R18: 27K, resistor:R-EU_R0805
- added 1R19, 1R21, 1R23: 680, resistor:R-EU_0207/10
- added 1R20, 1R22, 1R24: 470K, resistor:R-EU_0207/10
- added 1R25: 2K2, resistor:R-EU_R0805
- added 1R26: 270, resistor:R-EU_R1206W
- added 1RC2: 22K, resistor:R-EU_R0805
- added 1RC2*1: 4K3, resistor:R-EU_R1206W
- added 1Z2: 8MHz, crystal:CRYSTALHC49U70
- added 3C12: 47u, resistor:CPOL-EUE2.5-6
- added 4R6, 4R7: 100, resistor:R-EU_R0805
- added 4Y3, 4Y4: РЭС55А, relay_ussr:РЭС55А
- added D7: MEGA328P-AU, avr-6:MEGA48/88/168-AU
- added D8: TL431, v-reg:TL431CLP
- added DA6: 78L05, v-reg:78LXX
- added H2: LCD, pinhead:PINHD-1X16
- added ISP: (no value), con-lstb:MA03-2
- added J_NO_LI, J_ONE5V: (no value), jumper:SJ
- added R14: 180K, resistor:R-EU_R0805
- added R15: 20.0k, resistor:R-EU_R0805
- added R16: 180.0k, resistor:R-EU_R0805
- added R4: 20K, resistor:R-EU_R0805
- added T4, T5, T6: (no value), pinhead:PINHD-1X1
- added TEST1: TT-P, transistor_tester:TT-P
- R24: device resistor:R-EU_R0805 -> resistor:R-EU_0204/7
- renumbered X2 to X1
Connections:
- net N$57 renamed +40V
- new net +5V/2: 1R26.2, 1RC2.1, 3C12.+, C18.1, DA6.OUT, H2.2, J_ONE5V.2
- new net E1: D7.PD5(T1/OC0B/PCINT21), H2.6
- new net N$60: 1RC2*1.2, 1RC2.2, H2.3
- new net N$61: 1R26.1, H2.15
- new net N$62: D7.PD3(INT1/OC2B/PCINT19), H2.14
- new net N$63: R14.2
- new net N$64: 1C6.1, D7.AREF
- new net N$68: 1C8.2, 1Z2.2, D7.PB6(XTAL1/TOSC1/PCINT6)
- new net N$69: 1C9.2, 1Z2.1, D7.PB7(XTAL2/TOSC2/PCINT7)
- new net N$70: 1C13.1, 1L2.1, D7.AVCC
- new net N$71: 4R6.2, 4Y3G$2.P
- new net N$72: 4R7.2, 4Y4G$2.P
- new net N$87: D7.PD0(RXD/PCINT16), H2.11
- new net N$88: D7.PD1(TXD/PCINT17), H2.12
- new net N$89: D7.PD2(INT0/PCINT18), H2.13
- new net PB3: 1R19.1, D7.PB0(ICP1/CLKO/PCINT0)
- new net PB4: 1R20.1, D7.PB1(OC1A/PCINT1)
- new net PB5: 1R21.1, D7.PB2(SS/OC1B/PCINT2)
- new net PC10: 1R21.2, 1R22.2, 4Y4G$2.O, D7.PC1(ADC1/PCINT9), T5.1, TEST1.2
- new net PC11: 1R23.2, 1R24.2, 4Y3G$2.O, D7.PC2(ADC2/PCINT10), T6.1, TEST1.3
- new net PC6: 1R10.2, 1R17.2, D7.PC5(ADC5/SCL/PCINT13)
- new net PC7: 1R25.2, D7.PC4(ADC4/SDA/PCINT12), D8.C, D8.R
- new net PC8: C9.1, D7.PC3(ADC3/PCINT11), R14.1, R4.2
- new net PC9: 1R19.2, 1R20.2, 4R6.1, 4R7.1, D7.PC0(ADC0/PCINT8), T4.1, TEST1.1
- new net PD1: 1R18.2, C17.1, D7.PD7(AIN1/PCINT23)
- new net PD2: D7.PD6(AIN0/OC0A/PCINT22)
- new net RS1: D7.PD4(T0/XCK/PCINT20), H2.4
- new net V+1: 1R10.1, 1R9.2
- net +5V: now also 1C7.1, 1L2.2, 1R18.1, 1R25.1, C10.1, D7.VCC@1, D7.VCC@2, ISP.2, J_NO_LI.2, J_ONE5V.1
- net +7V: now also DA6.IN, J_NO_LI.1
- net GND: now also 1C13.2, 1C6.2, 1C7.2, 1C8.1, 1C9.1, 1R17.1, 1RC2*1.1, 3C12.-, 3C13.2, C10.2, C17.2, C18.2, C9.2, D7.AGND, D7.GND@1, D7.GND@2, D8.A, DA6.GND, H2.1, H2.10, H2.16, H2.5, H2.7, H2.8, H2.9, ISP.6, R15.1, R4.1
- net MISO: now also 1R23.1, D7.PB4(MISO/PCINT4), ISP.1
- net MOSI: now also 1R22.1, D7.PB3(MOSI/OC2A/PCINT3), ISP.4
- net N$18: now also R16.2
- net PC3: now also 3C13.1, R15.2, R16.1
- net RESET: now also 1R9.1, D7.PC6(/RESET/PCINT14), ISP.5
- net SCK: now also 1R24.1, D7.PB5(SCK/PCINT5), ISP.3
- net UGND: now also DA1..

Commit message: .
Parts:
- removed 1Q1: NMOSD, DSS:NMOSD
- removed Q1: BF423, transistor-pnp:BF423
- removed R9: 100k, resistor:R-EU_R0805
- added R18, R25: 10k, resistor:R-EU_R0805
- added VT4: МП15, transistor-pnp:BF423
- added VT5: NMOSD, DSS:NMOSD
- added VT6: BF423, transistor-pnp:BF423
- R8: value 10k -> 100k
Connections:
- removed net ZENER_EN: R8.1
- new net !BUTTON: R18.1
- new net N$73: R25.2, R8.1, VT4.C
- new net N$74: R18.2, VT4.B
- net +5V/2: now also VT4.E
- net 1MA: now also VT6.E; no longer Q1.E
- net GND: now also R25.1, VT5.S; no longer 1Q1.S, 3R6.2, R9.2
- net N$18: now also VT6.C; no longer Q1.C
- net N$56: now also VT5.G; no longer 1Q1.G, R9.1
- net N$58: now also 3R6.2, VT5.D; no longer 1Q1.D
- net N$67: now also VT6.B; no longer Q1.B
Other:
- moved on the sheet: 2L4, 3C10, 3C13, 3C5, 3C6, 3C7, 3C8, 3C9, 3D2, 3L2, 3R1B1, 3R5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

Commit message: 34063 links
Parts:
- removed 1C10: 220u/6V, resistor:CPOL-EUE3.5-8
- removed 2C2: 0.47n, resistor:C-EUC0805K
- removed 2D1: SS12, diode:DIODE-DO41-10
- removed 2L1: 220uH, inductor-neosid:SD12-1000
- removed 2R1: 1R, resistor:R-EU_R0805
- removed 2R2: 180R, resistor:R-EU_R0805
- removed 2R3: 18K, resistor:R-EU_R0805
- removed 2R4: 56K, resistor:R-EU_R0805
- removed C14, C15: 100n, resistor:C-EUC0805K
- removed C16: 50u, resistor:CPOL-EUE2.5-6
- removed C9: 100n, resistor:C-EUC0805
- removed D3: MC34063AD, mc34063:MC34063AD
- removed R14: 180K, resistor:R-EU_R0805
- removed R4: 20K, resistor:R-EU_R0805
- added T7: (no value), transistor:-NPN-TO92-ECB
Connections:
- net PC6 renamed U_BAT
- net PC7 renamed +2V5
- removed net N$22: 2R2.2, D3.DC
- removed net N$24: 2L1.1, 2R1.2, 2R2.1, D3.IS
- removed net N$25: 2R3.2, 2R4.1, D3.FB
- removed net N$56: R8.2, VT5.G
- removed net N$63: R14.2
- removed net N$73: R25.2, R8.1, VT4.C
- removed net N$74: R18.2, VT4.B
- removed net PC8: C9.1, D7.PC3(ADC3/PCINT11), R14.1, R4.2
- removed net V+1: 1R10.1, 1R9.2
- net +5V: now also 1R9.2; no longer 1C10.+, 2D1.C, 2R4.2, C14.1
- net +5V/2: now also R25.2; no longer VT4.E
- net GND: now also R8.1, T7.E; no longer 1C10.-, 2C2.2, 2R3.1, C14.2, C15.2, C16.-, C9.2, D3.GND, D3.SWE, R25.1, R4.1
- net N$19: now also R18.2, T7.B; no longer 2C2.1, D3.TC
- net N$21: now also R25.1, R8.2, T7.C, VT5.G; no longer 2D1.A, 2L1.2, D3.SWC
- net PC3: now also D7.PC3(ADC3/PCINT11)
- net V+: now also 1R10.1; no longer 2R1.1, C15.1, C16.+, D3.VCC
Other:
- note added: "Напр. Батареи"
- note added: "Опорное 2.5в"
- note added: "Стабилитрон"
- moved on the sheet: 1L2, 1R10, 1R17, 1R25, C10, D8, ISP, R18, R25, R8, VT4

Commit message: add lnk
Parts:
- 1C5: value 220u/6V -> 1000u/6V
- 1R19, 1R20, 1R21, 1R22, 1R23, 1R24: device resistor:R-EU_0207/10 -> resistor:R-EU_M0805
- renumbered D7 to DD1
Connections:
- net PC10 renamed T2
- removed net PC11: 1R23.2, 1R24.2, 4Y3G$2.O, DD1.PC2(ADC2/PCINT10), T6.1, TEST1.3
- removed net PC9: 1R19.2, 1R20.2, 4R6.1, 4R7.1, DD1.PC0(ADC0/PCINT8), T4.1, TEST1.1
- new net T1: 1R19.2, 1R20.2, 4R6.1, 4R7.1, DD1.PC0(ADC0/PCINT8), T4.1, TEST1.3
- new net T3: 1R23.2, 1R24.2, 4Y3G$2.O, DD1.PC2(ADC2/PCINT10), T6.1, TEST1.1

Commit message: .
Parts:
- added 3R1B2: 2R, resistor:R-EU_R0805
- 1C13: device resistor:C-EUC0805 -> resistor:C-EUC0805K
- 3C6: value 47u/50V -> 22u/100V
- 3D2: value 1N5819 -> RK19(1N5819)
- 3L2: value 180uH -> 230uH
- 3R1B1: value 1R -> 2R
Connections:
- net N$54: now also 3R1B2.2
- net V+: now also 3R1B2.1
Other:
- moved on the sheet: 3R1B1
Changed lines of the file:
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@@
 <part name="ZEN_A1" library="pinhead" deviceset="PINHD-1X1" device=""/>
 <part name="DA5" library="mc34063-2" deviceset="MC34063" device="AD"/>
-<part name="3L2" library="rcl" deviceset="L-US" device="6000-XXX-RC" value="180uH"/>
-<part name="3D2" library="diode" deviceset="SCHOTTKY-DIODE" device="SMD" value="1N5819"/>
+<part name="3L2" library="rcl" deviceset="L-US" device="6000-XXX-RC" value="230uH"/>
+<part name="3D2" library="diode" deviceset="SCHOTTKY-DIODE" device="SMD" value="RK19(1N5819)"/>
 <part name="3C5" library="resistor" deviceset="C-EU" device="C0805K" value="1n"/>
-<part name="3C6" library="resistor" deviceset="CPOL-EU" device="E2.5-6" value="47u/50V"/>
+<part name="3C6" library="resistor" deviceset="CPOL-EU" device="E2.5-6" value="22u/100V"/>
 <part name="3C7" library="resistor" deviceset="C-EU" device="C0805K" value="100n"/>
 <part name="U$31" library="lib-user" deviceset="GND" device=""/>
@@
 <part name="U$34" library="lib-user" deviceset="GND" device=""/>
 <part name="R8" library="resistor" deviceset="R-EU_" device="R0805" value="100k"/>
-<part name="3R1B1" library="resistor" deviceset="R-EU_" device="R0805" value="1R"/>
+<part name="3R1B1" library="resistor" deviceset="R-EU_" device="R0805" value="2R"/>
 <part name="SUPPLY6" library="supply2" deviceset="V+" device=""/>
 <part name="2L4" library="rcl" deviceset="L-US" device="6000-XXX-RC" value="220uH"/>
@@
 <part name="1R25" library="resistor" deviceset="R-EU_" device="R0805" value="2K2"/>
 <part name="1L2" library="rcl" deviceset="L-US" device="IRF-24" value="10mkhn"/>
-<part name="1C13" library="resistor" deviceset="C-EU" device="C0805" value="100n"/>
+<part name="1C13" library="resistor" deviceset="C-EU" device="C0805K" value="100n"/>
 <part name="U$54" library="lib-user" deviceset="GND" device=""/>
 <part name="4Y3" library="relay_ussr" deviceset="РЭС55" device="А" value="РЭС55А"/>
@@
 <part name="T7" library="transistor" deviceset="*-NPN-" device="TO92-ECB"/>
 <part name="U$12" library="lib-user" deviceset="GND" device=""/>
+<part name="3R1B2" library="resistor" deviceset="R-EU_" device="R0805" value="2R"/>
 </parts>
 <sheets>
@@
 <attribute name="VALUE" x="119.38" y="53.34" size="1.778" layer="96"/>
 </instance>
-<instance part="3L2" gate="G$1" x="127" y="83.82" rot="R90"/>
+<instance part="3L2" gate="G$1" x="127" y="83.82" smashed="yes" rot="R90">
+<attribute name="NAME" x="124.46" y="87.63" size="1.778" layer="95" rot="R180"/>
+<attribute name="VALUE" x="134.62" y="87.63" size="1.778" layer="96" rot="R180"/>
+</instance>
 <instance part="3D2" gate="G$1" x="149.86" y="73.66" smashed="yes">
 <attribute name="NAME" x="149.86" y="79.2226" size="1.778" layer="95"/>
@@
 <instance part="U$34" gate="G$1" x="144.78" y="25.4"/>
 <instance part="R8" gate="G$1" x="129.54" y="25.4" rot="R90"/>
-<instance part="3R1B1" gate="G$1" x="91.44" y="73.66" smashed="yes" rot="R90">
-<attribute name="NAME" x="89.9414" y="67.31" size="1.778" layer="95" rot="R90"/>
-<attribute name="VALUE" x="88.138" y="80.01" size="1.778" layer="96" rot="R270"/>
+<instance part="3R1B1" gate="G$1" x="93.98" y="73.66" smashed="yes" rot="R90">
+<attribute name="NAME" x="92.4814" y="67.31" size="1.778" layer="95" rot="R90"/>
+<attribute name="VALUE" x="90.678" y="80.01" size="1.778" layer="96" rot="R270"/>
 </instance>
 <instance part="SUPPLY6" gate="1" x="81.28" y="63.5" smashed="yes" rot="R90">
@@
 </instance>
 <instance part="U$12" gate="G$1" x="106.68" y="15.24"/>
+<instance part="3R1B2" gate="G$1" x="88.9" y="73.66" smashed="yes" rot="R90">
+<attribute name="NAME" x="87.4014" y="67.31" size="1.778" layer="95" rot="R90"/>
+<attribute name="VALUE" x="85.598" y="80.01" size="1.778" layer="96" rot="R270"/>
+</instance>
 </instances>
 <busses>
@@
 <wire x1="111.76" y1="63.5" x2="99.06" y2="63.5" width="0.1524" layer="91"/>
 <pinref part="SUPPLY6" gate="1" pin="V+"/>
-<wire x1="99.06" y1="63.5" x2="88.9" y2="63.5" width="0.1524" layer="91"/>
+<wire x1="99.06" y1="63.5" x2="93.98" y2="63.5" width="0.1524" layer="91"/>
 <wire x1="99.06" y1="68.58" x2="99.06" y2="63.5" width="0.1524" layer="91"/>
 <junction x="99.06" y="63.5"/>
-<wire x1="91.44" y1="68.58" x2="91.44" y2="63.5" width="0.1524" layer="91"/>
-<wire x1="91.44" y1="63.5" x2="88.9" y2="63.5" width="0.1524" layer="91"/>
+<wire x1="93.98" y1="68.58" x2="93.98" y2="63.5" width="0.1524" layer="91"/>
+<wire x1="93.98" y1="63.5" x2="88.9" y2="63.5" width="0.1524" layer="91"/>
 <wire x1="88.9" y1="63.5" x2="83.82" y2="63.5" width="0.1524" layer="91"/>
-<junction x="91.44" y="63.5"/>
+<junction x="93.98" y="63.5"/>
+<pinref part="3R1B2" gate="G$1" pin="1"/>
+<wire x1="88.9" y1="68.58" x2="88.9" y2="63.5" width="0.1524" layer="91"/>
 </segment>
 </net>
@@
 <wire x1="104.14" y1="83.82" x2="99.06" y2="83.82" width="0.1524" layer="91"/>
 <wire x1="99.06" y1="83.82" x2="99.06" y2="78.74" width="0.1524" layer="91"/>
-<wire x1="91.44" y1="78.74" x2="91.44" y2="83.82" width="0.1524" layer="91"/>
-<wire x1="91.44" y1="83.82" x2="99.06" y2="83.82" width="0.1524" layer="91"/>
+<wire x1="93.98" y1="78.74" x2="93.98" y2="83.82" width="0.1524" layer="91"/>
+<wire x1="93.98" y1="83.82" x2="99.06" y2="83.82" width="0.1524" layer="91"/>
 <junction x="99.06" y="83.82"/>
 <junction x="109.22" y="83.82"/>
-</segment>
-</net>
+<pinref part="3R1B2" gate="G$1" pin="2"/>
+<wire x1="88.9" y1="78.74" x2="88.9" y2="83.82" width="0.1524" layer="91"/>
+<wire x1="88.9" y1="83.82" x2="93.98" y2="83.82" width="0.1524" layer="91"/>
+<junction x="93.98" y="83.82"/>
+</segment>
+</net>
