File: HW/EAGLE/b333.sch (EAGLE design)
At the start: 188 parts, among them Q5 NMOSD, X1 USB MICRO

Commit message: .
Parts:
- removed 1C1: 1n, resistor:C-EUC0805K
- removed 1C11, 1C12: 22p, resistor:C-EUC0805K
- removed 1C3, C3: 100n, resistor:C-EUC0805
- removed 1C4: 100n, resistor:C-EUC0805K
- removed 1L1: 10mkhn, rcl:L-USIRF-24
- removed 1R1, 1R3, 1R5: 680, resistor:R-EU_0207/10
- removed 1R11, 1R13: 10K, resistor:R-EU_R0805
- removed 1R12: 3K3, resistor:R-EU_R1206W
- removed 1R16: 2K2, resistor:R-EU_R0805
- removed 1R2, 1R4: 470K, resistor:R-EU_0207/10
- removed 1Z1: 8MHz, crystal:CRYSTALHC49U70
- removed D1: MEGA328P-AU, avr-6:MEGA48/88/168-AU
- removed D2: TL431, v-reg:TL431CLP
- removed H1: LCD, pinhead:PINHD-1X16
- removed S2: ISP, con-lstb:MA03-2
- removed TEST: TT-P, transistor_tester:TT-P
- added 3C14: 1n, resistor:C-EUC0805K
- added 3C15, 3C16: 22u/100V, resistor:CPOL-EUE2.5-6
- added 3C17: 100u, resistor:CPOL-EUE2.5-6
- added 3D3, 3D4: RK19(1N5819), diode:SCHOTTKY-DIODESMD
- added 3L3, 3L4: 230uH, rcl:L-US6000-XXX-RC
- added 3R10: 2K, resistor:R-EU_R0805
- added 3R11: 180R, resistor:R-EU_R0805
- added 3R12: 1R, resistor:R-EU_R0805
- added 3R1B3, 3R1B4: 2R, resistor:R-EU_R0805
- added 3R9: 62K, resistor:R-EU_R0805
- added C14: 33, rcl:C-EUC0805K
- added C15: 2n2, rcl:C-EUC0805K
- added C16: 47m, rcl:CPOL-EUE2-4
- added C19: 1n, rcl:C-EUC0805K
- added C9: 56, rcl:C-EUC0805K
- added D12, D3, D7: 1N4148DO35-7, diode:1N4148DO35-7
- added DA7: MC34063AD, mc34063-2:MC34063AD
- added JP1, JP2: (no value), pinhead:PINHD-1X1
- added Q1, Q2: 2N4126, transistor-pnp:2N4126
- added R14: 100, rcl:R-EU_M0805
- added R17: 470, rcl:R-EU_M0805
- added R26, R28, R32, R33: 1k, rcl:R-EU_M0805
- added R27: 8k2, rcl:R-EU_M0805
- added R29, R30: 10k, resistor:R-EU_R0805
- added R31: 300, rcl:R-EU_M0805
- added R34, R9: 15k, rcl:R-EU_M0805
- added R35: (no value), rcl:R-TRIMM3296W
- added R4: 100k, resistor:R-EU_R0805
- added T8: (no value), transistor:-NPN-TO92-ECB
- added T9: (no value), transistor:-NPN-TO92-EBC
- added VT1: NMOSD, DSS:NMOSD
Connections:
- removed net E: D1.PD5(T1/OC0B/PCINT21), H1.6
- removed net N$12: 1C12.2, 1Z1.1, D1.PB7(XTAL2/TOSC2/PCINT7)
- removed net N$4: 1C1.1, D1.AREF
- removed net N$41: D1.PD0(RXD/PCINT16), H1.11
- removed net N$42: D1.PD1(TXD/PCINT17), H1.12
- removed net N$43: D1.PD3(INT1/OC2B/PCINT19), H1.14
- removed net N$44: D1.PD2(INT0/PCINT18), H1.13
- removed net N$45: 1C3.1, 1L1.1, D1.AVCC
- removed net PB0: 1R1.1, D1.PB0(ICP1/CLKO/PCINT0)
- removed net PB1: 1R2.1, D1.PB1(OC1A/PCINT1)
- removed net PB2: 1R3.1, D1.PB2(SS/OC1B/PCINT2)
- removed net PC0: 1R1.2, 1R2.2, 4R1.1, 4R2.1, D1.PC0(ADC0/PCINT8), T1.1, TEST.1
- removed net PC5: 1R11.2, 1R12.2, D1.PC5(ADC5/SCL/PCINT13)
- removed net RS: D1.PD4(T0/XCK/PCINT20), H1.4
- removed net RS1: DD1.PD4(T0/XCK/PCINT20), H2.4
- new net !BUTTON1: R29.1
- new net N$100: D3.A, D7.A, Q2.C, R31.2
- new net N$101: C14.2, C15.1, C16.-, R33.1
- new net N$102: D7.C, R32.2, T9.B
- new net N$103: C15.2, C16.+, JP1.1
- new net N$110: 4R1.1, 4R2.1
- new net N$114: 1R6.1
- new net N$115: 1R6.2
- new net N$22: 3C14.1, DA7.TC
- new net N$24: 3D3.A, 3L3.2, 3L4.1, DA7.SWC
- new net N$25: 3R10.1, 3R9.1, DA7.FB
- new net N$52: 3R11.2, DA7.DC
- new net N$56: 3L3.1, 3R11.1, 3R12.2, 3R1B3.2, 3R1B4.2, DA7.IS
- new net N$57: 3R10.2, DA7.GND, DA7.SWE, VT1.D
- new net N$63: 3C16.+, 3D4.C
- new net N$73: 3D4.A, 3L4.2
- new net N$90: Q1.E, Q2.E, R14.1
- new net N$91: C14.1, D12.A, Q1.B, R33.2, R34.2, R9.1
- new net N$93: C9.1, Q2.B, R17.1, R26.2, R27.1
- new net N$94: 3C15.+, 3D3.C, 3R9.2
- new net N$95: R29.2, T8.B
- new net N$96: R30.1, R4.2, T8.C, VT1.G
- new net N$97: C19.1, D12.C, JP2.1, R14.2, R17.2, R28.2, R9.2
- new net PD4: D3.C, DD1.PD4(T0/XCK/PCINT20), H2.4, R27.2, R28.1, T9.C
- net +5V: no longer 1C4.1, 1L1.2, 1R16.1, C3.1, D1.VCC@1, D1.VCC@2, H1.2, S2.2
- net +5V/2: now also R30.2
- net GND: now also 3C14.2, 3C15.-, 3C16.-, 3C17.-, C19.2, C9.2, Q1.C, R26.1, R31.1, R32.1, R35.A, R35.S, R4.1, T8.E, T9.E, VT1.S; no longer 1C1.2, 1C11.1, 1C12.1, 1C3.2, 1C4.2, 1R12.1, C3.2, D1.AGND, D1.GND@1, D1.GND@2, D2.A, H1.1, H1.10, H1.16, H1.5, H1.7, H1.8, H1.9, S2.6
- net MISO: no longer 1R5.1, D1.PB4(MISO/PCINT4), S2.1
- net MOSI: no longer 1R4.1, D1.PB3(MOSI/OC2A/PCINT3), S2.4
- net N$11: no longer H1.15
- net N$3: now also R34.1, R35.E; no longer 1C11.2, 1Z1.2, D1.PB6(XTAL1/TOSC1/PCINT6)
- net N$6: no longer H1.3
- net PC1: no longer 1R3.2, 1R4.2, D1.PC1(ADC1/PCINT9), T2.1, TEST.2
- net PC2: no longer 1R5.2, 1R6.2, D1.PC2(ADC2/PCINT10), T3.1, TEST.3
- net PC3: no longer D1.PC3(ADC3/PCINT11)
- net PC4: no longer 1R16.2, D1.PC4(ADC4/SDA/PCINT12), D2.C, D2.R
- net PD6: no longer D1.PD6(AIN0/OC0A/PCINT22)
- net PD7: no longer D1.PD7(AIN1/PCINT23)
- net RESET: no longer 1R13.1, D1.PC6(/RESET/PCINT14), S2.5
- net SCK: no longer 1R6.1, D1.PB5(SCK/PCINT5), S2.3
- net V+: now also 3C17.+, 3R12.1, 3R1B3.1, 3R1B4.1, DA7.VCC; no longer 1R11.1, 1R13.2

Commit message: .
Parts:
- added J_PD4: (no value), jumper:SJ
- 3R9: value 62K -> 120k
Connections:
- net N$64 renamed AREF
- net N$70 renamed AVCC
- removed net N$63: 3C16.+, 3D4.C
- new net N$12: 3C15.+, 3D3.C
- new net N$4: DD1.PD4(T0/XCK/PCINT20), J_PD4.1
- net N$94: now also 3C16.+, 3D4.C; no longer 3C15.+, 3D3.C
- net PD4: now also J_PD4.2; no longer DD1.PD4(T0/XCK/PCINT20)
Other:
- moved on the sheet: 3C16, 3D4, 3L4
Changed lines of the file:
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@@
 <part name="3D3" library="diode" deviceset="SCHOTTKY-DIODE" device="SMD" value="RK19(1N5819)"/>
 <part name="3C14" library="resistor" deviceset="C-EU" device="C0805K" value="1n"/>
-<part name="3R9" library="resistor" deviceset="R-EU_" device="R0805" value="62K"/>
+<part name="3R9" library="resistor" deviceset="R-EU_" device="R0805" value="120k"/>
 <part name="3R10" library="resistor" deviceset="R-EU_" device="R0805" value="2K"/>
 <part name="3R11" library="resistor" deviceset="R-EU_" device="R0805" value="180R"/>
@@
 <part name="R35" library="rcl" deviceset="R-TRIMM" device="3296W"/>
 <part name="GND10" library="supply1" deviceset="GND" device=""/>
+<part name="J_PD4" library="jumper" deviceset="SJ" device=""/>
 </parts>
 <sheets>
@@
 <instance part="P+12" gate="1" x="124.46" y="162.56" smashed="yes">
 <attribute name="VALUE" x="127" y="165.1" size="1.778" layer="96" rot="R180"/>
+</instance>
+<instance part="J_PD4" gate="1" x="142.24" y="91.44" smashed="yes">
+<attribute name="NAME" x="139.7" y="88.9" size="1.778" layer="95"/>
+<attribute name="VALUE" x="139.7" y="87.63" size="1.778" layer="96"/>
 </instance>
 </instances>
@@
 <segment>
 <pinref part="H2" gate="A" pin="4"/>
-<pinref part="DD1" gate="1" pin="PD4(T0/XCK/PCINT20)"/>
-<wire x1="134.62" y1="91.44" x2="172.72" y2="91.44" width="0.1524" layer="91"/>
+<wire x1="147.32" y1="91.44" x2="172.72" y2="91.44" width="0.1524" layer="91"/>
 <wire x1="172.72" y1="91.44" x2="172.72" y2="106.68" width="0.1524" layer="91"/>
 <wire x1="172.72" y1="106.68" x2="246.38" y2="106.68" width="0.1524" layer="91"/>
 <wire x1="246.38" y1="106.68" x2="246.38" y2="139.7" width="0.1524" layer="91"/>
+<pinref part="J_PD4" gate="1" pin="2"/>
+<label x="149.86" y="91.44" size="1.778" layer="95"/>
 </segment>
 </net>
@@
 </segment>
 </net>
-<net name="N$64" class="0">
+<net name="AREF" class="0">
 <segment>
 <pinref part="1C6" gate="G$1" pin="1"/>
@@
 <pinref part="DD1" gate="1" pin="AREF"/>
 <wire x1="71.12" y1="86.36" x2="73.66" y2="86.36" width="0.1524" layer="91"/>
+<label x="66.04" y="86.36" size="1.778" layer="95"/>
 </segment>
 </net>
@@
 </segment>
 </net>
-<net name="N$70" class="0">
+<net name="AVCC" class="0">
 <segment>
 <pinref part="DD1" gate="1" pin="AVCC"/>
@@
 <wire x1="60.96" y1="86.36" x2="60.96" y2="88.9" width="0.1524" layer="91"/>
 <junction x="60.96" y="88.9"/>
+<label x="63.5" y="88.9" size="1.778" layer="95"/>
 </segment>
 </net>
@@
 <wire x1="144.78" y1="162.56" x2="144.78" y2="160.02" width="0.1524" layer="91"/>
 <pinref part="P+1" gate="1" pin="V+"/>
+</segment>
+</net>
+<net name="N$4" class="0">
+<segment>
+<pinref part="J_PD4" gate="1" pin="1"/>
+<pinref part="DD1" gate="1" pin="PD4(T0/XCK/PCINT20)"/>
+<wire x1="137.16" y1="91.44" x2="134.62" y2="91.44" width="0.1524" layer="91"/>
 </segment>
 </net>
@@
 </instance>
 <instance part="U$13" gate="G$1" x="160.02" y="-55.88"/>
-<instance part="3L4" gate="G$1" x="167.64" y="-35.56" smashed="yes" rot="R90">
-<attribute name="NAME" x="165.1" y="-31.75" size="1.778" layer="95" rot="R180"/>
-<attribute name="VALUE" x="175.26" y="-31.75" size="1.778" layer="96" rot="R180"/>
-</instance>
-<instance part="3D4" gate="G$1" x="180.34" y="-35.56" smashed="yes">
-<attribute name="NAME" x="180.34" y="-29.9974" size="1.778" layer="95"/>
-<attribute name="VALUE" x="177.8" y="-32.7914" size="1.778" layer="96"/>
-</instance>
-<instance part="3C16" gate="G$1" x="187.96" y="-48.26" smashed="yes">
-<attribute name="NAME" x="186.563" y="-65.5574" size="1.778" layer="95"/>
-<attribute name="VALUE" x="184.023" y="-68.0974" size="1.778" layer="96"/>
-</instance>
-<instance part="U$14" gate="G$1" x="187.96" y="-53.34"/>
+<instance part="3L4" gate="G$1" x="152.4" y="-35.56" smashed="yes" rot="R90">
+<attribute name="NAME" x="149.86" y="-31.75" size="1.778" layer="95" rot="R180"/>
+<attribute name="VALUE" x="160.02" y="-31.75" size="1.778" layer="96" rot="R180"/>
+</instance>
+<instance part="3D4" gate="G$1" x="165.1" y="-35.56" smashed="yes">
+<attribute name="NAME" x="165.1" y="-29.9974" size="1.778" layer="95"/>
+<attribute name="VALUE" x="162.56" y="-32.7914" size="1.778" layer="96"/>
+</instance>
+<instance part="3C16" gate="G$1" x="175.26" y="-40.64" smashed="yes">
+<attribute name="NAME" x="173.863" y="-57.9374" size="1.778" layer="95"/>
+<attribute name="VALUE" x="171.323" y="-60.4774" size="1.778" layer="96"/>
+</instance>
+<instance part="U$14" gate="G$1" x="175.26" y="-48.26"/>
 </instances>
 <busses>
@@
 <pinref part="3C16" gate="G$1" pin="-"/>
 <pinref part="U$14" gate="G$1" pin="GND"/>
+<wire x1="175.26" y1="-45.72" x2="175.26" y2="-48.26" width="0.1524" layer="91"/>
 </segment>
 </net>
@@
 <wire x1="139.7" y1="-45.72" x2="142.24" y2="-45.72" width="0.1524" layer="91"/>
 <pinref part="3L4" gate="G$1" pin="1"/>
-<wire x1="160.02" y1="-35.56" x2="139.7" y2="-35.56" width="0.1524" layer="91"/>
+<wire x1="144.78" y1="-35.56" x2="139.7" y2="-35.56" width="0.1524" layer="91"/>
 <junction x="139.7" y="-35.56"/>
 </segment>
@@
 <segment>
 <pinref part="3R9" gate="G$1" pin="2"/>
-<pinref part="3D3" gate="G$1" pin="C"/>
-<wire x1="147.32" y1="-45.72" x2="152.4" y2="-45.72" width="0.1524" layer="91"/>
-<wire x1="129.54" y1="-76.2" x2="152.4" y2="-76.2" width="0.1524" layer="91"/>
-<wire x1="152.4" y1="-76.2" x2="152.4" y2="-45.72" width="0.1524" layer="91"/>
-<wire x1="152.4" y1="-45.72" x2="160.02" y2="-45.72" width="0.1524" layer="91"/>
-<pinref part="3C15" gate="G$1" pin="+"/>
-<wire x1="160.02" y1="-45.72" x2="160.02" y2="-48.26" width="0.1524" layer="91"/>
+<wire x1="129.54" y1="-76.2" x2="170.18" y2="-76.2" width="0.1524" layer="91"/>
+<pinref part="3D4" gate="G$1" pin="C"/>
+<wire x1="167.64" y1="-35.56" x2="170.18" y2="-35.56" width="0.1524" layer="91"/>
+<pinref part="3C16" gate="G$1" pin="+"/>
+<wire x1="170.18" y1="-35.56" x2="175.26" y2="-35.56" width="0.1524" layer="91"/>
+<wire x1="175.26" y1="-35.56" x2="175.26" y2="-38.1" width="0.1524" layer="91"/>
+<wire x1="170.18" y1="-76.2" x2="170.18" y2="-35.56" width="0.1524" layer="91"/>
+<junction x="170.18" y="-35.56"/>
 </segment>
 </net>
@@
 </segment>
 </net>
-<net name="N$63" class="0">
-<segment>
-<pinref part="3D4" gate="G$1" pin="C"/>
-<wire x1="182.88" y1="-35.56" x2="187.96" y2="-35.56" width="0.1524" layer="91"/>
-<pinref part="3C16" gate="G$1" pin="+"/>
-<wire x1="187.96" y1="-35.56" x2="187.96" y2="-45.72" width="0.1524" layer="91"/>
-</segment>
-</net>
 <net name="N$73" class="0">
 <segment>
 <pinref part="3D4" gate="G$1" pin="A"/>
 <pinref part="3L4" gate="G$1" pin="2"/>
-<wire x1="177.8" y1="-35.56" x2="175.26" y2="-35.56" width="0.1524" layer="91"/>
+<wire x1="162.56" y1="-35.56" x2="160.02" y2="-35.56" width="0.1524" layer="91"/>
 </segment>
 </net>
 <net name="N$74" class="0">
 <segment>
-<wire x1="116.84" y1="-30.48" x2="175.26" y2="-30.48" width="0.1524" layer="91"/>
-</segment>
-</net>
+<wire x1="116.84" y1="-30.48" x2="157.48" y2="-30.48" width="0.1524" layer="91"/>
+</segment>
+</net>
+<net name="N$12" class="0">
+<segment>
+<pinref part="3C15" gate="G$1" pin="+"/>
+<wire x1="160.02" y1="-45.72" x2="160.02" y2="-48.26" width="0.1524" layer="91"/>
+<pinref part="3D3" gate="G$1" pin="C"/>
+<wire x1="147.32" y1="-45.72" x2="160.02" y2="-45.72" width="0.1524" layer="91"/>
+</segment>
+</net>

Commit message: .
Connections:
- new net N$45: 3D3.A
- net N$24: no longer 3D3.A
Other:
- moved on the sheet: 3C14, 3D3, 3L3, 3L4
Changed lines of the file:
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@@
 <part name="GND10" library="supply1" deviceset="GND" device=""/>
 <part name="J_PD4" library="jumper" deviceset="SJ" device=""/>
+<part name="U$3" library="lib-user" deviceset="GND" device=""/>
 </parts>
 <sheets>
@@
 <wire x1="73.66" y1="91.44" x2="73.66" y2="0" width="0.254" layer="90"/>
 <wire x1="73.66" y1="91.44" x2="276.86" y2="91.44" width="0.254" layer="90"/>
+<wire x1="124.46" y1="-33.02" x2="154.94" y2="-33.02" width="0.4064" layer="94" style="shortdash"/>
 </plain>
 <instances>
@@
 <attribute name="VALUE" x="114.3" y="-66.04" size="1.778" layer="96"/>
 </instance>
-<instance part="3L3" gate="G$1" x="121.92" y="-35.56" smashed="yes" rot="R90">
-<attribute name="NAME" x="119.38" y="-31.75" size="1.778" layer="95" rot="R180"/>
-<attribute name="VALUE" x="129.54" y="-31.75" size="1.778" layer="96" rot="R180"/>
-</instance>
-<instance part="3D3" gate="G$1" x="144.78" y="-45.72" smashed="yes">
-<attribute name="NAME" x="144.78" y="-40.1574" size="1.778" layer="95"/>
-<attribute name="VALUE" x="142.24" y="-42.9514" size="1.778" layer="96"/>
-</instance>
-<instance part="3C14" gate="G$1" x="147.32" y="-66.04" smashed="yes" rot="MR0">
-<attribute name="NAME" x="141.224" y="-63.881" size="1.778" layer="95" rot="MR180"/>
-<attribute name="VALUE" x="141.224" y="-66.421" size="1.778" layer="96" rot="MR180"/>
+<instance part="3L3" gate="G$1" x="129.54" y="-35.56" smashed="yes" rot="R90">
+<attribute name="NAME" x="127" y="-26.67" size="1.778" layer="95" rot="R180"/>
+<attribute name="VALUE" x="137.16" y="-26.67" size="1.778" layer="96" rot="R180"/>
+</instance>
+<instance part="3D3" gate="G$1" x="149.86" y="-45.72" smashed="yes">
+<attribute name="NAME" x="149.86" y="-40.1574" size="1.778" layer="95"/>
+<attribute name="VALUE" x="147.32" y="-42.9514" size="1.778" layer="96"/>
+</instance>
+<instance part="3C14" gate="G$1" x="147.32" y="-60.96" smashed="yes" rot="MR0">
+<attribute name="NAME" x="141.224" y="-58.801" size="1.778" layer="95" rot="MR180"/>
+<attribute name="VALUE" x="141.224" y="-61.341" size="1.778" layer="96" rot="MR180"/>
 </instance>
 <instance part="3R9" gate="G$1" x="124.46" y="-76.2"/>
@@
 <attribute name="VALUE" x="127" y="-93.98" size="1.778" layer="96"/>
 </instance>
-<instance part="U$27" gate="G$1" x="139.7" y="-93.98"/>
+<instance part="U$27" gate="G$1" x="139.7" y="-91.44"/>
 <instance part="R4" gate="G$1" x="124.46" y="-93.98" rot="R90"/>
 <instance part="3R1B3" gate="G$1" x="88.9" y="-45.72" smashed="yes" rot="R90">
@@
 </instance>
 <instance part="U$13" gate="G$1" x="160.02" y="-55.88"/>
-<instance part="3L4" gate="G$1" x="152.4" y="-35.56" smashed="yes" rot="R90">
-<attribute name="NAME" x="149.86" y="-31.75" size="1.778" layer="95" rot="R180"/>
-<attribute name="VALUE" x="160.02" y="-31.75" size="1.778" layer="96" rot="R180"/>
+<instance part="3L4" gate="G$1" x="149.86" y="-35.56" smashed="yes" rot="R90">
+<attribute name="NAME" x="147.32" y="-26.67" size="1.778" layer="95" rot="R180"/>
+<attribute name="VALUE" x="157.48" y="-26.67" size="1.778" layer="96" rot="R180"/>
 </instance>
 <instance part="3D4" gate="G$1" x="165.1" y="-35.56" smashed="yes">
@@
 </instance>
 <instance part="U$14" gate="G$1" x="175.26" y="-48.26"/>
+<instance part="U$3" gate="G$1" x="147.32" y="-68.58"/>
 </instances>
 <busses>
@@
 </segment>
 <segment>
+<pinref part="3C14" gate="G$1" pin="2"/>
+<wire x1="147.32" y1="-66.04" x2="147.32" y2="-68.58" width="0.1524" layer="91"/>
+<pinref part="U$3" gate="G$1" pin="GND"/>
+</segment>
+<segment>
 <pinref part="U$27" gate="G$1" pin="GND"/>
 <pinref part="VT1" gate="A" pin="S"/>
-<wire x1="139.7" y1="-93.98" x2="139.7" y2="-91.44" width="0.1524" layer="91"/>
 <wire x1="139.7" y1="-91.44" x2="139.7" y2="-88.9" width="0.1524" layer="91"/>
-<junction x="139.7" y="-91.44"/>
-<pinref part="3C14" gate="G$1" pin="2"/>
-<wire x1="147.32" y1="-71.12" x2="147.32" y2="-91.44" width="0.1524" layer="91"/>
-<wire x1="147.32" y1="-91.44" x2="139.7" y2="-91.44" width="0.1524" layer="91"/>
 </segment>
 <segment>
@@
 <pinref part="DA7" gate="G$1" pin="TC"/>
 <wire x1="137.16" y1="-55.88" x2="147.32" y2="-55.88" width="0.1524" layer="91"/>
-<wire x1="147.32" y1="-55.88" x2="147.32" y2="-63.5" width="0.1524" layer="91"/>
+<wire x1="147.32" y1="-55.88" x2="147.32" y2="-58.42" width="0.1524" layer="91"/>
 </segment>
 </net>
@@
 <segment>
 <pinref part="DA7" gate="G$1" pin="SWC"/>
-<pinref part="3D3" gate="G$1" pin="A"/>
 <wire x1="137.16" y1="-45.72" x2="139.7" y2="-45.72" width="0.1524" layer="91"/>
 <pinref part="3L3" gate="G$1" pin="2"/>
-<wire x1="129.54" y1="-35.56" x2="139.7" y2="-35.56" width="0.1524" layer="91"/>
+<wire x1="137.16" y1="-35.56" x2="139.7" y2="-35.56" width="0.1524" layer="91"/>
 <wire x1="139.7" y1="-45.72" x2="139.7" y2="-35.56" width="0.1524" layer="91"/>
-<junction x="139.7" y="-45.72"/>
-<wire x1="139.7" y1="-45.72" x2="142.24" y2="-45.72" width="0.1524" layer="91"/>
 <pinref part="3L4" gate="G$1" pin="1"/>
-<wire x1="144.78" y1="-35.56" x2="139.7" y2="-35.56" width="0.1524" layer="91"/>
+<wire x1="142.24" y1="-35.56" x2="139.7" y2="-35.56" width="0.1524" layer="91"/>
 <junction x="139.7" y="-35.56"/>
 </segment>
@@
 <pinref part="3R1B3" gate="G$1" pin="2"/>
 <pinref part="3L3" gate="G$1" pin="1"/>
-<wire x1="104.14" y1="-35.56" x2="114.3" y2="-35.56" width="0.1524" layer="91"/>
+<wire x1="104.14" y1="-35.56" x2="121.92" y2="-35.56" width="0.1524" layer="91"/>
 <wire x1="99.06" y1="-35.56" x2="93.98" y2="-35.56" width="0.1524" layer="91"/>
 <wire x1="93.98" y1="-35.56" x2="93.98" y2="-40.64" width="0.1524" layer="91"/>
@@
 <pinref part="3D4" gate="G$1" pin="A"/>
 <pinref part="3L4" gate="G$1" pin="2"/>
-<wire x1="162.56" y1="-35.56" x2="160.02" y2="-35.56" width="0.1524" layer="91"/>
-</segment>
-</net>
-<net name="N$74" class="0">
-<segment>
-<wire x1="116.84" y1="-30.48" x2="157.48" y2="-30.48" width="0.1524" layer="91"/>
+<wire x1="162.56" y1="-35.56" x2="157.48" y2="-35.56" width="0.1524" layer="91"/>
 </segment>
 </net>
@@
 <wire x1="160.02" y1="-45.72" x2="160.02" y2="-48.26" width="0.1524" layer="91"/>
 <pinref part="3D3" gate="G$1" pin="C"/>
-<wire x1="147.32" y1="-45.72" x2="160.02" y2="-45.72" width="0.1524" layer="91"/>
-</segment>
-</net>
+<wire x1="152.4" y1="-45.72" x2="160.02" y2="-45.72" width="0.1524" layer="91"/>
+</segment>
+</net>
+<net name="N$45" class="0">
+<segment>
+<pinref part="3D3" gate="G$1" pin="A"/>
+<wire x1="144.78" y1="-45.72" x2="147.32" y2="-45.72" width="0.1524" layer="91"/>
+</segment>
+</net>

Commit message: .
Changed lines of the file:
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@@
 <setting verticaltext="up"/>
 </settings>
-<grid distance="0.1" unitdist="inch" unit="mil" style="lines" multiple="1" display="yes" altdistance="0.01" altunitdist="inch" altunit="inch"/>
+<grid distance="100" unitdist="mil" unit="mil" style="lines" multiple="1" display="yes" altdistance="0.01" altunitdist="inch" altunit="inch"/>
 <layers>
 <layer number="1" name="Top" color="4" fill="1" visible="no" active="no"/>
@@
 <wire x1="73.66" y1="91.44" x2="276.86" y2="91.44" width="0.254" layer="90"/>
 <wire x1="124.46" y1="-33.02" x2="154.94" y2="-33.02" width="0.4064" layer="94" style="shortdash"/>
+<circle x="125.73" y="-36.195" radius="0.1778" width="0.762" layer="94"/>
+<circle x="146.05" y="-36.195" radius="0.1778" width="0.762" layer="94"/>
 </plain>
 <instances>

Commit message: sch
Parts:
- removed 3C15: 22u/100V, resistor:CPOL-EUE2.5-6
- removed 3D3, 3D4: RK19(1N5819), diode:SCHOTTKY-DIODESMD
- added D1: UF4007, diode:1N4004
- 3L1A: value 230uH -> 100uH
- 3L1B: value 230uH -> 6800uH
- renumbered 3L3 to 3L1A, 3L4 to 3L1B
Connections:
- net N$24 renamed Z_GREEN
- net N$56 renamed Z_BLUE
- removed net N$45: 3D3.A
- removed net N$57: 3R10.2, DA7.GND, DA7.SWE, VT1.D
- removed net N$73: 3D4.A, 3L1B.2
- new net Z_YELLOW: 3L1B.2, D1.A
- net GND: no longer 3C15.-
- net N$12: now also 3R10.1, DA7.GND, DA7.SWE, VT1.D; no longer 3C15.+, 3D3.C
- net N$25: now also 3R10.2; no longer 3R10.1
- net N$94: now also D1.C; no longer 3D4.C
Other:
- moved on the sheet: 3C14, 3R10, 3R9

Commit message: .
Parts:
- removed 3D2: RK19(1N5819), diode:SCHOTTKY-DIODESMD
- removed 3L1B: 6800uH, rcl:L-US6000-XXX-RC
- removed 3L2: 230uH, rcl:L-US6000-XXX-RC
- added 3C15: 100n, resistor:C-EU025-025X050
- added 3L2B: (no value), pinhead:PINHD-1X1
- 3C16: device resistor:CPOL-EUE2.5-6 -> resistor:CPOL-EUE5-8.5
- 3R9: value 120k -> 130k
Connections:
- removed net N$26: 3D2.A, 3L2.2, DA5.SWC
- removed net N$92: 2L4.1, 3C6.+, 3C7.1, 3D2.C, 3R5.2
- removed net N$94: 3C16.+, 3R9.2, D1.C
- new net N$24: 3C15.2, 3C16.+, 3R9.2, D1.C
- new net N$45: 2L4.1, 3C6.+, 3C7.1
- net GND: now also 3C15.1
- net N$51: no longer 3R5.1, 3R6.1
- net N$54: no longer 3L2.1
- net N$58: no longer 3R6.2
- net Z_GREEN: no longer 3L1B.1
- net Z_YELLOW: now also 3L2B.1; no longer 3L1B.2
Other:
- note added: "+20V"
- note added: "10mm"
- note added: "13-14mm"
- note added: "2k"
- note added: "30k"
- note added: "34R1"
- note added: "34R2"
- note added: "5mm"
- note added: "6800uH"
- note added: "7mm"
- note added: "I 49w 0.32mm > 105uH II 400w 0.15mm > 6.8mH"
- note added: "SS16"
- moved on the sheet: 3C14, 3C16, 3C17, 3C5, 3C8, 3L1A, 3R10, 3R11, 3R12, 3R1B1, 3R1B2, 3R1B3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

Commit message: .
Parts:
- removed 3C6: 22u/100V, resistor:CPOL-EUE2.5-6
- removed 3C7: 100n, resistor:C-EUC0805K
- removed 3L1A: 100uH, rcl:L-US6000-XXX-RC
- added 3L2G, 3L2Y: (no value), b333:PINHD-1X1
- added L: L, b333:L
- 3C16: device resistor:CPOL-EUE5-8.5 -> resistor:CPOL-EUTT5D9L
- 3L2B: device pinhead:PINHD-1X1 -> b333:PINHD-1X1
Connections:
- removed net N$45: 2L4.1, 3C6.+, 3C7.1
- net +40V: now also 3C10.2; no longer 3C10.1
- net GND: now also 3C10.1; no longer 3C10.2, 3C6.-, 3C7.2
- net N$24: now also 2L4.1
- net Z_BLUE: now also 3L2B.1; no longer 3L1A.1
- net Z_GREEN: now also 3L2G.1; no longer 3L1A.2
- net Z_YELLOW: now also 3L2Y.1; no longer 3L2B.1
Other:
- note added: "100uH"
- note removed: "10mm"
- note removed: "13-14mm"
- note removed: "5mm"
- note removed: "7mm"
- moved on the sheet: 2L4, 3C14, 3C15, 3C16, 3C17, 3C9, 3R10, 3R11, 3R12, 3R1B3, 3R1B4, 3R9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
