File: HW/EAGLE/b333.sch (EAGLE design)
At the start: 195 parts, among them Q1 2N4126, Q2 2N4126, Q5 NMOSD, X1 USB MICRO

Commit message: .
Parts:
- DIS1: device display-lcd:TUXGR_16X2_R2 -> b333:TUXGR_16X2_R2
Connections:
- net GND: no longer SL1.1
Changed lines of the file:
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@@
 <grid distance="100" unitdist="mil" unit="mil" style="lines" multiple="1" display="yes" altdistance="0.01" altunitdist="inch" altunit="inch"/>
 <layers>
-<layer number="1" name="Top" color="4" fill="1" visible="no" active="no"/>
-<layer number="2" name="Route2" color="1" fill="3" visible="no" active="no"/>
-<layer number="3" name="Route3" color="4" fill="3" visible="no" active="no"/>
-<layer number="4" name="Route4" color="1" fill="4" visible="no" active="no"/>
-<layer number="5" name="Route5" color="4" fill="4" visible="no" active="no"/>
-<layer number="6" name="Route6" color="1" fill="8" visible="no" active="no"/>
-<layer number="7" name="Route7" color="4" fill="8" visible="no" active="no"/>
-<layer number="8" name="Route8" color="1" fill="2" visible="no" active="no"/>
-<layer number="9" name="Route9" color="4" fill="2" visible="no" active="no"/>
-<layer number="10" name="Route10" color="1" fill="7" visible="no" active="no"/>
-<layer number="11" name="Route11" color="4" fill="7" visible="no" active="no"/>
-<layer number="12" name="Route12" color="1" fill="5" visible="no" active="no"/>
-<layer number="13" name="Route13" color="4" fill="5" visible="no" active="no"/>
-<layer number="14" name="Route14" color="1" fill="6" visible="no" active="no"/>
-<layer number="15" name="Route15" color="4" fill="6" visible="no" active="no"/>
-<layer number="16" name="Bottom" color="1" fill="1" visible="no" active="no"/>
-<layer number="17" name="Pads" color="2" fill="1" visible="no" active="no"/>
-<layer number="18" name="Vias" color="2" fill="1" visible="no" active="no"/>
-<layer number="19" name="Unrouted" color="6" fill="1" visible="no" active="no"/>
-<layer number="20" name="Dimension" color="15" fill="1" visible="no" active="no"/>
-<layer number="21" name="tPlace" color="7" fill="1" visible="no" active="no"/>
-<layer number="22" name="bPlace" color="7" fill="1" visible="no" active="no"/>
-<layer number="23" name="tOrigins" color="15" fill="1" visible="no" active="no"/>
-<layer number="24" name="bOrigins" color="15" fill="1" visible="no" active="no"/>
-<layer number="25" name="tNames" color="7" fill="1" visible="no" active="no"/>
-<layer number="26" name="bNames" color="7" fill="1" visible="no" active="no"/>
-<layer number="27" name="tValues" color="7" fill="1" visible="no" active="no"/>
-<layer number="28" name="bValues" color="7" fill="1" visible="no" active="no"/>
+<layer number="1" name="Top" color="4" fill="1" visible="yes" active="no"/>
+<layer number="2" name="Route2" color="1" fill="3" visible="yes" active="no"/>
+<layer number="3" name="Route3" color="4" fill="3" visible="yes" active="no"/>
+<layer number="4" name="Route4" color="1" fill="4" visible="yes" active="no"/>
+<layer number="5" name="Route5" color="4" fill="4" visible="yes" active="no"/>
+<layer number="6" name="Route6" color="1" fill="8" visible="yes" active="no"/>
+<layer number="7" name="Route7" color="4" fill="8" visible="yes" active="no"/>
+<layer number="8" name="Route8" color="1" fill="2" visible="yes" active="no"/>
+<layer number="9" name="Route9" color="4" fill="2" visible="yes" active="no"/>
+<layer number="10" name="Route10" color="1" fill="7" visible="yes" active="no"/>
+<layer number="11" name="Route11" color="4" fill="7" visible="yes" active="no"/>
+<layer number="12" name="Route12" color="1" fill="5" visible="yes" active="no"/>
+<layer number="13" name="Route13" color="4" fill="5" visible="yes" active="no"/>
+<layer number="14" name="Route14" color="1" fill="6" visible="yes" active="no"/>
+<layer number="15" name="Route15" color="4" fill="6" visible="yes" active="no"/>
+<layer number="16" name="Bottom" color="1" fill="1" visible="yes" active="no"/>
+<layer number="17" name="Pads" color="2" fill="1" visible="yes" active="no"/>
+<layer number="18" name="Vias" color="2" fill="1" visible="yes" active="no"/>
+<layer number="19" name="Unrouted" color="6" fill="1" visible="yes" active="no"/>
+<layer number="20" name="Dimension" color="15" fill="1" visible="yes" active="no"/>
+<layer number="21" name="tPlace" color="7" fill="1" visible="yes" active="no"/>
+<layer number="22" name="bPlace" color="7" fill="1" visible="yes" active="no"/>
+<layer number="23" name="tOrigins" color="15" fill="1" visible="yes" active="no"/>
+<layer number="24" name="bOrigins" color="15" fill="1" visible="yes" active="no"/>
+<layer number="25" name="tNames" color="7" fill="1" visible="yes" active="no"/>
+<layer number="26" name="bNames" color="7" fill="1" visible="yes" active="no"/>
+<layer number="27" name="tValues" color="7" fill="1" visible="yes" active="no"/>
+<layer number="28" name="bValues" color="7" fill="1" visible="yes" active="no"/>
 <layer number="29" name="tStop" color="7" fill="3" visible="no" active="no"/>
 <layer number="30" name="bStop" color="7" fill="6" visible="no" active="no"/>
@@
 <layer number="35" name="tGlue" color="7" fill="4" visible="no" active="no"/>
 <layer number="36" name="bGlue" color="7" fill="5" visible="no" active="no"/>
-<layer number="37" name="tTest" color="7" fill="1" visible="no" active="no"/>
-<layer number="38" name="bTest" color="7" fill="1" visible="no" active="no"/>
+<layer number="37" name="tTest" color="7" fill="1" visible="yes" active="no"/>
+<layer number="38" name="bTest" color="7" fill="1" visible="yes" active="no"/>
 <layer number="39" name="tKeepout" color="4" fill="11" visible="no" active="no"/>
 <layer number="40" name="bKeepout" color="1" fill="11" visible="no" active="no"/>
@@
 <layer number="44" name="Drills" color="7" fill="1" visible="no" active="no"/>
 <layer number="45" name="Holes" color="7" fill="1" visible="no" active="no"/>
-<layer number="46" name="Milling" color="3" fill="1" visible="no" active="no"/>
-<layer number="47" name="Measures" color="7" fill="1" visible="no" active="no"/>
-<layer number="48" name="Document" color="7" fill="1" visible="no" active="no"/>
-<layer number="49" name="Reference" color="7" fill="1" visible="no" active="no"/>
-<layer number="50" name="dxf" color="7" fill="1" visible="no" active="no"/>
-<layer number="51" name="tDocu" color="7" fill="1" visible="no" active="no"/>
-<layer number="52" name="bDocu" color="7" fill="1" visible="no" active="no"/>
-<layer number="53" name="tGND_GNDA" color="7" fill="9" visible="no" active="no"/>
-<layer number="54" name="bGND_GNDA" color="1" fill="9" visible="no" active="no"/>
-<layer number="56" name="wert" color="7" fill="1" visible="no" active="no"/>
-<layer number="57" name="tCAD" color="7" fill="1" visible="no" active="no"/>
+<layer number="46" name="Milling" color="3" fill="1" visible="yes" active="no"/>
+<layer number="47" name="Measures" color="7" fill="1" visible="yes" active="no"/>
+<layer number="48" name="Document" color="7" fill="1" visible="yes" active="no"/>
+<layer number="49" name="Reference" color="7" fill="1" visible="yes" active="no"/>
+<layer number="50" name="dxf" color="7" fill="1" visible="yes" active="no"/>
+<layer number="51" name="tDocu" color="6" fill="1" visible="yes" active="no"/>
+<layer number="52" name="bDocu" color="7" fill="1" visible="yes" active="no"/>
+<layer number="53" name="tGND_GNDA" color="7" fill="9" visible="yes" active="no"/>
+<layer number="54" name="bGND_GNDA" color="1" fill="9" visible="yes" active="no"/>
+<layer number="56" name="wert" color="7" fill="1" visible="yes" active="no"/>
+<layer number="57" name="tCAD" color="7" fill="1" visible="yes" active="no"/>
 <layer number="90" name="Modules" color="5" fill="1" visible="yes" active="yes"/>
 <layer number="91" name="Nets" color="2" fill="1" visible="yes" active="yes"/>
@@
 <part name="T5" library="pinhead" deviceset="PINHD-1X1" device=""/>
 <part name="T6" library="pinhead" deviceset="PINHD-1X1" device=""/>
-<part name="DIS1" library="display-lcd" deviceset="TUXGR_16X2_R2" device=""/>
+<part name="DIS1" library="b333" deviceset="TUXGR_16X2_R2" device=""/>
 <part name="D8" library="v-reg" deviceset="TL431CLP" device="" value="TL431"/>
 <part name="U$53" library="lib-user" deviceset="GND" device=""/>
@@
 </segment>
 <segment>
-<pinref part="SL1" gate="G$1" pin="1"/>
-<pinref part="U$7" gate="G$1" pin="GND"/>
-<wire x1="114.3" y1="93.98" x2="114.3" y2="91.44" width="0.1524" layer="91"/>
-</segment>
-<segment>
 <pinref part="U$65" gate="G$1" pin="GND"/>
 <pinref part="R8" gate="G$1" pin="1"/>
@@
 <junction x="195.58" y="58.42"/>
 <junction x="200.66" y="58.42"/>
-</segment>
-</net>
+<label x="198.12" y="81.28" size="1.778" layer="95" rot="R180"/>
+<junction x="200.66" y="81.28"/>
+</segment>
+</net>

Commit message: .
Parts:
- 3C16: device resistor:CPOL-EUTT5D9L -> ct-pack:CPOL-EUTT5D9L
Changed lines of the file:
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@@
 <part name="U$65" library="lib-user" deviceset="GND" device=""/>
 <part name="3R1B4" library="resistor" deviceset="R-EU_" device="R1206" value="2R"/>
-<part name="3C16" library="resistor" deviceset="CPOL-EU" device="TT5D9L" value="22u/100V"/>
+<part name="3C16" library="ct-pack" deviceset="CPOL-EU" device="TT5D9L" value="22u/100V"/>
 <part name="U$14" library="lib-user" deviceset="GND" device=""/>
 <part name="FRAME3" library="frames" deviceset="DINA4_L" device=""/>

Commit message: .sh
Parts:
- removed 0S1: TEST, switch-omron:10-XX
- removed 1Q3, 1Q4, Q5: NMOSD, DSS:NMOSD
- removed 1R14: 270, resistor:R-EU_R1206W
- removed 1R15: 27K, resistor:R-EU_R0805
- removed 1R6: 470K, resistor:R-EU_0207/10
- removed 1R7, R1: 1M, resistor:R-EU_R0805
- removed 1R8: 300, resistor:R-EU_R0805
- removed 1RC1: 22K, resistor:R-EU_R0805
- removed 1RC2*: 4K3, resistor:R-EU_R1206W
- removed 3C1: 100u, resistor:CPOL-EUE2.5-6
- removed 3C2: 1n, resistor:C-EUC0805K
- removed 3C3: 47u/50V, resistor:CPOL-EUE2.5-6
- removed 3C4, C2: 100n, resistor:C-EUC0805K
- removed 3D1: 1N5819, diode:DIODE-DO41-10
- removed 3L1: 180uH, inductor-neosid:SD12-1000
- removed 3R1, 3R1B: 1R, resistor:R-EU_R0805
- removed 3R2: 180R, resistor:R-EU_R0805
- removed 3R3, R2, R3: 2K, resistor:R-EU_R0805
- removed 3R4: 62K, resistor:R-EU_R0805
- removed 4R1, 4R2: 100, resistor:R-EU_R0805
- removed 4R3: 270, resistor:R-EU_R0805
- removed 4R4: 47K, resistor:R-EU_R1206W
- removed 4R5: 47K, resistor:R-EU_R0805
- removed 4Y1, 4Y2: РЭС55А, relay_ussr:РЭС55А
- removed C1: 100n, resistor:C-EUC0805
- removed D4: MC34063AD, mc34063:MC34063AD
- removed D5, D6: (no value), diode:DIODE-SOD80C
- removed J1, J2, J3, J4: (no value), jumper:SJ
- removed OK1: PC817, optocoupler:PC817
- removed R5: 20K, resistor:R-EU_R0805
- removed R6: 180K, resistor:R-EU_R0805
- removed R7: 10K, resistor:R-EU_R1206W
- removed S1: 9077-2, switch-misc:9077-2
- removed T1, T2, T3, ZEN_A, ZEN_K: (no value), pinhead:PINHD-1X1
- removed VD2: LL4148, diode:1N4148DO35-7
- added 3R5: 20K, resistor:R-EU_R0805
- added R18: 10.0k, resistor:R-EU_R0805
- added TEST2: TT-P, transistor_tester:TT-P
- added VT3: FS8205A, FS8205A:DMN3024LSD
- added X2: USB MICRO, SmartPrj:MYCON2_USB-MINI-B
- 3C10, 3C13: device resistor:C-EUC0805K -> resistor:C-EU025-025X050
- 3C15: device resistor:C-EU025-025X050 -> resistor:C-EU050-025X075
- 3C9: value 47u/50V -> 10u/100V
- 3R9: value 130k -> 120k
- R16: value 180.0k -> 330.0k
- VT6: value BF423 -> КТ502
Connections:
- net +40V renamed +90.5V
- removed net KEY: 0S1.S, 0S1.S1, D6.A, R2.1, S11.S, S12.S
- removed net N$1: 4R4.1, 4R5.1, Q5.G
- removed net N$10: 1Q4.D, 3C2.2, 3R3.1, D4.GND, J1.1, J2.1, ZEN_A.1
- removed net N$11: 1R14.1
- removed net N$110: 4R1.1, 4R2.1
- removed net N$114: 1R6.1
- removed net N$115: 1R6.2
- removed net N$18: R16.2, VT6.C, ZEN_K1.1
- removed net N$2: D5.A
- removed net N$20: 1R7.1, D6.C, OK1.EMIT
- removed net N$27: 3C2.1, D4.TC
- removed net N$28: 3D1.A, 3L1.2, D4.SWC, J3.1
- removed net N$29: 3R3.2, 3R4.1, D4.FB, J2.2
- removed net N$30: 3C3.+, 3C4.1, 3D1.C, 3R4.2, J3.2, J4.2, R7.2
- removed net N$31: 4R3.2, 4Y1G$1.2, 4Y2G$1.2
- removed net N$32: 3R2.2, D4.DC
- removed net N$33: 3L1.1, 3R1.2, 3R1B.2, 3R2.1, D4.IS
- removed net N$34: 1R8.2, OK1.A
- removed net N$46: 4R1.2, 4Y1G$2.P
- removed net N$47: 4R2.2, 4Y2G$2.P
- removed net N$48: 1Q3.G, 1R7.2, R1.1
- removed net N$49: D4.SWE, J1.2, VD2.A
- removed net N$5: D5.C
- removed net N$50: 1Q4.G, R2.2, R3.1
- removed net N$6: 1RC1.2, 1RC2*.2
- removed net N$7: 4Y1G$1.1, 4Y2G$1.1, Q5.D
- removed net N$9: J4.1, R6.2, R7.1, ZEN_K.1
- removed net PC1: 4Y2G$2.O
- removed net PC2: 4Y1G$2.O
- removed net PC4: 4R4.2
- removed net PD6: 1R8.1
- removed net PD7: 1R15.2, C2.1, VD2.C
- removed net V-: 1Q3.S, R1.2
- new net N$19: 2L4.1, 3C15.2, 3C16.+, 3R5.2, D1.C
- new net N$23: 3R5.1, 3R9.2
- new net ZENER_A: DD1.PC3(ADC3/PCINT11), R18.2, VT6.C, ZEN_K1.1
- net +5V: no longer 0S1.P, 0S1.P1, 1R14.2, 1R15.1, 1RC1.1, 4R3.1
- net GND: no longer 1Q3.D, 1Q4.S, 1RC2*.1, 3C1.-, 3C3.-, 3C4.2, 4R5.2, 4Y1G$3.G, 4Y2G$3.G, C1.2, C2.2, OK1.C, Q5.S, R3.2, R5.1
- net N$24: now also R16.2, R18.1; no longer 2L4.1, 3C15.2, 3C16.+, 3R9.2, D1.C
- net PC3: no longer C1.1, DD1.PC3(ADC3/PCINT11), R5.2, R6.1
- net V+: no longer 3C1.+, 3R1.1, 3R1B.1, D4.VCC, OK1.COL, S11.P, S12.P
Other:
- note removed: "3C3 3C4"
- note removed: "3R1"
- note removed: "3R2 3R3 3R4"
- note removed: "J1 J2 J3 J4"
- note removed: "TEST"
- note removed: "V+ батарея 4,5в"
- note removed: "Напряжение"
- note removed: "Токовый режим"
- note removed: "Установлены"

Commit message: .
Parts:
- renumbered 3C10 to 6C6, 3C13 to 6C7, 3C14 to 6C2, 3C15 to 6C4, 3C16 to 6C3, 3C17 to 6C1, 3C9 to 6C5, 3R10 to 6R5, 3R11 to 6R2, 3R12 to 6R1C, 3R1B3 to 6R1B, 3R1B4 to 6R1A, 3R5 to 6R3, 3R9 to 6R4, D1 to 6VD1, D10 to 6VD3, D11 to 6VD4, D9 to 6VD2, R10 to 6R7, R11 to 6R8, R12 to 6R6, R13 to 6R9, R15 to 6R12, R16 to 6R11, R18 to 6R10, R29 to 6R13, R4 to 6R15, R8 to 6R14, VT1 to 6VT2, VT4 to 6VT3

Commit message: -rcllbr
Parts:
- 2L2: value 220uH -> 100uH; device rcl:L-US6000-XXX-RC -> ct-pack:L_LH7X10MM

Commit message: .
Parts:
- added 2R1: 1R, resistor:R-EU_R0805
- 2R7: value 18K -> 3.9k
- 2R8: value 56K -> 18k
Connections:
- net N$14: now also 2R1.2
- net V+: now also 2R1.1
Other:
- moved on the sheet: 2R6
