File: HW_EAGLE/b333.sch (EAGLE design)
At the start: 149 parts, among them Q1 2N4126, Q2 2N4126, X1 USB MICRO, X2 USB MICRO

Commit message: .
Parts:
- added JP3: (no value), b333:PINHD-X16-8
- 2L2: device ct-pack:L_LH7X10MM -> ct-pack:L_LV7X10MM
- 2L4: device rcl:L-US6000-XXX-RC -> ct-pack:L_LV7X10MM
- 5MA: device jumper:JP2N -> ct-pack:JUMPERJP2
- DIS1: value TUXGR_16X2_R2 -> LCD_16X2_R2; device b333:TUXGR_16X2_R2 -> b333:LCD_16X2_R2
Other:
- moved on the sheet: DIS1
Changed lines of the file:
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@@
 <parts>
 <part name="DA3" library="mc34063-2" deviceset="MC34063" device="AD"/>
-<part name="2L2" library="ct-pack" deviceset="L_" device="LH7X10MM" value="100uH"/>
+<part name="2L2" library="ct-pack" deviceset="L_" device="LV7X10MM" value="100uH"/>
 <part name="2C1" library="resistor" deviceset="C-EU" device="C0805K" value="150"/>
 <part name="U$6" library="lib-user" deviceset="GND" device=""/>
@@
 <part name="ZEN_K1" library="pinhead" deviceset="PINHD-1X1" device=""/>
 <part name="ZEN_A1" library="pinhead" deviceset="PINHD-1X1" device=""/>
-<part name="2L4" library="rcl" deviceset="L-US" device="6000-XXX-RC" value="220uH"/>
+<part name="2L4" library="ct-pack" deviceset="L_" device="LV7X10MM" value="220uH"/>
 <part name="U$36" library="lib-user" deviceset="GND" device=""/>
 <part name="6C5" library="resistor" deviceset="CPOL-EU" device="E2.5-6" value="10u/100V"/>
@@
 <part name="6R9" library="resistor" deviceset="R-EU_" device="R0805" value="39k"/>
 <part name="U$39" library="lib-user" deviceset="GND" device=""/>
-<part name="5MA" library="jumper" deviceset="JP2N" device="" value="10MA"/>
+<part name="5MA" library="ct-pack" deviceset="JUMPER" device="JP2" value="10MA"/>
 <part name="U$40" library="lib-user" deviceset="GND" device=""/>
 <part name="U$41" library="lib-user" deviceset="GND" device=""/>
@@
 <part name="T5" library="pinhead" deviceset="PINHD-1X1" device=""/>
 <part name="T6" library="pinhead" deviceset="PINHD-1X1" device=""/>
-<part name="DIS1" library="b333" deviceset="TUXGR_16X2_R2" device=""/>
+<part name="DIS1" library="b333" deviceset="LCD_16X2_R2" device=""/>
 <part name="D8" library="v-reg" deviceset="TL431CLP" device="" value="TL431"/>
 <part name="U$53" library="lib-user" deviceset="GND" device=""/>
@@
 <part name="6R10" library="resistor" deviceset="R-EU_" device="R0805" value="10.0k"/>
 <part name="2R1" library="resistor" deviceset="R-EU_" device="R0805" value="1R"/>
+<part name="JP3" library="b333" deviceset="PINHD-X16-8" device=""/>
 </parts>
 <sheets>
@@
 <attribute name="VALUE" x="217.17" y="125.73" size="1.778" layer="96" rot="R90"/>
 </instance>
-<instance part="DIS1" gate="G$1" x="256.54" y="154.94"/>
+<instance part="DIS1" gate="G$1" x="256.54" y="165.1"/>
 <instance part="D8" gate="G$1" x="124.46" y="139.7" smashed="yes" rot="MR90">
 <attribute name="NAME" x="120.65" y="133.35" size="1.778" layer="95" rot="MR90"/>
@@
 <attribute name="NAME" x="198.12" y="187.96" size="1.27" layer="95" rot="R180"/>
 </instance>
+<instance part="JP3" gate="A" x="256.54" y="152.4" rot="R90"/>
 </instances>
 <busses>

Commit message: rtrim
Parts:
- added 1C3: 100n, resistor:C-EUC0805K
- added 1R4, 1R5, 1R6: 10k, resistor:R-EU_R0805
- added R2: 10k, ct-pack:R-TRIMM3296W
- R35: device rcl:R-TRIMM3296W -> ct-pack:R-TRIMM3296W
Connections:
- net N$4 renamed PD4MC
- removed net N$72: 4R7.2, 4Y4G$2.P
- removed net N$97: C19.1, D12.C, JP2.1, R14.2, R17.2, R28.2, R9.2
- new net FO: 1R6.2, D3.C, R27.2, R28.1, T9.C
- new net N$1: 4Y4G$2.O, 4Y4G$2.P, 4Y4G$2.S
- new net N$2: C19.1, D12.C, JP2.1, R14.2, R17.2, R2.E, R28.2, R9.2
- new net N$6: 1R5.2, R2.A, R2.S
- new net N$7: 1C3.1, 1R6.1
- new net PD3: 1C3.2, 1R4.2, 1R5.1
- net GND: now also 1R4.1
- net PD4: no longer D3.C, R27.2, R28.1, T9.C
- net T2: no longer 4Y4G$2.O
Other:
- moved on the sheet: 4Y4, R28

Commit message: .
Parts:
- 1C2: value 220u/6V -> 330u/6V
- 2L2: value 100uH -> 30uH
- 2L3: value 220uH -> 330uH
Other:
- moved on the sheet: R19, R24, X1

Commit message: .
Parts:
- added C1: 100n, resistor:C-EUC0805K
- 2L2: device ct-pack:L_LV7X10MM -> ct-pack:L_LH7X10MM
Connections:
- net +5V/2: now also 6VT3.E
- net GND: no longer 6C1.-
- net N$12: now also C1.2
- net N$13: now also 2L2.1; no longer 2L2.2
- net N$14: now also 2L2.2; no longer 2L2.1
- net V+: now also C1.1; no longer 6C1.+, 6VT3.E

Commit message: .
Parts:
- removed C1: 100n, resistor:C-EUC0805K
- added 6C1A: 100u, resistor:CPOL-EUE2.5-6
- added D1: (no value), diode:ZENER-DIODESOD80C
- 6C1: value 100u -> 100n; device resistor:CPOL-EUE2.5-6 -> resistor:C-EUC0805K
- 6C5: device resistor:CPOL-EUE2.5-6 -> ct-pack:CPOL-EUE2.5-6
Connections:
- net ZENER_A renamed ZENER
- net GND: now also D1.A
- net N$12: now also 6C1.2; no longer C1.2
- net PC3: now also D1.C
- net V+: now also 6C1.1; no longer C1.1
Other:
- moved on the sheet: ZEN_A1, ZEN_K1
Changed lines of the file:
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@@
 <part name="2L4" library="ct-pack" deviceset="L_" device="LV7X10MM" value="220uH"/>
 <part name="U$36" library="lib-user" deviceset="GND" device=""/>
-<part name="6C5" library="resistor" deviceset="CPOL-EU" device="E2.5-6" value="10u/100V"/>
+<part name="6C5" library="ct-pack" deviceset="CPOL-EU" device="E2.5-6" value="10u/100V"/>
 <part name="6C6" library="resistor" deviceset="C-EU" device="025-025X050" value="100n"/>
 <part name="U$37" library="lib-user" deviceset="GND" device=""/>
@@
 <part name="6R2" library="resistor" deviceset="R-EU_" device="R0805" value="180R"/>
 <part name="6R1C" library="resistor" deviceset="R-EU_" device="R1206"/>
-<part name="6C1" library="resistor" deviceset="CPOL-EU" device="E2.5-6" value="100u"/>
+<part name="6C1A" library="resistor" deviceset="CPOL-EU" device="E2.5-6" value="100u"/>
 <part name="U$15" library="lib-user" deviceset="GND" device=""/>
 <part name="6VT2" library="DSS" deviceset="NMOS" device="D"/>
@@
 <part name="1C3" library="resistor" deviceset="C-EU" device="C0805K" value="100n"/>
 <part name="1R6" library="resistor" deviceset="R-EU_" device="R0805" value="10k"/>
-<part name="C1" library="resistor" deviceset="C-EU" device="C0805K" value="100n"/>
+<part name="6C1" library="resistor" deviceset="C-EU" device="C0805K" value="100n"/>
+<part name="D1" library="diode" deviceset="ZENER-DIODE" device="SOD80C"/>
+<part name="U$1" library="lib-user" deviceset="GND" device=""/>
 </parts>
 <sheets>
@@
 </segment>
 </net>
-<net name="ZENER_A" class="0">
+<net name="ZENER" class="0">
 <segment>
 <pinref part="DD1" gate="1" pin="PC3(ADC3/PCINT11)"/>
@@
 <instance part="U$29" gate="G$1" x="99.06" y="157.48"/>
 <instance part="U$30" gate="G$1" x="106.68" y="157.48"/>
-<instance part="ZEN_K1" gate="G$1" x="261.62" y="63.5" smashed="yes" rot="R270">
-<attribute name="NAME" x="265.43" y="66.675" size="1.778" layer="95"/>
-<attribute name="VALUE" x="256.54" y="69.85" size="1.778" layer="96" rot="R270"/>
-</instance>
-<instance part="ZEN_A1" gate="G$1" x="261.62" y="55.88" smashed="yes" rot="R90">
-<attribute name="NAME" x="265.43" y="53.975" size="1.778" layer="95"/>
-<attribute name="VALUE" x="266.7" y="49.53" size="1.778" layer="96" rot="R90"/>
+<instance part="ZEN_K1" gate="G$1" x="269.24" y="73.66" smashed="yes" rot="R270">
+<attribute name="NAME" x="265.43" y="69.215" size="1.778" layer="95"/>
+<attribute name="VALUE" x="264.16" y="80.01" size="1.778" layer="96" rot="R270"/>
+</instance>
+<instance part="ZEN_A1" gate="G$1" x="269.24" y="55.88" smashed="yes" rot="R90">
+<attribute name="NAME" x="265.43" y="59.055" size="1.778" layer="95"/>
+<attribute name="VALUE" x="274.32" y="49.53" size="1.778" layer="96" rot="R90"/>
 </instance>
 <instance part="2L4" gate="G$1" x="185.42" y="58.42" smashed="yes" rot="R90">
@@
 <attribute name="VALUE" x="193.04" y="62.23" size="1.778" layer="96" rot="R180"/>
 </instance>
-<instance part="U$36" gate="G$1" x="261.62" y="43.18"/>
+<instance part="U$36" gate="G$1" x="269.24" y="43.18"/>
 <instance part="6C5" gate="G$1" x="195.58" y="53.34" smashed="yes">
 <attribute name="NAME" x="199.263" y="46.2026" size="1.778" layer="95"/>
@@
 <attribute name="VALUE" x="88.138" y="67.31" size="1.778" layer="96" rot="R270"/>
 </instance>
-<instance part="6C1" gate="G$1" x="81.28" y="48.26" rot="MR0"/>
+<instance part="6C1A" gate="G$1" x="81.28" y="48.26" rot="MR0"/>
 <instance part="U$15" gate="G$1" x="81.28" y="40.64"/>
 <instance part="6VT2" gate="A" x="134.62" y="27.94" smashed="yes">
@@
 <attribute name="VALUE" x="11.43" y="177.038" size="1.778" layer="96" rot="MR0"/>
 </instance>
-<instance part="C1" gate="G$1" x="96.52" y="45.72" rot="MR0"/>
+<instance part="6C1" gate="G$1" x="96.52" y="45.72" rot="MR0"/>
+<instance part="D1" gate="G$1" x="261.62" y="50.8" rot="R90"/>
+<instance part="U$1" gate="G$1" x="261.62" y="43.18"/>
 </instances>
 <busses>
@@
 <segment>
 <pinref part="ZEN_A1" gate="G$1" pin="1"/>
-<wire x1="261.62" y1="53.34" x2="261.62" y2="43.18" width="0.1524" layer="91"/>
+<wire x1="269.24" y1="53.34" x2="269.24" y2="43.18" width="0.1524" layer="91"/>
 <pinref part="U$36" gate="G$1" pin="GND"/>
 </segment>
@@
 <pinref part="6R14" gate="G$1" pin="1"/>
 <wire x1="116.84" y1="10.16" x2="116.84" y2="12.7" width="0.1524" layer="91"/>
+</segment>
+<segment>
+<pinref part="D1" gate="G$1" pin="A"/>
+<pinref part="U$1" gate="G$1" pin="GND"/>
+<wire x1="261.62" y1="48.26" x2="261.62" y2="43.18" width="0.1524" layer="91"/>
 </segment>
 </net>
@@
 <pinref part="6R1A" gate="G$1" pin="1"/>
 <wire x1="81.28" y1="58.42" x2="81.28" y2="53.34" width="0.1524" layer="91"/>
-<pinref part="C1" gate="G$1" pin="1"/>
+<pinref part="6C1" gate="G$1" pin="1"/>
 <wire x1="96.52" y1="48.26" x2="96.52" y2="53.34" width="0.1524" layer="91"/>
 <junction x="96.52" y="53.34"/>
@@
 </segment>
 </net>
-<net name="ZENER_A" class="0">
+<net name="ZENER" class="0">
 <segment>
 <pinref part="VT6" gate="G$1" pin="C"/>
@@
 <wire x1="241.3" y1="73.66" x2="241.3" y2="86.36" width="0.1524" layer="91"/>
 <wire x1="241.3" y1="86.36" x2="254" y2="86.36" width="0.1524" layer="91"/>
-<wire x1="254" y1="86.36" x2="261.62" y2="86.36" width="0.1524" layer="91"/>
+<wire x1="254" y1="86.36" x2="269.24" y2="86.36" width="0.1524" layer="91"/>
 <pinref part="ZEN_K1" gate="G$1" pin="1"/>
-<wire x1="261.62" y1="66.04" x2="261.62" y2="86.36" width="0.1524" layer="91"/>
+<wire x1="269.24" y1="76.2" x2="269.24" y2="86.36" width="0.1524" layer="91"/>
 <pinref part="6R10" gate="G$1" pin="2"/>
 <wire x1="254" y1="83.82" x2="254" y2="86.36" width="0.1524" layer="91"/>
@@
 <wire x1="137.16" y1="33.02" x2="137.16" y2="35.56" width="0.1524" layer="91"/>
 <junction x="137.16" y="35.56"/>
-<pinref part="C1" gate="G$1" pin="2"/>
+<pinref part="6C1" gate="G$1" pin="2"/>
 <wire x1="96.52" y1="40.64" x2="96.52" y2="35.56" width="0.1524" layer="91"/>
 <wire x1="96.52" y1="35.56" x2="137.16" y2="35.56" width="0.1524" layer="91"/>
@@
 <wire x1="243.84" y1="53.34" x2="243.84" y2="58.42" width="0.1524" layer="91"/>
 <wire x1="254" y1="58.42" x2="254" y2="55.88" width="0.1524" layer="91"/>
-</segment>
-</net>
+<pinref part="D1" gate="G$1" pin="C"/>
+<wire x1="261.62" y1="53.34" x2="261.62" y2="58.42" width="0.1524" layer="91"/>
+<wire x1="261.62" y1="58.42" x2="254" y2="58.42" width="0.1524" layer="91"/>
+</segment>
+</net>
