File: HW_EAGLE/b333.sch (EAGLE design)
At the start: 152 parts, among them Q1 2N4126, Q2 2N4126, X1 USB MICRO

Commit message: .
Parts:
- removed Z1: 5v6, diode:ZENER-DIODESOD80C
- added 6VD5: 5v6, diode:ZENER-DIODESOD80C
- renumbered C1 to 3C1
Connections:
- net GND: now also 6VD5.A; no longer Z1.A
- net PC3: now also 6VD5.C; no longer Z1.C
Other:
- moved on the sheet: 1C3, 1R4, 1R5, 1R6, 6C7, 6R10, 6R11, 6R12, C14, C15, C16, C19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

Commit message: .
Parts:
- removed 1RC2*1: 4K3, resistor:R-EU_R1206W
- added 1RC3: 4K3, resistor:R-EU_R1206W
- 1R26: device resistor:R-EU_R1206W -> resistor:R-EU_R0805
- 5R3: device resistor:R-EU_R0805 -> resistor:R-EU_0204/7
Connections:
- net GND: now also 1RC3.1; no longer 1RC2*1.1
- net N$60: now also 1RC3.2; no longer 1RC2*1.2
Changed lines of the file:
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@@
 <layer number="23" name="tOrigins" color="15" fill="1" visible="yes" active="no"/>
 <layer number="24" name="bOrigins" color="15" fill="1" visible="yes" active="no"/>
-<layer number="25" name="tNames" color="7" fill="1" visible="yes" active="no"/>
+<layer number="25" name="tNames" color="6" fill="1" visible="yes" active="no"/>
 <layer number="26" name="bNames" color="7" fill="1" visible="yes" active="no"/>
 <layer number="27" name="tValues" color="7" fill="1" visible="yes" active="no"/>
@@
 <part name="U$10" library="lib-user" deviceset="GND" device=""/>
 <part name="3C1" library="resistor" deviceset="CPOL-EU" device="E2.5-6" value="50u"/>
-<part name="5R3" library="resistor" deviceset="R-EU_" device="R0805" value="3.9k"/>
+<part name="5R3" library="resistor" deviceset="R-EU_" device="0204/7" value="3.9k"/>
 <part name="5R4" library="resistor" deviceset="R-EU_" device="R0805" value="18k"/>
 <part name="2D2" library="diode" deviceset="SCHOTTKY-DIODE" device="SMD" value="SS12"/>
@@
 <part name="U$50" library="lib-user" deviceset="GND" device=""/>
 <part name="U$51" library="lib-user" deviceset="GND" device=""/>
-<part name="1RC2*1" library="resistor" deviceset="R-EU_" device="R1206W" value="4K3"/>
+<part name="1RC3" library="resistor" deviceset="R-EU_" device="R1206W" value="4K3"/>
 <part name="1RC2" library="resistor" deviceset="R-EU_" device="R0805" value="22K"/>
 <part name="1C7" library="resistor" deviceset="C-EU" device="C0805K" value="100n"/>
@@
 <part name="C17" library="resistor" deviceset="C-EU" device="C0805K" value="100n"/>
 <part name="P+9" library="supply1" deviceset="+5V" device=""/>
-<part name="1R26" library="resistor" deviceset="R-EU_" device="R1206W" value="270"/>
+<part name="1R26" library="resistor" deviceset="R-EU_" device="R0805" value="270"/>
 <part name="U$56" library="lib-user" deviceset="GND" device=""/>
 <part name="P+13" library="supply1" deviceset="+5V" device=""/>
@@
 <instance part="U$50" gate="G$1" x="45.72" y="81.28"/>
 <instance part="U$51" gate="G$1" x="259.08" y="124.46"/>
-<instance part="1RC2*1" gate="G$1" x="236.22" y="119.38" smashed="yes">
-<attribute name="NAME" x="232.41" y="120.8786" size="1.778" layer="95"/>
-<attribute name="VALUE" x="232.41" y="116.078" size="1.778" layer="96"/>
+<instance part="1RC3" gate="G$1" x="243.84" y="119.38" smashed="yes" rot="R90">
+<attribute name="NAME" x="242.3414" y="115.57" size="1.778" layer="95" rot="R90"/>
+<attribute name="VALUE" x="247.142" y="115.57" size="1.778" layer="96" rot="R90"/>
 </instance>
 <instance part="1RC2" gate="G$1" x="236.22" y="127" smashed="yes">
@@
 <attribute name="VALUE" x="278.13" y="123.698" size="1.778" layer="96"/>
 </instance>
-<instance part="U$56" gate="G$1" x="228.6" y="116.84"/>
+<instance part="U$56" gate="G$1" x="243.84" y="111.76"/>
 <instance part="P+13" gate="1" x="154.94" y="50.8" smashed="yes">
 <attribute name="VALUE" x="157.48" y="53.34" size="1.778" layer="96" rot="R180"/>
@@
 </segment>
 <segment>
-<wire x1="238.76" y1="129.54" x2="238.76" y2="149.86" width="0.1524" layer="91"/>
-<wire x1="248.92" y1="149.86" x2="248.92" y2="129.54" width="0.1524" layer="91"/>
-<wire x1="248.92" y1="129.54" x2="238.76" y2="129.54" width="0.1524" layer="91"/>
-<wire x1="261.62" y1="139.7" x2="261.62" y2="129.54" width="0.1524" layer="91"/>
-<wire x1="261.62" y1="129.54" x2="259.08" y2="129.54" width="0.1524" layer="91"/>
-<junction x="248.92" y="129.54"/>
-<wire x1="259.08" y1="129.54" x2="256.54" y2="129.54" width="0.1524" layer="91"/>
-<wire x1="256.54" y1="129.54" x2="254" y2="129.54" width="0.1524" layer="91"/>
-<wire x1="254" y1="129.54" x2="248.92" y2="129.54" width="0.1524" layer="91"/>
-<wire x1="259.08" y1="139.7" x2="259.08" y2="129.54" width="0.1524" layer="91"/>
-<junction x="259.08" y="129.54"/>
-<wire x1="256.54" y1="139.7" x2="256.54" y2="129.54" width="0.1524" layer="91"/>
-<junction x="256.54" y="129.54"/>
-<wire x1="254" y1="139.7" x2="254" y2="129.54" width="0.1524" layer="91"/>
-<junction x="254" y="129.54"/>
-<wire x1="276.86" y1="149.86" x2="276.86" y2="129.54" width="0.1524" layer="91"/>
-<wire x1="276.86" y1="129.54" x2="261.62" y2="129.54" width="0.1524" layer="91"/>
-<junction x="261.62" y="129.54"/>
+<wire x1="238.76" y1="134.62" x2="238.76" y2="149.86" width="0.1524" layer="91"/>
+<wire x1="248.92" y1="149.86" x2="248.92" y2="134.62" width="0.1524" layer="91"/>
+<wire x1="248.92" y1="134.62" x2="238.76" y2="134.62" width="0.1524" layer="91"/>
+<wire x1="261.62" y1="139.7" x2="261.62" y2="134.62" width="0.1524" layer="91"/>
+<wire x1="261.62" y1="134.62" x2="259.08" y2="134.62" width="0.1524" layer="91"/>
+<junction x="248.92" y="134.62"/>
+<wire x1="259.08" y1="134.62" x2="256.54" y2="134.62" width="0.1524" layer="91"/>
+<wire x1="256.54" y1="134.62" x2="254" y2="134.62" width="0.1524" layer="91"/>
+<wire x1="254" y1="134.62" x2="248.92" y2="134.62" width="0.1524" layer="91"/>
+<wire x1="259.08" y1="139.7" x2="259.08" y2="134.62" width="0.1524" layer="91"/>
+<junction x="259.08" y="134.62"/>
+<wire x1="256.54" y1="139.7" x2="256.54" y2="134.62" width="0.1524" layer="91"/>
+<junction x="256.54" y="134.62"/>
+<wire x1="254" y1="139.7" x2="254" y2="134.62" width="0.1524" layer="91"/>
+<junction x="254" y="134.62"/>
+<wire x1="276.86" y1="149.86" x2="276.86" y2="134.62" width="0.1524" layer="91"/>
+<wire x1="276.86" y1="134.62" x2="261.62" y2="134.62" width="0.1524" layer="91"/>
+<junction x="261.62" y="134.62"/>
 <pinref part="U$51" gate="G$1" pin="GND"/>
-<wire x1="259.08" y1="124.46" x2="259.08" y2="129.54" width="0.1524" layer="91"/>
+<wire x1="259.08" y1="124.46" x2="259.08" y2="134.62" width="0.1524" layer="91"/>
 <pinref part="JP3" gate="A" pin="5"/>
 <pinref part="JP3" gate="A" pin="1"/>
@@
 </segment>
 <segment>
-<pinref part="1RC2*1" gate="G$1" pin="1"/>
-<wire x1="231.14" y1="119.38" x2="228.6" y2="119.38" width="0.1524" layer="91"/>
+<pinref part="1RC3" gate="G$1" pin="1"/>
 <pinref part="U$56" gate="G$1" pin="GND"/>
-<wire x1="228.6" y1="119.38" x2="228.6" y2="116.84" width="0.1524" layer="91"/>
+<wire x1="243.84" y1="114.3" x2="243.84" y2="111.76" width="0.1524" layer="91"/>
 </segment>
 <segment>
@@
 <wire x1="243.84" y1="127" x2="243.84" y2="149.86" width="0.1524" layer="91"/>
 <wire x1="241.3" y1="127" x2="243.84" y2="127" width="0.1524" layer="91"/>
-<pinref part="1RC2*1" gate="G$1" pin="2"/>
-<wire x1="241.3" y1="119.38" x2="243.84" y2="119.38" width="0.1524" layer="91"/>
-<wire x1="243.84" y1="119.38" x2="243.84" y2="127" width="0.1524" layer="91"/>
+<pinref part="1RC3" gate="G$1" pin="2"/>
+<wire x1="243.84" y1="124.46" x2="243.84" y2="127" width="0.1524" layer="91"/>
 <junction x="243.84" y="127"/>
 <pinref part="JP3" gate="A" pin="3"/>
@@
 <wire x1="147.32" y1="91.44" x2="149.86" y2="91.44" width="0.1524" layer="91"/>
 <wire x1="149.86" y1="91.44" x2="149.86" y2="106.68" width="0.1524" layer="91"/>
-<wire x1="149.86" y1="106.68" x2="246.38" y2="106.68" width="0.1524" layer="91"/>
-<wire x1="246.38" y1="106.68" x2="246.38" y2="149.86" width="0.1524" layer="91"/>
+<wire x1="149.86" y1="106.68" x2="248.92" y2="106.68" width="0.1524" layer="91"/>
 <pinref part="J_PD4" gate="1" pin="2"/>
 <label x="142.24" y="106.68" size="1.778" layer="95"/>
+<wire x1="246.38" y1="127" x2="246.38" y2="149.86" width="0.1524" layer="91"/>
 <wire x1="149.86" y1="106.68" x2="142.24" y2="106.68" width="0.1524" layer="91"/>
 <junction x="149.86" y="106.68"/>
 <pinref part="JP3" gate="A" pin="4"/>
+<wire x1="248.92" y1="106.68" x2="248.92" y2="127" width="0.1524" layer="91"/>
+<wire x1="248.92" y1="127" x2="246.38" y2="127" width="0.1524" layer="91"/>
 </segment>
 </net>

Commit message: .
Parts:
- 5C3: device resistor:CPOL-EUE2-5 -> resistor:CPOL-EUE2.5-7
Changed lines of the file:
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@@
 <part name="5R4" library="resistor" deviceset="R-EU_" device="R0805" value="18k"/>
 <part name="2D2" library="diode" deviceset="SCHOTTKY-DIODE" device="SMD" value="SS12"/>
-<part name="5C3" library="resistor" deviceset="CPOL-EU" device="E2-5" value="330u/6V"/>
+<part name="5C3" library="resistor" deviceset="CPOL-EU" device="E2.5-7" value="330u/6V"/>
 <part name="5C4" library="resistor" deviceset="C-EU" device="C0805K" value="100n"/>
 <part name="U$18" library="lib-user" deviceset="GND" device=""/>

Commit message: .
Parts:
- GREEN, RED: device led:LEDCHIP-LED0805 -> led:LED5MM
- R19: device resistor:R-EU_R0805 -> resistor:R-EU_M0805
- R21: device resistor:R-EU_R0805 -> resistor:R-EU_R1206W
- R24: device resistor:R-EU_0204/7 -> resistor:R-EU_0207/10
Connections:
- removed net N$82: R22.1, RED.A
- removed net N$83: GREEN.A, R23.1
- new net N$4: R22.2, RED.C
- new net N$5: GREEN.C, R23.2
- net N$80: now also R22.1; no longer RED.C
- net N$81: now also R23.1; no longer GREEN.C
- net N$84: now also GREEN.A, RED.A; no longer R22.2, R23.2
Other:
- moved on the sheet: GREEN, R22, R23, RED
Changed lines of the file:
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@@
 <part name="U$41" library="lib-user" deviceset="GND" device=""/>
 <part name="DA1" library="TP4056" deviceset="TP4056" device=""/>
-<part name="R19" library="resistor" deviceset="R-EU_" device="R0805" value="0.5"/>
+<part name="R19" library="resistor" deviceset="R-EU_" device="M0805" value="0.5"/>
 <part name="VT2" library="TP4056+" deviceset="FS8205A" device="" value="FS8205A"/>
 <part name="DA2" library="TP4056+" deviceset="DW01" device="" value="DW01A"/>
 <part name="R20" library="resistor" deviceset="R-EU_" device="R0805" value="1k"/>
 <part name="C11" library="rcl" deviceset="C-EU" device="C0805" value="100n"/>
-<part name="R21" library="resistor" deviceset="R-EU_" device="R0805" value="100"/>
-<part name="RED" library="led" deviceset="LED" device="CHIP-LED0805"/>
-<part name="GREEN" library="led" deviceset="LED" device="CHIP-LED0805"/>
+<part name="R21" library="resistor" deviceset="R-EU_" device="R1206W" value="100"/>
+<part name="RED" library="led" deviceset="LED" device="5MM"/>
+<part name="GREEN" library="led" deviceset="LED" device="5MM"/>
 <part name="R22" library="resistor" deviceset="R-EU_" device="R0805" value="1k"/>
 <part name="R23" library="resistor" deviceset="R-EU_" device="R0805" value="1k"/>
 <part name="C12" library="rcl" deviceset="C-EU" device="C0805" value="100n"/>
-<part name="R24" library="resistor" deviceset="R-EU_" device="0204/7" value="1k2"/>
+<part name="R24" library="resistor" deviceset="R-EU_" device="0207/10" value="1k2"/>
 <part name="X1" library="SmartPrj" deviceset="MYCON2_USB-MINI-B" device="" value="USB MICRO"/>
 <part name="B-" library="TP4056_18650" deviceset="B-" device=""/>
@@
 <attribute name="VALUE" x="214.63" y="154.178" size="1.778" layer="96"/>
 </instance>
-<instance part="RED" gate="G$1" x="256.54" y="134.62" rot="MR0"/>
-<instance part="GREEN" gate="G$1" x="246.38" y="134.62" rot="MR0"/>
-<instance part="R22" gate="G$1" x="256.54" y="144.78" smashed="yes" rot="MR90">
-<attribute name="NAME" x="255.27" y="146.2786" size="1.778" layer="95" rot="MR0"/>
-<attribute name="VALUE" x="255.27" y="141.478" size="1.778" layer="96" rot="MR0"/>
-</instance>
-<instance part="R23" gate="G$1" x="246.38" y="144.78" smashed="yes" rot="MR90">
-<attribute name="NAME" x="245.11" y="146.2786" size="1.778" layer="95" rot="MR0"/>
-<attribute name="VALUE" x="245.11" y="141.478" size="1.778" layer="96" rot="MR0"/>
+<instance part="RED" gate="G$1" x="256.54" y="147.32" rot="MR0"/>
+<instance part="GREEN" gate="G$1" x="246.38" y="147.32" rot="MR0"/>
+<instance part="R22" gate="G$1" x="256.54" y="134.62" smashed="yes" rot="MR90">
+<attribute name="NAME" x="255.27" y="136.1186" size="1.778" layer="95" rot="MR0"/>
+<attribute name="VALUE" x="255.27" y="131.318" size="1.778" layer="96" rot="MR0"/>
+</instance>
+<instance part="R23" gate="G$1" x="246.38" y="134.62" smashed="yes" rot="MR90">
+<attribute name="NAME" x="245.11" y="136.1186" size="1.778" layer="95" rot="MR0"/>
+<attribute name="VALUE" x="245.11" y="131.318" size="1.778" layer="96" rot="MR0"/>
 </instance>
 <instance part="C12" gate="G$1" x="238.76" y="116.84"/>
@@
 <segment>
 <wire x1="231.14" y1="124.46" x2="256.54" y2="124.46" width="0.1524" layer="91"/>
+<pinref part="DA1" gate="G$1" pin="CHRG"/>
+<pinref part="R22" gate="G$1" pin="1"/>
 <wire x1="256.54" y1="124.46" x2="256.54" y2="129.54" width="0.1524" layer="91"/>
-<pinref part="RED" gate="G$1" pin="C"/>
-<pinref part="DA1" gate="G$1" pin="CHRG"/>
 </segment>
 </net>
 <net name="N$81" class="0">
 <segment>
-<pinref part="GREEN" gate="G$1" pin="C"/>
-<wire x1="246.38" y1="127" x2="246.38" y2="129.54" width="0.1524" layer="91"/>
 <wire x1="231.14" y1="127" x2="246.38" y2="127" width="0.1524" layer="91"/>
 <pinref part="DA1" gate="G$1" pin="STDBY"/>
-</segment>
-</net>
-<net name="N$82" class="0">
-<segment>
-<pinref part="R22" gate="G$1" pin="1"/>
-<pinref part="RED" gate="G$1" pin="A"/>
-<wire x1="256.54" y1="139.7" x2="256.54" y2="137.16" width="0.1524" layer="91"/>
-</segment>
-</net>
-<net name="N$83" class="0">
-<segment>
 <pinref part="R23" gate="G$1" pin="1"/>
-<pinref part="GREEN" gate="G$1" pin="A"/>
-<wire x1="246.38" y1="139.7" x2="246.38" y2="137.16" width="0.1524" layer="91"/>
+<wire x1="246.38" y1="129.54" x2="246.38" y2="127" width="0.1524" layer="91"/>
 </segment>
 </net>
 <net name="N$84" class="0">
 <segment>
-<pinref part="R23" gate="G$1" pin="2"/>
-<wire x1="246.38" y1="149.86" x2="246.38" y2="152.4" width="0.1524" layer="91"/>
-<pinref part="R22" gate="G$1" pin="2"/>
-<wire x1="256.54" y1="152.4" x2="256.54" y2="149.86" width="0.1524" layer="91"/>
 <wire x1="256.54" y1="152.4" x2="246.38" y2="152.4" width="0.1524" layer="91"/>
 <wire x1="246.38" y1="152.4" x2="238.76" y2="152.4" width="0.1524" layer="91"/>
@@
 <wire x1="203.2" y1="137.16" x2="238.76" y2="137.16" width="0.1524" layer="91"/>
 <junction x="238.76" y="137.16"/>
-<junction x="246.38" y="152.4"/>
 <junction x="203.2" y="129.54"/>
 <pinref part="DA1" gate="G$1" pin="VCC"/>
 <wire x1="205.74" y1="129.54" x2="203.2" y2="129.54" width="0.1524" layer="91"/>
 <pinref part="DA1" gate="G$1" pin="CE"/>
+<pinref part="GREEN" gate="G$1" pin="A"/>
+<wire x1="246.38" y1="149.86" x2="246.38" y2="152.4" width="0.1524" layer="91"/>
+<pinref part="RED" gate="G$1" pin="A"/>
+<wire x1="256.54" y1="149.86" x2="256.54" y2="152.4" width="0.1524" layer="91"/>
+<junction x="246.38" y="152.4"/>
 </segment>
 </net>
@@
 </segment>
 </net>
+<net name="N$4" class="0">
+<segment>
+<pinref part="R22" gate="G$1" pin="2"/>
+<pinref part="RED" gate="G$1" pin="C"/>
+<wire x1="256.54" y1="139.7" x2="256.54" y2="142.24" width="0.1524" layer="91"/>
+</segment>
+</net>
+<net name="N$5" class="0">
+<segment>
+<pinref part="R23" gate="G$1" pin="2"/>
+<pinref part="GREEN" gate="G$1" pin="C"/>
+<wire x1="246.38" y1="139.7" x2="246.38" y2="142.24" width="0.1524" layer="91"/>
+</segment>
+</net>
