File: HW_EAGLE/b333.sch (EAGLE design)
At the start: 153 parts, among them Q1 2N4126, Q2 2N4126, X1 USB MICRO

Commit message: .
Parts:
- U$5: device TP4056++:MOD_TP4056 -> TP4056+mod:MOD_TP4056
Connections:
- new net N$10: U$5.P2+B
- new net N$11: U$5.P2-OUT
- new net N$20: U$5.P2+OUT
- new net N$25: U$5.P1+
- new net N$9: U$5.P1-
Changed lines of the file:
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@@
 <grid distance="100" unitdist="mil" unit="mil" style="lines" multiple="1" display="yes" altdistance="0.01" altunitdist="inch" altunit="inch"/>
 <layers>
-<layer number="1" name="Top" color="4" fill="1" visible="no" active="no"/>
-<layer number="2" name="Route2" color="1" fill="3" visible="no" active="no"/>
-<layer number="3" name="Route3" color="4" fill="3" visible="no" active="no"/>
-<layer number="4" name="Route4" color="1" fill="4" visible="no" active="no"/>
-<layer number="5" name="Route5" color="4" fill="4" visible="no" active="no"/>
-<layer number="6" name="Route6" color="1" fill="8" visible="no" active="no"/>
-<layer number="7" name="Route7" color="4" fill="8" visible="no" active="no"/>
-<layer number="8" name="Route8" color="1" fill="2" visible="no" active="no"/>
-<layer number="9" name="Route9" color="4" fill="2" visible="no" active="no"/>
-<layer number="10" name="Route10" color="1" fill="7" visible="no" active="no"/>
-<layer number="11" name="Route11" color="4" fill="7" visible="no" active="no"/>
-<layer number="12" name="Route12" color="1" fill="5" visible="no" active="no"/>
-<layer number="13" name="Route13" color="4" fill="5" visible="no" active="no"/>
-<layer number="14" name="Route14" color="1" fill="6" visible="no" active="no"/>
-<layer number="15" name="Route15" color="4" fill="6" visible="no" active="no"/>
-<layer number="16" name="Bottom" color="1" fill="1" visible="no" active="no"/>
-<layer number="17" name="Pads" color="2" fill="1" visible="no" active="no"/>
-<layer number="18" name="Vias" color="2" fill="1" visible="no" active="no"/>
-<layer number="19" name="Unrouted" color="6" fill="1" visible="no" active="no"/>
-<layer number="20" name="Dimension" color="15" fill="1" visible="no" active="no"/>
-<layer number="21" name="tPlace" color="6" fill="1" visible="no" active="no"/>
-<layer number="22" name="bPlace" color="7" fill="1" visible="no" active="no"/>
-<layer number="23" name="tOrigins" color="15" fill="1" visible="no" active="no"/>
-<layer number="24" name="bOrigins" color="15" fill="1" visible="no" active="no"/>
-<layer number="25" name="tNames" color="6" fill="1" visible="no" active="no"/>
-<layer number="26" name="bNames" color="7" fill="1" visible="no" active="no"/>
-<layer number="27" name="tValues" color="7" fill="1" visible="no" active="no"/>
-<layer number="28" name="bValues" color="7" fill="1" visible="no" active="no"/>
+<layer number="1" name="Top" color="4" fill="1" visible="yes" active="no"/>
+<layer number="2" name="Route2" color="1" fill="3" visible="yes" active="no"/>
+<layer number="3" name="Route3" color="4" fill="3" visible="yes" active="no"/>
+<layer number="4" name="Route4" color="1" fill="4" visible="yes" active="no"/>
+<layer number="5" name="Route5" color="4" fill="4" visible="yes" active="no"/>
+<layer number="6" name="Route6" color="1" fill="8" visible="yes" active="no"/>
+<layer number="7" name="Route7" color="4" fill="8" visible="yes" active="no"/>
+<layer number="8" name="Route8" color="1" fill="2" visible="yes" active="no"/>
+<layer number="9" name="Route9" color="4" fill="2" visible="yes" active="no"/>
+<layer number="10" name="Route10" color="1" fill="7" visible="yes" active="no"/>
+<layer number="11" name="Route11" color="4" fill="7" visible="yes" active="no"/>
+<layer number="12" name="Route12" color="1" fill="5" visible="yes" active="no"/>
+<layer number="13" name="Route13" color="4" fill="5" visible="yes" active="no"/>
+<layer number="14" name="Route14" color="1" fill="6" visible="yes" active="no"/>
+<layer number="15" name="Route15" color="4" fill="6" visible="yes" active="no"/>
+<layer number="16" name="Bottom" color="1" fill="1" visible="yes" active="no"/>
+<layer number="17" name="Pads" color="2" fill="1" visible="yes" active="no"/>
+<layer number="18" name="Vias" color="2" fill="1" visible="yes" active="no"/>
+<layer number="19" name="Unrouted" color="6" fill="1" visible="yes" active="no"/>
+<layer number="20" name="Dimension" color="15" fill="1" visible="yes" active="no"/>
+<layer number="21" name="tPlace" color="6" fill="1" visible="yes" active="no"/>
+<layer number="22" name="bPlace" color="7" fill="1" visible="yes" active="no"/>
+<layer number="23" name="tOrigins" color="15" fill="1" visible="yes" active="no"/>
+<layer number="24" name="bOrigins" color="15" fill="1" visible="yes" active="no"/>
+<layer number="25" name="tNames" color="6" fill="1" visible="yes" active="no"/>
+<layer number="26" name="bNames" color="7" fill="1" visible="yes" active="no"/>
+<layer number="27" name="tValues" color="7" fill="1" visible="yes" active="no"/>
+<layer number="28" name="bValues" color="7" fill="1" visible="yes" active="no"/>
 <layer number="29" name="tStop" color="7" fill="3" visible="no" active="no"/>
 <layer number="30" name="bStop" color="7" fill="6" visible="no" active="no"/>
@@
 <layer number="35" name="tGlue" color="7" fill="4" visible="no" active="no"/>
 <layer number="36" name="bGlue" color="7" fill="5" visible="no" active="no"/>
-<layer number="37" name="tTest" color="7" fill="1" visible="no" active="no"/>
-<layer number="38" name="bTest" color="7" fill="1" visible="no" active="no"/>
+<layer number="37" name="tTest" color="7" fill="1" visible="yes" active="no"/>
+<layer number="38" name="bTest" color="7" fill="1" visible="yes" active="no"/>
 <layer number="39" name="tKeepout" color="4" fill="11" visible="no" active="no"/>
 <layer number="40" name="bKeepout" color="1" fill="11" visible="no" active="no"/>
@@
 <layer number="44" name="Drills" color="7" fill="1" visible="no" active="no"/>
 <layer number="45" name="Holes" color="7" fill="1" visible="no" active="no"/>
-<layer number="46" name="Milling" color="3" fill="1" visible="no" active="no"/>
-<layer number="47" name="Measures" color="14" fill="1" visible="no" active="no"/>
-<layer number="48" name="Document" color="7" fill="1" visible="no" active="no"/>
-<layer number="49" name="Reference" color="7" fill="1" visible="no" active="no"/>
-<layer number="50" name="dxf" color="7" fill="1" visible="no" active="no"/>
-<layer number="51" name="tDocu" color="7" fill="1" visible="no" active="no"/>
-<layer number="52" name="bDocu" color="7" fill="1" visible="no" active="no"/>
-<layer number="53" name="tGND_GNDA" color="7" fill="9" visible="no" active="no"/>
-<layer number="54" name="bGND_GNDA" color="1" fill="9" visible="no" active="no"/>
-<layer number="56" name="wert" color="7" fill="1" visible="no" active="no"/>
-<layer number="57" name="tCAD" color="7" fill="1" visible="no" active="no"/>
+<layer number="46" name="Milling" color="3" fill="1" visible="yes" active="no"/>
+<layer number="47" name="Measures" color="14" fill="1" visible="yes" active="no"/>
+<layer number="48" name="Document" color="7" fill="1" visible="yes" active="no"/>
+<layer number="49" name="Reference" color="7" fill="1" visible="yes" active="no"/>
+<layer number="50" name="dxf" color="7" fill="1" visible="yes" active="no"/>
+<layer number="51" name="tDocu" color="7" fill="1" visible="yes" active="no"/>
+<layer number="52" name="bDocu" color="7" fill="1" visible="yes" active="no"/>
+<layer number="53" name="tGND_GNDA" color="7" fill="9" visible="yes" active="no"/>
+<layer number="54" name="bGND_GNDA" color="1" fill="9" visible="yes" active="no"/>
+<layer number="56" name="wert" color="7" fill="1" visible="yes" active="no"/>
+<layer number="57" name="tCAD" color="7" fill="1" visible="yes" active="no"/>
 <layer number="90" name="Modules" color="5" fill="1" visible="yes" active="yes"/>
 <layer number="91" name="Nets" color="2" fill="1" visible="yes" active="yes"/>
@@
 <part name="GND15" library="supply1" deviceset="GND" device=""/>
 <part name="GND17" library="supply1" deviceset="GND" device=""/>
-<part name="U$5" library="TP4056++" deviceset="MOD_TP4056" device=""/>
+<part name="U$5" library="TP4056+mod" deviceset="MOD_TP4056" device=""/>
 </parts>
 <sheets>
@@
 </segment>
 </net>
+<net name="N$9" class="0">
+<segment>
+<pinref part="U$5" gate="G$1" pin="P1-"/>
+<wire x1="25.4" y1="91.44" x2="25.4" y2="88.9" width="0.1524" layer="91"/>
+<junction x="25.4" y="88.9"/>
+</segment>
+</net>
+<net name="N$11" class="0">
+<segment>
+<pinref part="U$5" gate="G$1" pin="P2-OUT"/>
+<wire x1="35.56" y1="96.52" x2="35.56" y2="88.9" width="0.1524" layer="91"/>
+<junction x="35.56" y="88.9"/>
+</segment>
+</net>
+<net name="N$18" class="0">
+<segment>
+<wire x1="25.4" y1="86.36" x2="35.56" y2="86.36" width="0.1524" layer="91"/>
+<junction x="25.4" y="86.36"/>
+<junction x="35.56" y="86.36"/>
+</segment>
+</net>
+<net name="N$10" class="0">
+<segment>
+<pinref part="U$5" gate="G$1" pin="P2+B"/>
+<wire x1="35.56" y1="104.14" x2="38.1" y2="104.14" width="0.1524" layer="91"/>
+<junction x="38.1" y="104.14"/>
+</segment>
+</net>
+<net name="N$20" class="0">
+<segment>
+<pinref part="U$5" gate="G$1" pin="P2+OUT"/>
+<wire x1="35.56" y1="106.68" x2="38.1" y2="106.68" width="0.1524" layer="91"/>
+<junction x="38.1" y="106.68"/>
+</segment>
+</net>
+<net name="N$25" class="0">
+<segment>
+<pinref part="U$5" gate="G$1" pin="P1+"/>
+<wire x1="25.4" y1="111.76" x2="38.1" y2="111.76" width="0.1524" layer="91"/>
+<junction x="38.1" y="111.76"/>
+</segment>
+</net>
+<net name="N$26" class="0">
+<segment>
+<wire x1="40.64" y1="111.76" x2="40.64" y2="106.68" width="0.1524" layer="91"/>
+<junction x="40.64" y="104.14"/>
+<junction x="40.64" y="106.68"/>
+<wire x1="40.64" y1="106.68" x2="40.64" y2="104.14" width="0.1524" layer="91"/>
+<junction x="40.64" y="111.76"/>
+</segment>
+</net>

Commit message: .
Connections:
- new net N$27: U$5.P2-B
Changed lines of the file:
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@@
+</segment>
+</net>
+<net name="N$27" class="0">
+<segment>
+<pinref part="U$5" gate="G$1" pin="P2-B"/>
+<wire x1="35.56" y1="99.06" x2="38.1" y2="99.06" width="0.1524" layer="91"/>
+<junction x="38.1" y="99.06"/>
+</segment>
+</net>
+<net name="N$28" class="0">
+<segment>
+<wire x1="40.64" y1="99.06" x2="43.18" y2="99.06" width="0.1524" layer="91"/>
+<junction x="40.64" y="99.06"/>
 </segment>
 </net>

Commit message: .
Parts:
- added S1: 9077-2, switch-misc:9077-2
- 6R15: device resistor:R-EU_R0805 -> resistor:R-EU_R1206W
Changed lines of the file:
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@@
 <part name="6VT2" library="DSS" deviceset="NMOS" device="D"/>
 <part name="U$27" library="lib-user" deviceset="GND" device=""/>
-<part name="6R15" library="resistor" deviceset="R-EU_" device="R0805" value="100k"/>
+<part name="6R15" library="resistor" deviceset="R-EU_" device="R1206W" value="100k"/>
 <part name="6R1B" library="resistor" deviceset="R-EU_" device="R1206" value="1R"/>
 <part name="SUPPLY1" library="supply2" deviceset="V+" device=""/>
@@
 <part name="GND17" library="supply1" deviceset="GND" device=""/>
 <part name="U$5" library="TP4056+mod" deviceset="MOD_TP4056" device=""/>
+<part name="S1" library="switch-misc" deviceset="9077-2" device=""/>
 </parts>
 <sheets>
@@
 <instance part="GND17" gate="1" x="218.44" y="111.76" rot="MR0"/>
 <instance part="U$5" gate="G$1" x="25.4" y="101.6"/>
+<instance part="S1" gate="1" x="30.48" y="66.04" rot="R270"/>
+<instance part="S1" gate="2" x="30.48" y="55.88" rot="R270"/>
 </instances>
 <busses>

Commit message: pp pin
Parts:
- added BS1, BS2, D0, D1, D2, D4, D5, D6, OE, PAGEL, R/B, WR, XA0, XA1, XTAL1: (no value), pinhead:PINHD-1X1
- added VD3, VD7: 1N4148DO35-7, diode:1N4148DO35-7
- D3, D7: value 1N4148DO35-7 -> (none); device diode:1N4148DO35-7 -> pinhead:PINHD-1X1
Connections:
- net +2V5 renamed PC4
- net N$87 renamed PD0
- net U_BAT renamed PC5
- removed net E1: DD1.PD5(T1/OC0B/PCINT21), JP3.6
- removed net N$62: DD1.PD3(INT1/OC2B/PCINT19), JP3.14
- removed net N$68: 1C8.2, 1Z2.2, DD1.PB6(XTAL1/TOSC1/PCINT6)
- removed net N$88: DD1.PD1(TXD/PCINT17), JP3.12
- removed net N$89: DD1.PD2(INT0/PCINT18), JP3.13
- removed net PB3: 1R19.1, DD1.PB0(ICP1/CLKO/PCINT0)
- removed net PB4: 1R20.1, DD1.PB1(OC1A/PCINT1)
- removed net PB5: 1R21.1, DD1.PB2(SS/OC1B/PCINT2)
- new net ADC6: DD1.ADC6
- new net ADC7: DD1.ADC7
- new net PB0: 1R19.1, D0.1, DD1.PB0(ICP1/CLKO/PCINT0)
- new net PB1: 1R20.1, D1.1, DD1.PB1(OC1A/PCINT1)
- new net PB2: 1R21.1, D2.1, DD1.PB2(SS/OC1B/PCINT2)
- new net PB6: 1C8.2, 1Z2.2, DD1.PB6(XTAL1/TOSC1/PCINT6), XTAL1.1
- new net PD5: DD1.PD5(T1/OC0B/PCINT21), JP3.6, XA0.1
- new net PD6: DD1.PD6(AIN0/OC0A/PCINT22), XA1.1
- new net PD7: 1R18.2, C17.1, DD1.PD7(AIN1/PCINT23), PAGEL.1
- net FO: now also VD3.C; no longer D3.C
- net N$100: now also VD3.A, VD7.A; no longer D3.A, D7.A
- net N$102: now also VD7.C; no longer D7.C
- net PD1: now also DD1.PD1(TXD/PCINT17), JP3.12, R/B.1; no longer 1R18.2, C17.1, DD1.PD7(AIN1/PCINT23)
- net PD2: now also DD1.PD2(INT0/PCINT18), JP3.13, OE.1; no longer DD1.PD6(AIN0/OC0A/PCINT22)
- net PD3: now also DD1.PD3(INT1/OC2B/PCINT19), JP3.14, WR.1
- net PD4: now also BS1.1

Commit message: .
Connections:
- net PD4: no longer BS1.1
- net PD4MC: now also BS1.1
Changed lines of the file:
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@@
 <wire x1="248.92" y1="127" x2="246.38" y2="127" width="0.1524" layer="91"/>
-</segment>
-<segment>
-<pinref part="BS1" gate="G$1" pin="1"/>
-<wire x1="267.97" y1="64.77" x2="255.27" y2="64.77" width="0.1524" layer="91"/>
-<label x="255.27" y="64.77" size="1.778" layer="95"/>
 </segment>
 </net>
@@
 <wire x1="137.16" y1="91.44" x2="134.62" y2="91.44" width="0.1524" layer="91"/>
 </segment>
-</net>
+<segment>
+<pinref part="BS1" gate="G$1" pin="1"/>
+<wire x1="267.97" y1="64.77" x2="255.27" y2="64.77" width="0.1524" layer="91"/>
+<label x="255.27" y="64.77" size="1.778" layer="95"/>
+</segment>
+</net>
