File: HW_EAGLE/b333.brd (EAGLE design)
At the start: 150 parts, among them Q1 2N4126, Q2 2N4126, X1 USB MICRO, X2 USB MICRO

Commit message: .
Parts:
- added JP3: (no value), b333:1X16-8
- 2L2: device ct-pack:LH7X10MM -> ct-pack:LV7X10MM
- 2L4: device rcl:6000-XXXX-RC -> ct-pack:LV7X10MM
- 5MA: device jumper:JP2 -> ct-pack:JP2
- DIS1: value TUXGR_16X2_R2 -> LCD_16X2_R2; device b333:TUXGR_16X2_R2 -> b333:LCD_16X2_R2
- moved C10 319.9 mm to (128.0, 12.7)
- moved 4R7 303.5 mm to (167.6, 27.0)
- moved 1R18 303.5 mm to (104.8, 25.7)
- moved 4R6 303.5 mm to (152.4, 25.7)
- moved C17 303.5 mm to (152.1, 22.9)
- moved DA6 75.1 mm to (205.4, 22.9), turned to 90 degrees
- moved J_ONE5V 47.3 mm to (220.3, 13.7), turned to 90 degrees
- moved 4Y4 41.3 mm to (207.3, 58.4), turned to 180 degrees
- moved 4Y3 14.4 mm to (173.4, 57.8), turned to 180 degrees
- moved 2L4 10.2 mm to (228.3, 84.8)
- moved 6C6 9.51 mm to (218.4, 80.6), turned to 270 degrees
- moved 6C5 9.38 mm to (214.0, 80.6), flipped to the top, turned to 90 degrees
- moved C4 6.70 mm to (261.9, 21.3)
- moved 2L2 5.97 mm to (254.6, 22.2)
- moved 3C12 5.41 mm to (275.3, 9.84), turned to 270 degrees
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Routing:
- net GND: track 268.5 -> 291.6 mm
- net N$19: track 19.8 -> 40.1 mm
- net +90.5V: track 8.30 -> 23.3 mm
- net N$14: track 21.6 -> 8.86 mm
- net N$13: track 20.7 -> 11.1 mm
- net V+: track 57.7 -> 62.5 mm
- net N$17: track 19.7 -> 17.0 mm

Commit message: rtrim
Parts:
- added 1C3: 100n, resistor:C0805K
- added 1R4, 1R5, 1R6: 10k, resistor:R0805
- added R2: 10k, ct-pack:RTRIM3296W
- R35: device rcl:RTRIM3296W -> ct-pack:RTRIM3296W
- moved 4Y4 42.6 mm to (166.4, 46.7)
- moved 4Y3 34.1 mm to (205.1, 45.4)
- moved JP2 6.35 mm to (77.8, 97.8)
Connections:
- net N$4 renamed PD4MC
- removed net N$72: 4R7.2, 4Y4.P
- removed net N$97: C19.1, D12.C, JP2.1, R14.2, R17.2, R28.2, R9.2
- new net FO: 1R6.2, D3.C, R27.2, R28.1, T9.C
- new net N$1: 4Y4.O, 4Y4.P, 4Y4.S
- new net N$2: C19.1, D12.C, JP2.1, R14.2, R17.2, R2.3, R28.2, R9.2
- new net N$6: 1R5.2, R2.1, R2.2
- new net N$7: 1C3.1, 1R6.1
- new net PD3: 1C3.2, 1R4.2, 1R5.1
- net GND: now also 1R4.1
- net PD4: no longer D3.C, R27.2, R28.1, T9.C
- net T2: no longer 4Y4.O
Routing:
- net PD4: track 71.0 -> 36.7 mm
- net N$2: track 0.00 -> 28.1 mm
- net GND: track 291.6 -> 268.4 mm
- net N$97: track 21.7 -> 0.00 mm
- net FO: track 0.00 -> 12.5 mm
- net N$6: track 0.00 -> 4.57 mm
- net PD3: track 0.00 -> 4.02 mm
- net N$7: track 0.00 -> 2.14 mm

Commit message: .
Parts:
- 1C2: value 220u/6V -> 330u/6V
- 2L2: value 100uH -> 30uH
- 2L3: value 220uH -> 330uH
- moved DA6 179.8 mm to (319.7, 161.6), flipped to the bottom
- moved J_NO_LI 172.0 mm to (313.4, 167.3), flipped to the bottom
- moved DA4A 171.6 mm to (313.1, 163.5), flipped to the bottom
- moved C8 167.6 mm to (309.6, 167.3), flipped to the bottom
- moved DA4 165.5 mm to (307.7, 161.6), flipped to the bottom
- moved 3C11 164.1 mm to (306.4, 165.4)
- moved J_ONE5V 162.4 mm to (304.8, 152.4), flipped to the bottom
- moved C7 151.8 mm to (293.4, 159.7), flipped to the bottom
- moved 2L3 148.9 mm to (289.6, 164.1)
- moved 1C5 146.5 mm to (286.1, 154.3)
- moved 2R8 144.6 mm to (282.9, 159.7), flipped to the bottom
- moved C5 143.7 mm to (281.3, 163.5), flipped to the bottom
- moved 1C2 143.6 mm to (281.0, 166.1)
- moved C18 143.4 mm to (244.5, 147.6), flipped to the bottom
- moved 2R7 143.2 mm to (280.4, 159.1), flipped to the bottom
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Routing:
- net N$17: track 17.0 -> 21.9 mm, vias 0 -> 1
- net GND: track 268.4 -> 271.8 mm
- net +5V: track 46.5 -> 47.5 mm, vias 0 -> 1
- net V+: vias 0 -> 1

Commit message: .
Parts:
- added C1: 100n, resistor:C0805K
- 2L2: device ct-pack:LV7X10MM -> ct-pack:LH7X10MM
- moved DA6 126.8 mm to (204.8, 108.0), flipped to the top
- moved 2R7 109.6 mm to (198.1, 86.7), turned to 0 degrees
- moved 2R8 107.8 mm to (203.8, 86.4), turned to 180 degrees
- moved C5 101.8 mm to (206.4, 94.6), turned to 90 degrees
- moved 1C2 100.8 mm to (209.9, 94.6), turned to 90 degrees
- moved 1R26 98.3 mm to (197.8, 106.7), turned to 0 degrees
- moved 2R1 96.5 mm to (197.2, 97.5)
- moved 2R6 96.5 mm to (197.2, 99.7)
- moved DA3 95.4 mm to (203.2, 99.4), turned to 270 degrees
- moved 2C1 95.0 mm to (208.9, 99.4), turned to 90 degrees
- moved 2D2 94.6 mm to (212.4, 99.7), turned to 90 degrees
- moved C4 92.7 mm to (202.2, 90.2), turned to 270 degrees
- moved 2L2 91.6 mm to (203.8, 98.1), turned to 180 degrees
- moved C6 90.5 mm to (203.5, 95.6), turned to 180 degrees
- moved 2R5 90.4 mm to (199.4, 103.2), turned to 270 degrees
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Connections:
- net +5V/2: now also 6VT3.E
- net GND: no longer 6C1.-
- net N$12: now also C1.2
- net N$13: now also 2L2.1; no longer 2L2.2
- net N$14: now also 2L2.2; no longer 2L2.1
- net V+: now also C1.1; no longer 6C1.+, 6VT3.E
Routing:
- net E1: track 61.1 -> 27.5 mm
- net PD4: track 36.7 -> 12.3 mm
- net N$16: track 1.96 -> 18.2 mm
- net GND: track 271.8 -> 258.9 mm
- net N$89: track 14.8 -> 3.62 mm
- net N$88: track 14.9 -> 3.90 mm
- net N$87: track 16.1 -> 5.32 mm
- net N$62: track 18.1 -> 9.47 mm
- net N$14: track 8.86 -> 17.2 mm
- net +5V: track 47.5 -> 40.4 mm
- net N$12: track 16.4 -> 21.0 mm
- net +5V/2: track 0.00 -> 3.67 mm
- net N$95: track 3.41 -> 0.00 mm
- net N$17: track 21.9 -> 18.6 mm, vias 1 -> 0
- net Z_BLUE: track 20.1 -> 21.8 mm
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
Commit message: .
Parts:
- removed C1: 100n, resistor:C0805K
- added 6C1A: 100u, resistor:E2,5-6
- added D1: (no value), diode:SOD80C
- 6C1: value 100u -> 100n; device resistor:E2,5-6 -> resistor:C0805K
- 6C5: device resistor:E2,5-6 -> ct-pack:E2,5-6
- moved 4Y3 38.9 mm to (173.7, 22.5)
- moved 6C1 36.3 mm to (222.6, 104.1), flipped to the bottom, turned to 0 degrees
- moved 6R9 12.5 mm to (226.7, 66.4), turned to 90 degrees
- moved ZEN_K1 11.5 mm to (224.2, 65.7), flipped to the top, turned to 180 degrees
- moved 6R12 10.3 mm to (216.5, 69.5), turned to 270 degrees
- moved ZEN_A1 9.16 mm to (211.5, 65.7), flipped to the top, turned to 180 degrees
- moved 6C6 8.67 mm to (209.9, 79.4)
- moved 6VD4 7.81 mm to (229.2, 71.1)
- moved 6R8 6.87 mm to (223.2, 79.4)
- moved VT6 6.55 mm to (224.2, 70.2), turned to 180 degrees
- moved 6R6 5.85 mm to (218.1, 79.4)
- moved 6C7 5.84 mm to (213.7, 69.8), turned to 90 degrees
- moved 6VD3 5.72 mm to (227.6, 74.9), turned to 0 degrees
- moved 6VD2 4.13 mm to (225.7, 79.1)
- moved 5MA 3.86 mm to (220.7, 74.9), flipped to the top
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Connections:
- net ZENER_A renamed ZENER
- net GND: now also D1.A
- net N$12: now also 6C1.2; no longer C1.2
- net PC3: now also D1.C
- net V+: now also 6C1.1; no longer C1.1
Routing:
- net GND: track 258.9 -> 301.9 mm
- net ZENER: track 33.2 -> 70.5 mm
- net PC3: track 0.00 -> 8.13 mm
- net +90.5V: track 23.7 -> 31.8 mm
- net N$67: track 9.83 -> 6.14 mm
- net N$22: track 8.02 -> 5.02 mm
- net N$19: track 40.3 -> 42.2 mm
- net Z_GREEN: track 2.82 -> 4.65 mm
- net N$24: track 0.00 -> 1.79 mm
- net 1MA: track 7.09 -> 8.45 mm
- net N$52: track 3.95 -> 2.64 mm
- net V+: track 61.3 -> 60.2 mm
- net N$17: track 18.6 -> 19.2 mm
- net N$96: track 4.90 -> 5.53 mm
- net N$12: track 21.0 -> 20.5 mm
Other:
- board outline added: 80 x 50.5 mm

Commit message: .
Parts:
- 2R1, 2R6: device resistor:R0805 -> resistor:R1206
- moved 2L3 121.5 mm to (173.0, 93.0)
- moved 3C11 121.5 mm to (183.2, 80.0)
- moved C7 121.5 mm to (179.4, 88.9)
- moved DA4 121.5 mm to (180.0, 84.5)
- moved J_ONE5V 121.5 mm to (184.8, 99.7)
- moved 1C5 121.5 mm to (179.7, 92.1)
- moved C8 121.5 mm to (178.1, 78.7)
- moved DA4A 121.5 mm to (174.6, 82.5)
- moved J_NO_LI 121.5 mm to (174.3, 78.7)
- moved DIS1 104.5 mm to (296.2, 96.8)
- moved 3C12 54.8 mm to (200.7, 124.5), turned to 0 degrees
- moved C18 51.5 mm to (201.6, 119.1), turned to 180 degrees
- moved 1C2 20.0 mm to (190.2, 98.1)
- moved C4 3.18 mm to (199.1, 90.2)
- moved 2R1 3.18 mm to (195.3, 100.0), turned to 90 degrees
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Routing:
- net N$17: track 19.2 -> 7.25 mm
- net GND: track 301.9 -> 299.1 mm
- net N$14: track 17.2 -> 15.3 mm
- net V+: track 60.2 -> 58.8 mm

Commit message: .
Parts:
- removed D1: (no value), diode:SOD80C
- added Z1: 5v6, diode:SOD80C
- moved DIS1 104.5 mm to (191.8, 94.6)
- moved 6R9 16.0 mm to (213.4, 75.2), turned to 180 degrees
- moved 6VD4 13.5 mm to (218.1, 78.7)
- moved 6VD3 7.96 mm to (220.7, 78.7), turned to 270 degrees
- moved 6R6 7.94 mm to (224.5, 74.6), turned to 0 degrees
- moved 6R8 7.75 mm to (229.6, 74.9)
- moved 6R7 7.75 mm to (227.0, 74.9)
- moved 5MA 7.41 mm to (227.0, 71.1)
- moved VT6 6.43 mm to (218.8, 73.7), turned to 0 degrees
- moved 6R11 4.26 mm to (216.9, 69.5), turned to 270 degrees
- moved 6C7 3.18 mm to (210.5, 69.8), turned to 270 degrees
- moved 6VD2 2.56 mm to (223.2, 78.7)
- moved ZEN_K1 2.54 mm to (221.6, 65.7)
- moved 6R12 1.59 mm to (214.9, 69.5), turned to 90 degrees
Connections:
- net GND: now also Z1.A; no longer D1.A
- net PC3: now also DD1.26, Z1.C; no longer D1.C
- net ZENER: no longer DD1.26
Routing:
- net ZENER: track 70.5 -> 11.4 mm, vias 1 -> 0
- net +90.5V: track 31.8 -> 44.4 mm
- net PC3: track 8.13 -> 16.2 mm, vias 0 -> 1
- net 1MA: track 8.45 -> 15.4 mm
- net GND: track 299.1 -> 292.8 mm
- net N$24: track 1.79 -> 3.05 mm
- net N$55: track 3.59 -> 2.96 mm

Commit message: .
Parts:
- removed 1C2: 330u/6V, resistor:E2-5
- removed 1C5: 1000u/6V, resistor:E2-5
- removed 2C1: 150, resistor:C0805K
- removed 2R1, 2R6: 1R, resistor:R1206
- removed 2R5: 180R, resistor:R0805
- removed 2R7: 3.9k, resistor:R0805
- removed 2R8: 18k, resistor:R0805
- removed 3C11, 3C12: 47u, resistor:E2,5-6
- removed 6C1A: 100u, resistor:E2,5-6
- removed B+OUT+, B-1, GND: B-, TP4056_18650:PAD-
- removed C18, C5, C6, C7, C8: 100n, resistor:C0805K
- removed C4: 50u, resistor:E2,5-6
- removed H2: LCD, pinhead:1X16
- removed TEST2: TT-P, transistor_tester:TT-P
- removed VT3: FS8205A, FS8205A:TSSOP-8
- removed X2: USB MICRO, SmartPrj:CON2_USB_MICRO_B_AT
- added 5C1, 5C10, 5C4, 5C6, 5C8: 100n, resistor:C0805K
- added 5C2: 150, resistor:C0805K
- added 5C3: 330u/6V, resistor:E2-5
- added 5C5: 1000u/6V, resistor:E2-5
- added 5C7, 5C9: 47u, resistor:E2,5-6
- added 5R1, 5R1B: 1R, resistor:R1206
- added 5R2: 180R, resistor:R0805
- added 5R3: 3.9k, resistor:R0805
- added 5R4: 18k, resistor:R0805
- added B+, B-: B-, TP4056_18650:PAD-
- added C1: 50u, resistor:E2,5-6
- added H1: LCD, pinhead:1X16
- added TEST: TT-P, transistor_tester:TT-P
- DA2: device DW01:SOT23-6 -> TP4056+:SOT23-6
- VT2: device FS8205A:TSSOP-8 -> TP4056+:TSSOP-8
- ZEN_A1, ZEN_K1: device pinhead:1X01 -> pinhead:1X02
- moved DA4 77.2 mm to (129.2, 142.6)
- moved J_NO_LI 77.2 mm to (123.5, 136.8)
- moved DA4A 77.2 mm to (123.8, 140.7)
- moved 4Y4 62.6 mm to (103.8, 43.8)
- moved C12 61.3 mm to (76.5, 92.7)
- moved 6R10 58.4 mm to (160.0, 65.1), turned to 270 degrees
- moved R20 58.1 mm to (64.1, 92.1)
- moved ZEN_K1 57.8 mm to (163.8, 64.8)
- moved R23 57.5 mm to (80.6, 98.1)
- moved R22 57.5 mm to (80.6, 96.2)
- moved 2D2 57.2 mm to (155.3, 98.4)
- moved 6VT3 57.2 mm to (153.0, 107.6)
- moved C11 57.2 mm to (70.2, 83.8)
- moved 6C7 56.8 mm to (153.7, 69.5)
- moved Z1 56.8 mm to (156.2, 69.8)
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Connections:
- removed net +3V7: B+OUT+.B-, C13.1, DA1.5, R21.2
- removed net UGND: C12.2, C13.2, DA1.., DA1.1, DA1.3, R20.1, R24.1, VT2.6, VT2.7, X1.P5, X1.S1, X1.S2, X1.S3, X1.S4, X1.S5, X1.S6
- removed net VBUS: X2.P1
- net +5V: now also 5C7.+, 5C8.1; no longer 3C11.+, C8.1
- net +5V/2: now also 5C10.1, 5C9.+, JP3.2; no longer 3C12.+, C18.1, H2.2
- net +7V: now also 5C5.+, 5C6.1; no longer 1C5.+, C7.1
- net B-: now also B-.B-; no longer B-1.B-
- net E1: now also JP3.6; no longer H2.6
- net GND: now also 5C1.2, 5C10.2, 5C2.2, 5C3.-, 5C4.2, 5C5.-, 5C6.2, 5C7.-, 5C8.2, 5C9.-, 5R3.1, C1.-, C12.2, C13.2, DA1.., DA1.1, DA1.3, JP3.1, JP3.16, JP3.5, R20.1, R24.1, VT2.6, VT2.7, X1.P5, X1.S1, X1.S2, X1.S3, X1.S4, X1.S5, X1.S6, ZEN_A1.2; no longer 1C2.-, 1C5.-, 2C1.2, 2R7.1, 3C11.-, 3C12.-, C18.2, C4.-, C5.2, C6.2, C7.2, C8.2, GND.B-, H2.1, H2.10, H2.16, H2.5, H2.7, H2.8, H2.9
- net N$14: now also 5R1.2, 5R1B.2, 5R2.1; no longer 2R1.2, 2R5.1, 2R6.2
- net N$15: now also 5R2.2; no longer 2R5.2
- net N$16: now also 5R3.2, 5R4.1; no longer 2R7.2, 2R8.1
- net N$17: now also 5C3.+, 5C4.1, 5R4.2; no longer 1C2.+, 2R8.2, C5.1
- net N$60: now also JP3.3; no longer H2.3
- net N$61: now also JP3.15; no longer H2.15
- net N$62: now also JP3.14; no longer H2.14
- net N$8: now also 5C2.1; no longer 2C1.1
- net N$87: now also JP3.11; no longer H2.11
- net N$88: now also JP3.12; no longer H2.12
- net N$89: now also JP3.13; no longer H2.13
- net PD4: now also JP3.4; no longer H2.4
- net V+: now also 5C1.1, 5R1.1, 5R1B.1, B+.B-, C1.+, C13.1, DA1.5, R21.2; no longer 2R1.1, 2R6.1, C4.+, C6.1
- net ZENER: now also ZEN_K1.2
Routing:
- net UGND: track 61.5 -> 0.00 mm
- net GND: track 292.8 -> 338.0 mm
- net +3V7: track 24.1 -> 0.00 mm, vias 2 -> 0
- net PC3: track 16.2 -> 34.9 mm
- net V+: track 58.8 -> 77.4 mm, vias 2 -> 4
- net N$16: track 18.2 -> 0.00 mm
- net N$62: track 9.47 -> 24.6 mm
- net N$89: track 3.62 -> 17.8 mm
- net N$88: track 3.90 -> 16.2 mm
- net PD4: track 12.3 -> 1.14 mm, vias 2 -> 1
- net N$17: track 7.25 -> 18.0 mm
- net N$87: track 5.32 -> 13.7 mm
- net N$77: track 32.0 -> 24.1 mm
- net B-: track 26.7 -> 19.3 mm
- net N$3: track 0.00 -> 6.24 mm
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