File: HW_EAGLE/b333.brd (EAGLE design)
At the start: 80 x 50.5 mm, 154 parts, among them Q1 2N4126, Q2 2N4126, X1 USB MICRO

Commit message: .
Parts:
- removed TEST1: TT-P, transistor_tester:TT-P
Connections:
- net T1: no longer TEST1.P$5
- net T2: no longer TEST1.P$2, TEST1.P$3, TEST1.P$4
- net T3: no longer TEST1.P$1
Routing:
- net T1: track 26.7 -> 23.6 mm
- net T2: track 26.1 -> 23.4 mm
- net T3: track 27.7 -> 25.2 mm
Changed lines of the file:
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@@
 <element name="C17" library="resistor" package="C0805K" value="100n" x="106.3625" y="34.29"/>
 <element name="1R26" library="resistor" package="R1206W" value="270" x="141.2875" y="105.7275"/>
-<element name="TEST1" library="transistor_tester" package="TT-P" value="TT-P" x="116.205" y="69.215"/>
 <element name="ISP" library="con-lstb" package="MA03-2" value="" x="127.9525" y="75.8825" rot="R270"/>
 <element name="DA6" library="ct-pack" package="SOT89R" value="78L05" x="148.2725" y="106.9975" rot="R90"/>
@@
 <via x="109.5375" y="89.8525" extent="1-16" drill="0.6" shape="square"/>
 <wire x1="109.5375" y1="89.8525" x2="111.94781875" y2="90.1242125" width="0.3048" layer="16"/>
-<contactref element="TEST1" pad="P$5"/>
-<wire x1="118.745" y1="76.2" x2="121.285" y2="74.295" width="0.3048" layer="16"/>
 <wire x1="118.745" y1="76.2" x2="112.395" y2="82.55" width="0.3048" layer="1"/>
 <wire x1="112.395" y1="82.55" x2="109.5375" y2="89.8525" width="0.3048" layer="1"/>
-<wire x1="121.285" y1="64.77" x2="121.285" y2="74.295" width="0" layer="19" extent="1-1"/>
+<wire x1="121.285" y1="64.77" x2="118.745" y2="76.2" width="0" layer="19" extent="16-16"/>
 <wire x1="110.275" y1="26.035" x2="121.285" y2="64.77" width="0" layer="19" extent="1-1"/>
 <wire x1="111.2275" y1="20.32" x2="110.275" y2="26.035" width="0" layer="19" extent="1-1"/>
@@
 <contactref element="1R22" pad="2"/>
 <contactref element="1R21" pad="2"/>
-<contactref element="TEST1" pad="P$3"/>
-<contactref element="TEST1" pad="P$4"/>
-<contactref element="TEST1" pad="P$2"/>
 <wire x1="117.475" y1="78.425" x2="115.2525" y2="78.425" width="0.3048" layer="16"/>
 <wire x1="115.2525" y1="78.425" x2="115.2525" y2="76.835" width="0.3048" layer="16"/>
@@
 <via x="107.95" y="90.4875" extent="1-16" drill="0.6" shape="square"/>
 <wire x1="107.95" y1="90.4875" x2="111.8089" y2="90.912059375" width="0.3048" layer="16"/>
-<wire x1="115.2525" y1="76.835" x2="116.205" y2="74.295" width="0.3048" layer="16"/>
 <wire x1="115.2525" y1="76.835" x2="108.2675" y2="87.63" width="0.3048" layer="1"/>
 <wire x1="108.2675" y1="87.63" x2="107.95" y2="90.4875" width="0.3048" layer="1"/>
-<wire x1="116.205" y1="74.295" x2="118.745" y2="74.295" width="0" layer="19" extent="1-1"/>
-<wire x1="113.665" y1="74.295" x2="116.205" y2="74.295" width="0" layer="19" extent="1-1"/>
-<wire x1="116.205" y1="64.77" x2="116.205" y2="74.295" width="0" layer="19" extent="1-1"/>
+<wire x1="116.205" y1="64.77" x2="115.2525" y2="76.835" width="0" layer="19" extent="16-16"/>
 </signal>
 <signal name="T3">
@@
 <via x="107.315" y="91.7575" extent="1-16" drill="0.6" shape="square"/>
 <wire x1="107.315" y1="91.7575" x2="113.0196375" y2="92.64116875" width="0.3048" layer="16"/>
-<contactref element="TEST1" pad="P$1"/>
 <wire x1="110.8075" y1="78.425" x2="110.8075" y2="76.835" width="0.3048" layer="16"/>
-<wire x1="110.8075" y1="76.835" x2="111.125" y2="74.295" width="0.3048" layer="16"/>
 <wire x1="110.8075" y1="76.835" x2="106.9975" y2="87.63" width="0.3048" layer="1"/>
 <wire x1="106.9975" y1="87.63" x2="107.315" y2="91.7575" width="0.3048" layer="1"/>
-<wire x1="111.125" y1="64.77" x2="111.125" y2="74.295" width="0" layer="19" extent="1-1"/>
+<wire x1="111.125" y1="64.77" x2="110.8075" y2="76.835" width="0" layer="19" extent="16-16"/>
 <wire x1="140.6525" y1="31.4325" x2="111.125" y2="64.77" width="0" layer="19" extent="1-1"/>
 </signal>

Commit message: r
Parts:
- moved TEST 35.8 mm to (115.3, 69.2)
- moved 2D2 0.95 mm to (155.3, 99.4)
Connections:
- net T1: now also TEST.P$5
- net T2: now also TEST.P$2, TEST.P$3, TEST.P$4
- net T3: now also TEST.P$1
Routing:
- net GND: track 338.0 -> 354.1 mm, vias 4 -> 6
- net T3: track 25.2 -> 28.9 mm
- net T2: track 23.4 -> 25.9 mm
- net N$14: track 13.1 -> 12.1 mm
- net N$13: track 8.50 -> 7.96 mm

Commit message: .
Parts:
- moved 5C6 2.31 mm to (145.1, 75.6)
- moved 5C5 1.62 mm to (147.3, 75.6)
- moved 1R17 0.32 mm to (113.7, 97.2)
- renumbered C1 to 3C1, Z1 to 6VD5
Routing:
- net +7V: track 7.36 -> 4.80 mm
- net RESET: track 29.6 -> 30.3 mm

Commit message: .
Parts:
- 1R26: device resistor:R1206W -> resistor:R0805
- 5R3: device resistor:R0805 -> resistor:0204/7
- moved 5R4 6.63 mm to (142.9, 90.8)
- moved 5R3 5.13 mm to (144.5, 92.7), flipped to the top, turned to 180 degrees
- moved 3C1 4.55 mm to (143.2, 86.4)
- moved 5C4 1.31 mm to (148.9, 90.2)
- moved 1R26 0.95 mm to (140.3, 105.7), flipped to the bottom, turned to 180 degrees
- moved 1RC2 0.32 mm to (107.0, 106.0)
- moved 6VT3 0.32 mm to (153.0, 107.3)
- moved DA6 0.32 mm to (148.3, 107.3), flipped to the bottom
- renumbered 1RC2*1 to 1RC3
Routing:
- net V+: track 77.4 -> 92.0 mm
- net +5V/2: track 3.04 -> 15.5 mm
- net GND: track 354.1 -> 360.5 mm
- net N$16: track 0.00 -> 5.13 mm
- net N$61: track 0.00 -> 3.80 mm
- net N$60: track 0.00 -> 3.20 mm
- net N$17: track 18.2 -> 17.7 mm

Commit message: .
Parts:
- 5C3: device resistor:E2-5 -> resistor:E2,5-7
- moved DA4 23.9 mm to (119.1, 121.0), turned to 180 degrees
- moved 1R5 21.5 mm to (32.4, 90.5)
- moved C14 21.5 mm to (10.8, 82.2)
- moved C15 21.5 mm to (10.8, 76.8)
- moved C16 21.5 mm to (10.8, 74.3)
- moved C19 21.5 mm to (7.30, 83.8)
- moved D12 21.5 mm to (10.8, 89.2)
- moved D7 21.5 mm to (23.8, 81.3)
- moved JP1 21.5 mm to (10.5, 69.8)
- moved Q1 21.5 mm to (15.6, 86.7)
- moved Q2 21.5 mm to (20.3, 86.7)
- moved R14 21.5 mm to (14.9, 92.4)
- moved R27 21.5 mm to (24.8, 88.3)
- moved R28 21.5 mm to (25.4, 92.4)
- moved R32 21.5 mm to (33.3, 80.3)
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Routing:
- net V+: track 92.0 -> 71.5 mm, vias 4 -> 3
- net N$77: track 24.1 -> 5.67 mm
- net B-: track 19.3 -> 6.24 mm
- net N$76: track 17.4 -> 8.82 mm
- net GND: track 360.5 -> 352.6 mm
- net N$78: track 8.79 -> 4.34 mm
- net N$79: track 7.30 -> 3.36 mm
- net N$85: track 3.73 -> 1.56 mm
- net N$17: track 17.7 -> 19.0 mm
- net +5V: track 40.6 -> 39.4 mm
- net N$84: track 27.2 -> 26.0 mm

Commit message: .
Parts:
- GREEN, RED: device led:CHIP-LED0805 -> led:LED5MM
- R19: device resistor:R0805 -> resistor:M0805
- R21: device resistor:R0805 -> resistor:R1206W
- R24: device resistor:0204/7 -> resistor:0207/10
- moved VT2 26.4 mm to (83.5, 105.7), turned to 270 degrees
- moved RED 21.0 mm to (70.8, 85.4), turned to 90 degrees
- moved R22 20.5 mm to (70.8, 89.5), turned to 270 degrees
- moved R23 18.6 mm to (72.7, 89.5), turned to 270 degrees
- moved B- 18.1 mm to (86.0, 100.6), turned to 180 degrees
- moved GREEN 17.7 mm to (77.8, 85.4), turned to 90 degrees
- moved DA2 16.9 mm to (80.6, 101.6)
- moved R20 16.6 mm to (79.1, 105.4), turned to 270 degrees
- moved C11 16.2 mm to (80.6, 98.4)
- moved 1C3 16.0 mm to (50.5, 85.1)
- moved 1R5 16.0 mm to (47.9, 86.7)
- moved R28 16.0 mm to (41.0, 88.6)
- moved R32 16.0 mm to (48.9, 76.5)
- moved R35 16.0 mm to (33.0, 70.5)
- moved R14 16.0 mm to (30.5, 88.6)
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Connections:
- removed net N$82: R22.1, RED.A
- removed net N$83: GREEN.A, R23.1
- new net N$4: R22.2, RED.K
- new net N$5: GREEN.K, R23.2
- net N$80: now also R22.1; no longer RED.C
- net N$81: now also R23.1; no longer GREEN.C
- net N$84: now also GREEN.A, RED.A; no longer R22.2, R23.2
Routing:
- net N$77: track 5.67 -> 30.9 mm
- net V+: track 71.5 -> 87.8 mm, vias 3 -> 2
- net B-: track 6.24 -> 17.4 mm
- net N$84: track 26.0 -> 35.2 mm
- net N$5: track 0.00 -> 6.72 mm
- net N$76: track 8.82 -> 2.53 mm
- net GND: track 352.6 -> 346.3 mm
- net PD4: track 1.14 -> 5.59 mm
- net N$4: track 0.00 -> 2.01 mm
- net N$60: track 3.20 -> 4.95 mm
- net N$78: track 4.34 -> 2.66 mm
- net N$85: track 1.56 -> 3.18 mm
- net N$83: track 1.59 -> 0.00 mm
- net N$82: track 1.59 -> 0.00 mm
- net N$79: track 3.36 -> 4.88 mm
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
Commit message: .
Parts:
- added U$5: MOD_TP4056, TP4056++:MOD_03962A
Changed lines of the file:
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@@
 <setting verticaltext="up"/>
 </settings>
-<grid distance="12.5" unitdist="mil" unit="mil" style="lines" multiple="1" display="yes" altdistance="0.025" altunitdist="inch" altunit="inch"/>
+<grid distance="50" unitdist="mil" unit="mil" style="lines" multiple="1" display="yes" altdistance="0.025" altunitdist="inch" altunit="inch"/>
 <layers>
 <layer number="1" name="Top" color="4" fill="1" visible="yes" active="yes"/>
@@
 <wire x1="175.26" y1="112.7125" x2="175.26" y2="130.4925" width="0.3048" layer="47"/>
 <wire x1="175.26" y1="130.4925" x2="164.1475" y2="130.4925" width="0.3048" layer="47"/>
-<rectangle x1="163.83" y1="116.5225" x2="165.735" y2="125.4125" layer="1"/>
+<rectangle x1="163.5125" y1="117.475" x2="165.4175" y2="126.365" layer="1"/>
 <rectangle x1="95.885" y1="117.1575" x2="98.1075" y2="124.1425" layer="1"/>
 <circle x="173.101" y="121.92" radius="1.5" width="0.4064" layer="1"/>
-<wire x1="105.0925" y1="164.465" x2="133.0325" y2="164.465" width="0.3048" layer="47"/>
-<wire x1="133.0325" y1="164.465" x2="133.0325" y2="181.9275" width="0.3048" layer="47"/>
-<wire x1="133.0325" y1="181.9275" x2="105.0925" y2="181.9275" width="0.3048" layer="47"/>
-<wire x1="105.0925" y1="181.9275" x2="105.0925" y2="164.465" width="0.3048" layer="47"/>
-<circle x="142.3035" y="115.57" radius="1.5" width="0.4064" layer="1"/>
-<circle x="140.081" y="116.205" radius="1.5" width="0.4064" layer="1"/>
-<circle x="137.2235" y="115.8875" radius="1.5" width="0.4064" layer="1"/>
 <wire x1="95.25" y1="61.2775" x2="95.25" y2="111.76" width="0.254" layer="20"/>
 <wire x1="95.25" y1="111.76" x2="175.26" y2="111.76" width="0.254" layer="20"/>
@@
 <element name="H1" library="pinhead" package="1X16" value="LCD" x="123.5075" y="153.3525"/>
 <element name="B+" library="TP4056_18650" package="PAD-" value="B-" x="77.1525" y="89.8525" rot="MR90"/>
+<element name="U$5" library="TP4056++" package="MOD_03962A" value="MOD_TP4056" x="213.995" y="136.8425"/>
 </elements>
 <signals>

Commit message: .
Parts:
- added U$11: (no value), b333:F18650
- U$5: device TP4056++:MOD_03962A -> TP4056+mod:MOD_03962A
- moved U$5 68.5 mm to (281.3, 149.5)
- moved DIS1 29.0 mm to (255.9, 116.2)
Connections:
- new net N$10: U$5.P2+B
- new net N$11: U$5.P2-OUT
- new net N$20: U$5.P2+OUT
- new net N$25: U$5.P1+
- new net N$9: U$5.P1-
Changed lines of the file:
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@@
 <wire x1="175.26" y1="61.2775" x2="95.25" y2="61.2775" width="0.254" layer="20"/>
 <circle x="172.72" y="63.5635" radius="1.5" width="0.4064" layer="1"/>
+<circle x="293.37" y="130.81" radius="2.5" width="0.2" layer="1"/>
 </plain>
 <attributes>
@@
 <element name="T5" library="pinhead" package="1X01" value="" x="122.555" y="62.5475"/>
 <element name="T6" library="pinhead" package="1X01" value="" x="117.475" y="62.5475"/>
-<element name="DIS1" library="b333" package="LCD_16X2_R2" value="LCD_16X2_R2" x="238.125" y="93.345">
-<attribute name="OC_NEWARK" value="unknown" x="228.2825" y="-42.2275" size="1.778" layer="27" display="off"/>
-<attribute name="MPN" value="" x="228.2825" y="-42.2275" size="1.778" layer="27" display="off"/>
-<attribute name="MF" value="" x="228.2825" y="-42.2275" size="1.778" layer="27" display="off"/>
-<attribute name="OC_FARNELL" value="unknown" x="228.2825" y="-42.2275" size="1.778" layer="27" display="off"/>
+<element name="DIS1" library="b333" package="LCD_16X2_R2" value="LCD_16X2_R2" x="255.905" y="116.205">
+<attribute name="OC_NEWARK" value="unknown" x="246.0625" y="-19.3675" size="1.778" layer="27" display="off"/>
+<attribute name="MPN" value="" x="246.0625" y="-19.3675" size="1.778" layer="27" display="off"/>
+<attribute name="MF" value="" x="246.0625" y="-19.3675" size="1.778" layer="27" display="off"/>
+<attribute name="OC_FARNELL" value="unknown" x="246.0625" y="-19.3675" size="1.778" layer="27" display="off"/>
 </element>
 <element name="D8" library="v-reg" package="TO92-CLP" value="TL431" x="120.015" y="98.1075" rot="R90"/>
@@
 <element name="H1" library="pinhead" package="1X16" value="LCD" x="123.5075" y="153.3525"/>
 <element name="B+" library="TP4056_18650" package="PAD-" value="B-" x="77.1525" y="89.8525" rot="MR90"/>
-<element name="U$5" library="TP4056++" package="MOD_03962A" value="MOD_TP4056" x="213.995" y="136.8425"/>
+<element name="U$5" library="TP4056+mod" package="MOD_03962A" value="MOD_TP4056" x="281.305" y="149.5425"/>
+<element name="U$11" library="b333" package="F18650" value="" x="251.1425" y="144.4625"/>
 </elements>
 <signals>
@@
 <wire x1="72.7075" y1="87.3125" x2="72.7075" y2="88.685" width="0.6096" layer="16"/>
 </signal>
+<signal name="N$9">
+<contactref element="U$5" pad="P1-"/>
+</signal>
+<signal name="N$11">
+<contactref element="U$5" pad="P2-OUT"/>
+</signal>
+<signal name="N$10">
+<contactref element="U$5" pad="P2+B"/>
+</signal>
+<signal name="N$20">
+<contactref element="U$5" pad="P2+OUT"/>
+</signal>
+<signal name="N$25">
+<contactref element="U$5" pad="P1+"/>
+</signal>
 </signals>
