File: HW_EAGLE/b333.brd (EAGLE design)
At the start: 80 x 50.5 mm, 155 parts, among them Q1 2N4126, Q2 2N4126, X1 USB MICRO

Commit message: .
Parts:
- moved U$5 1.27 mm to (280.0, 149.5)
Connections:
- new net N$27: U$5.P2-B
Changed lines of the file:
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@@
 <element name="H1" library="pinhead" package="1X16" value="LCD" x="123.5075" y="153.3525"/>
 <element name="B+" library="TP4056_18650" package="PAD-" value="B-" x="77.1525" y="89.8525" rot="MR90"/>
-<element name="U$5" library="TP4056+mod" package="MOD_03962A" value="MOD_TP4056" x="281.305" y="149.5425"/>
+<element name="U$5" library="TP4056+mod" package="MOD_03962A" value="MOD_TP4056" x="280.035" y="149.5425"/>
 <element name="U$11" library="b333" package="F18650" value="" x="251.1425" y="144.4625"/>
 </elements>
@@
 <contactref element="U$5" pad="P1+"/>
 </signal>
+<signal name="N$27">
+<contactref element="U$5" pad="P2-B"/>
+</signal>
 </signals>

Commit message: .
Parts:
- added S1: 9077-2, switch-misc:9077-2
- 6R15: device resistor:R0805 -> resistor:R1206W
- moved 6R15 3.17 mm to (158.1, 107.3), flipped to the bottom, turned to 180 degrees
- moved 6R14 2.62 mm to (156.2, 109.9), flipped to the bottom
- moved 6R13 0.63 mm to (144.1, 109.2), turned to 0 degrees
- moved U$11 0.63 mm to (251.1, 145.1)
Routing:
- net N$96: track 5.53 -> 1.65 mm, vias 1 -> 0
- net GND: track 346.3 -> 343.4 mm, vias 6 -> 5
- net N$21: track 6.32 -> 5.68 mm
Changed lines of the file:
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@@
 <setting verticaltext="up"/>
 </settings>
-<grid distance="50" unitdist="mil" unit="mil" style="lines" multiple="1" display="yes" altdistance="0.025" altunitdist="inch" altunit="inch"/>
+<grid distance="25" unitdist="mil" unit="mil" style="lines" multiple="1" display="yes" altdistance="0.025" altunitdist="inch" altunit="inch"/>
 <layers>
 <layer number="1" name="Top" color="4" fill="1" visible="yes" active="yes"/>
@@
 <circle x="97.8535" y="109.22" radius="1.5" width="0.4064" layer="1"/>
 <circle x="97.8535" y="78.105" radius="1.5" width="0.4064" layer="1"/>
-<dimension x1="35.8775" y1="102.87" x2="53.34" y2="69.215" x3="4.445" y3="86.0425" layer="21" dtype="vertical"/>
+<dimension x1="301.3075" y1="156.21" x2="300.99" y2="154.305" x3="212.09" y3="155.2575" layer="21" dtype="vertical"/>
 <dimension x1="24.4475" y1="67.6275" x2="63.5" y2="55.88" x3="43.97375" y3="144.4625" layer="21" dtype="horizontal"/>
 <circle x="172.72" y="78.1685" radius="1.5" width="0.4064" layer="1"/>
@@
 <element name="6R1C" library="resistor" package="R1206" value="" x="165.4175" y="91.7575" rot="MR180"/>
 <element name="6VT2" library="DSS" package="DPACK_1" value="NMOSD" x="164.465" y="107.95" rot="MR90"/>
-<element name="6R15" library="resistor" package="R0805" value="100k" x="158.115" y="104.14"/>
+<element name="6R15" library="resistor" package="R1206W" value="100k" x="158.115" y="107.315" rot="MR180"/>
 <element name="6R1B" library="resistor" package="R1206" value="1R" x="165.4175" y="93.98" rot="MR180"/>
-<element name="6R13" library="resistor" package="R0805" value="10k" x="144.78" y="109.22" rot="R90"/>
+<element name="6R13" library="resistor" package="R0805" value="10k" x="144.145" y="109.22"/>
 <element name="6R1A" library="resistor" package="R1206" value="1R" x="165.4175" y="89.535" rot="MR180"/>
 <element name="6C3" library="ct-pack" package="TT5D9L" value="22u/100V" x="155.575" y="85.09" smashed="yes">
@@
 <attribute name="VALUE" x="176.2125" y="93.0275" size="1.27" layer="27" rot="R90"/>
 </element>
-<element name="6R14" library="resistor" package="R0805" value="10k" x="156.845" y="107.315" rot="R270"/>
+<element name="6R14" library="resistor" package="R0805" value="10k" x="156.21" y="109.855" rot="MR270"/>
 <element name="U$8" library="b333" package="F18650" value="" x="129.2225" y="121.6025"/>
 <element name="TEST" library="transistor_tester" package="TT-P" value="TT-P" x="121.6025" y="66.9925"/>
@@
 <element name="B+" library="TP4056_18650" package="PAD-" value="B-" x="77.1525" y="89.8525" rot="MR90"/>
 <element name="U$5" library="TP4056+mod" package="MOD_03962A" value="MOD_TP4056" x="280.035" y="149.5425"/>
-<element name="U$11" library="b333" package="F18650" value="" x="251.1425" y="144.4625"/>
+<element name="U$11" library="b333" package="F18650" value="" x="251.1425" y="145.0975"/>
+<element name="S1" library="switch-misc" package="9077-2" value="9077-2" x="106.68" y="67.945"/>
 </elements>
 <signals>
@@
 <contactref element="6C6" pad="1"/>
 <contactref element="6R14" pad="1"/>
-<via x="157.48" y="110.1725" extent="1-16" drill="0.8" diameter="2.3"/>
-<wire x1="157.48" y1="110.1725" x2="157.1625" y2="109.22" width="0.3048" layer="1"/>
-<wire x1="156.845" y1="108.165" x2="157.1625" y2="109.22" width="0.3048" layer="1"/>
 <contactref element="1R4" pad="1"/>
 <wire x1="52.705" y1="84.24" x2="51.435" y2="81.915" width="0.3048" layer="16"/>
@@
 <wire x1="51.435" y1="75.565" x2="48.895" y2="75.5675" width="0.3048" layer="16"/>
 <wire x1="146.8725" y1="107.315" x2="149.1725" y2="107.315" width="0.3048" layer="16"/>
-<wire x1="157.48" y1="110.1725" x2="157.5375" y2="110.23" width="0.6096" layer="16"/>
-<wire x1="157.5375" y1="110.23" x2="159.665" y2="110.23" width="0.6096" layer="16"/>
 <wire x1="159.3375" y1="102.87" x2="158.115" y2="101.965" width="1.016" layer="16"/>
 <wire x1="158.115" y1="101.965" x2="158.115" y2="94.2975" width="1.016" layer="16"/>
@@
 <contactref element="6VD5" pad="A"/>
 <wire x1="155.575" y1="79.6925" x2="157.48" y2="79.6925" width="1.27" layer="16"/>
-<wire x1="150.8125" y1="74.6125" x2="150.8125" y2="78.74" width="1.27" layer="16"/>
+<wire x1="150.8125" y1="74.6125" x2="150.8125" y2="78.105" width="1.27" layer="16"/>
 <wire x1="153.035" y1="85.09" x2="153.035" y2="82.8675" width="1.27" layer="16"/>
 <wire x1="149.8125" y1="96.52" x2="149.285" y2="96.52" width="0.6096" layer="16"/>
@@
 <wire x1="153.035" y1="82.8675" x2="155.575" y2="81.5975" width="1.27" layer="16"/>
 <wire x1="155.575" y1="81.5975" x2="155.575" y2="79.6925" width="1.27" layer="16"/>
-<wire x1="157.48" y1="110.1725" x2="156.845" y2="109.5375" width="1.016" layer="16"/>
-<wire x1="156.845" y1="109.5375" x2="156.845" y2="105.3625" width="1.016" layer="16"/>
-<wire x1="156.845" y1="105.3625" x2="159.3375" y2="102.87" width="1.016" layer="16"/>
-<wire x1="150.8125" y1="78.74" x2="151.765" y2="79.6925" width="1.27" layer="16"/>
-<wire x1="151.765" y1="79.6925" x2="153.3525" y2="79.6925" width="1.27" layer="16"/>
+<wire x1="158.115" y1="110.23" x2="158.115" y2="104.0925" width="0.6096" layer="16"/>
+<wire x1="158.115" y1="104.0925" x2="159.3375" y2="102.87" width="1.016" layer="16"/>
+<wire x1="150.8125" y1="78.105" x2="152.4" y2="79.6925" width="1.27" layer="16"/>
+<wire x1="152.4" y1="79.6925" x2="153.3525" y2="79.6925" width="1.27" layer="16"/>
 <contactref element="JP3" pad="5"/>
 <contactref element="JP3" pad="1"/>
@@
 <wire x1="109.855" y1="91.7575" x2="111.4425" y2="92.3925" width="0.4064" layer="16"/>
 <wire x1="141.2875" y1="113.665" x2="141.2875" y2="109.22" width="0.6096" layer="16"/>
-<wire x1="157.48" y1="110.1725" x2="155.8925" y2="111.76" width="0.6096" layer="16"/>
 <wire x1="155.8925" y1="111.76" x2="150.495" y2="111.76" width="0.6096" layer="16"/>
 <wire x1="150.495" y1="111.76" x2="149.1725" y2="110.4375" width="0.6096" layer="16"/>
@@
 <wire x1="72.7075" y1="97.6825" x2="72.7075" y2="98.74" width="0.6096" layer="16"/>
 <wire x1="72.7075" y1="98.74" x2="73.345" y2="99.695" width="0.6096" layer="16"/>
+<wire x1="70.1675" y1="98.1075" x2="68.58" y2="99.695" width="0.6096" layer="16"/>
+<wire x1="68.58" y1="99.695" x2="68.58" y2="101.1555" width="0.6096" layer="16"/>
+<wire x1="155.8925" y1="111.76" x2="156.21" y2="111.4425" width="0.6096" layer="16"/>
+<wire x1="156.21" y1="111.4425" x2="156.21" y2="110.705" width="0.6096" layer="16"/>
+<wire x1="158.115" y1="110.23" x2="159.665" y2="110.23" width="0.8128" layer="16"/>
 <wire x1="118.745" y1="123.825" x2="119.65" y2="123.825" width="0" layer="19" extent="16-16"/>
 <wire x1="119.0625" y1="122.3675" x2="118.745" y2="123.825" width="0" layer="19" extent="16-16"/>
@@
 <wire x1="107.3625" y1="34.29" x2="131.7625" y2="73.3425" width="0" layer="19" extent="1-1"/>
 <wire x1="95.7825" y1="34.925" x2="107.3625" y2="34.29" width="0" layer="19" extent="1-1"/>
-<wire x1="70.1675" y1="98.1075" x2="68.58" y2="99.695" width="0.6096" layer="16"/>
-<wire x1="68.58" y1="99.695" x2="68.58" y2="101.1555" width="0.6096" layer="16"/>
+<wire x1="158.115" y1="110.23" x2="157.48" y2="110.705" width="0.8128" layer="16"/>
+<wire x1="157.48" y1="110.705" x2="156.21" y2="110.705" width="0.8128" layer="16"/>
 </signal>
 <signal name="ZENER">
@@
 <contactref element="6R13" pad="2"/>
 <contactref element="6VT3" pad="B"/>
-<wire x1="144.78" y1="110.07" x2="153.035" y2="109.855" width="0" layer="19" extent="1-1"/>
+<wire x1="144.995" y1="109.22" x2="153.035" y2="109.855" width="0" layer="19" extent="1-1"/>
 </signal>
 <signal name="N$96">
 <contactref element="6VT2" pad="G"/>
 <contactref element="6R15" pad="2"/>
-<via x="159.7025" y="107.6325" extent="1-16" drill="0.8" diameter="2.3"/>
-<wire x1="159.7025" y1="107.6325" x2="158.965" y2="104.14" width="0.3048" layer="1"/>
-<wire x1="159.665" y1="105.67" x2="159.7025" y2="107.6325" width="0.6096" layer="16"/>
+<wire x1="159.614" y1="107.315" x2="159.665" y2="105.67" width="0.6096" layer="16"/>
 </signal>
 <signal name="Z_YELLOW">
 <contactref element="6VD1" pad="A"/>
 <contactref element="3L2Y" pad="1"/>
-<wire x1="173.99" y1="101.9175" x2="171.7675" y2="103.505" width="0.3048" layer="16"/>
+<wire x1="173.99" y1="101.9175" x2="171.7675" y2="103.505" width="1.27" layer="16"/>
 </signal>
 <signal name="N$90">
@@
 <contactref element="6R15" pad="1"/>
 <contactref element="6VT3" pad="C"/>
-<wire x1="156.845" y1="106.465" x2="153.035" y2="107.315" width="0.3048" layer="1"/>
-<wire x1="157.265" y1="104.14" x2="156.845" y2="105.0925" width="0.3048" layer="1"/>
-<wire x1="156.845" y1="105.0925" x2="156.845" y2="106.465" width="0.3048" layer="1"/>
+<wire x1="153.035" y1="107.315" x2="156.616" y2="107.315" width="0.8128" layer="16"/>
+<wire x1="156.21" y1="109.005" x2="156.21" y2="107.315" width="0.8128" layer="16"/>
+<wire x1="156.21" y1="107.315" x2="156.616" y2="107.315" width="0.6096" layer="16"/>
 </signal>
 <signal name="GND1">

Commit message: pp pin
Parts:
- added BS1, BS2, D0, D1, D2, D4, D5, D6, OE, PAGEL, R/B, WR, XA0, XA1, XTAL1: (no value), pinhead:1X01
- added VD3, VD7: 1N4148DO35-7, diode:DO35-7
- D3, D7: value 1N4148DO35-7 -> (none); device diode:DO35-7 -> pinhead:1X01
- moved D3 137.6 mm to (172.1, 32.1), turned to 0 degrees
- moved D7 99.8 mm to (136.5, 100.3), turned to 0 degrees
- moved 4R6 21.3 mm to (129.2, 33.0)
- moved C10 18.9 mm to (107.3, 49.2)
- moved 1R18 18.2 mm to (107.6, 45.7)
- moved C17 15.3 mm to (112.7, 48.3)
- moved 4R7 15.3 mm to (124.8, 33.0)
- moved 1C7 2.93 mm to (130.5, 91.4), turned to 90 degrees
- moved J_PD4 2.56 mm to (130.2, 94.3), turned to 180 degrees
- moved 1C8 2.48 mm to (134.0, 88.6)
- moved 5R4 2.25 mm to (145.1, 90.5)
- moved 1C9 2.13 mm to (135.9, 88.6)
- moved ISP 1.62 mm to (132.7, 73.3)
- moved 1R9 1.59 mm to (132.1, 79.1)
- moved T4 0.95 mm to (126.7, 62.5)
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Connections:
- net +2V5 renamed PC4
- net N$87 renamed PD0
- net U_BAT renamed PC5
- removed net E1: DD1.9, JP3.6
- removed net N$62: DD1.1, JP3.14
- removed net N$68: 1C8.2, 1Z2.2, DD1.7
- removed net N$88: DD1.31, JP3.12
- removed net N$89: DD1.32, JP3.13
- removed net PB3: 1R19.1, DD1.12
- removed net PB4: 1R20.1, DD1.13
- removed net PB5: 1R21.1, DD1.14
- new net ADC6: DD1.19
- new net ADC7: DD1.22
- new net PB0: 1R19.1, D0.1, DD1.12
- new net PB1: 1R20.1, D1.1, DD1.13
- new net PB2: 1R21.1, D2.1, DD1.14
- new net PB6: 1C8.2, 1Z2.2, DD1.7, XTAL1.1
- new net PD5: DD1.9, JP3.6, XA0.1
- new net PD6: DD1.10, XA1.1
- new net PD7: 1R18.2, C17.1, DD1.11, PAGEL.1
- net FO: now also VD3.C; no longer D3.C
- net N$100: now also VD3.A, VD7.A; no longer D3.A, D7.A
- net N$102: now also VD7.C; no longer D7.C
- net PD1: now also DD1.31, JP3.12, R/B.1; no longer 1R18.2, C17.1, DD1.11
- net PD2: now also DD1.32, JP3.13, OE.1; no longer DD1.10
- net PD3: now also DD1.1, JP3.14, WR.1
- net PD4: now also BS1.1
Routing:
- net PD5: track 0.00 -> 26.7 mm, vias 0 -> 1
- net PD3: track 4.02 -> 30.5 mm
- net N$62: track 24.6 -> 0.00 mm
- net E1: track 22.2 -> 0.00 mm, vias 1 -> 0
- net PD1: track 0.00 -> 21.5 mm
- net PD2: track 0.00 -> 20.9 mm
- net N$89: track 17.8 -> 0.00 mm
- net N$88: track 16.2 -> 0.00 mm
- net PB6: track 0.00 -> 11.9 mm
- net N$68: track 7.32 -> 0.00 mm
- net PB3: track 6.88 -> 0.00 mm
- net PB0: track 0.00 -> 6.67 mm
- net GND: track 343.4 -> 337.9 mm
- net PB4: track 5.22 -> 0.00 mm
- net PB1: track 0.00 -> 5.22 mm
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
Commit message: .
Parts:
- moved 5C1 2.03 mm to (145.4, 93.3)
- moved 1R25 1.27 mm to (118.1, 92.7), turned to 180 degrees
- moved 5R3 0.64 mm to (144.5, 93.3)
- moved D5 0.32 mm to (136.5, 103.8)
Routing:
- net GND: track 337.9 -> 343.7 mm
- net N$16: track 5.13 -> 9.27 mm
- net V+: track 87.8 -> 89.7 mm
Changed lines of the file:
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@@
 <element name="5R1B" library="resistor" package="R1206" value="1R" x="139.065" y="101.6" rot="MR90"/>
 <element name="3C1" library="resistor" package="E2,5-6" value="50u" x="142.24" y="87.9475" rot="R270"/>
-<element name="5R3" library="resistor" package="0204/7" value="3.9k" x="144.4625" y="92.71" smashed="yes" rot="R180">
-<attribute name="NAME" x="146.3675" y="93.0021" size="0.9906" layer="25" ratio="10" rot="R180"/>
-<attribute name="VALUE" x="146.0881" y="93.1926" size="0.9906" layer="27" ratio="10" rot="R180"/>
+<element name="5R3" library="resistor" package="0204/7" value="3.9k" x="144.4625" y="93.345" smashed="yes" rot="R180">
+<attribute name="NAME" x="146.3675" y="93.6371" size="0.9906" layer="25" ratio="10" rot="R180"/>
+<attribute name="VALUE" x="146.0881" y="93.8276" size="0.9906" layer="27" ratio="10" rot="R180"/>
 </element>
 <element name="5R4" library="resistor" package="R0805" value="18k" x="145.0975" y="90.4875" rot="MR180"/>
@@
 </element>
 <element name="5C4" library="resistor" package="C0805K" value="100n" x="148.9075" y="90.17" rot="MR0"/>
-<element name="5C1" library="resistor" package="C0805K" value="100n" x="147.0025" y="94.615" rot="MR180"/>
+<element name="5C1" library="resistor" package="C0805K" value="100n" x="145.415" y="93.345" rot="MR180"/>
 <element name="2L3" library="ct-pack" package="LV7X10MM" value="330uH" x="147.955" y="80.645" rot="R180"/>
 <element name="5C5" library="resistor" package="E2-5" value="1000u/6V" x="147.32" y="74.6125" rot="R270"/>
@@
 </element>
 <element name="D8" library="v-reg" package="TO92-CLP" value="TL431" x="120.015" y="98.1075" rot="R90"/>
-<element name="1R25" library="resistor" package="R0805" value="2K2" x="116.84" y="92.71" rot="MR90"/>
+<element name="1R25" library="resistor" package="R0805" value="2K2" x="118.11" y="92.71" rot="MR180"/>
 <element name="1L2" library="rcl" package="IRF24" value="10mkhn" x="122.8725" y="84.455" rot="R20"/>
 <element name="1C13" library="resistor" package="C0805K" value="100n" x="115.8875" y="83.185" rot="MR0"/>
@@
 <element name="D2" library="pinhead" package="1X01" value="" x="139.3825" y="73.3425"/>
 <element name="D3" library="pinhead" package="1X01" value="" x="172.085" y="32.0675"/>
-<element name="D5" library="pinhead" package="1X01" value="" x="136.2075" y="103.8225"/>
+<element name="D5" library="pinhead" package="1X01" value="" x="136.525" y="103.8225"/>
 <element name="D6" library="pinhead" package="1X01" value="" x="171.1325" y="37.1475"/>
 <element name="D7" library="pinhead" package="1X01" value="" x="136.525" y="100.33"/>
@@
 <wire x1="117.5625" y1="122.7175" x2="116.205" y2="123.825" width="0" layer="19" extent="16-16"/>
 <wire x1="130.4925" y1="90.44" x2="134.3025" y2="119.8245" width="0" layer="19" extent="16-16"/>
-<wire x1="116.84" y1="91.86" x2="127.030428125" y2="87.816825" width="0" layer="19" extent="16-16"/>
+<wire x1="117.26" y1="92.71" x2="127.030428125" y2="87.816825" width="0" layer="19" extent="16-16"/>
 <wire x1="106.465" y1="49.2125" x2="133.985" y2="75.8825" width="0" layer="19" extent="1-16"/>
 <wire x1="106.7825" y1="45.72" x2="106.465" y2="49.2125" width="0" layer="19" extent="1-1"/>
@@
 <wire x1="153.67" y1="68.2625" x2="153.67" y2="64.77" width="0.6096" layer="16"/>
 <wire x1="147.9075" y1="90.17" x2="147.32" y2="87.9475" width="0.6096" layer="16"/>
-<wire x1="148.0025" y1="94.615" x2="147.955" y2="96.52" width="0.6096" layer="16"/>
+<wire x1="146.415" y1="93.345" x2="147.955" y2="96.52" width="0.6096" layer="16"/>
 <wire x1="142.24" y1="86.6775" x2="147.32" y2="87.9475" width="0.6096" layer="16"/>
 <wire x1="153.035" y1="85.09" x2="153.035" y2="89.2175" width="1.27" layer="16"/>
@@
 <via x="157.48" y="94.2975" extent="1-16" drill="0.6" diameter="2.3"/>
 <wire x1="157.48" y1="94.2975" x2="157.7975" y2="93.98" width="0.6096" layer="16"/>
-<wire x1="147.9075" y1="90.17" x2="148.225" y2="93.98" width="0.6096" layer="16"/>
-<wire x1="148.225" y1="93.98" x2="148.225" y2="94.3925" width="0.6096" layer="16"/>
-<wire x1="148.225" y1="94.3925" x2="148.0025" y2="94.615" width="0.6096" layer="16"/>
-<wire x1="150.495" y1="94.2975" x2="148.5425" y2="94.2975" width="1.27" layer="16"/>
-<wire x1="148.5425" y1="94.2975" x2="148.225" y2="93.98" width="0.6096" layer="16"/>
-<wire x1="114.8875" y1="85.09" x2="111.4425" y2="85.09" width="0.4064" layer="16"/>
-<wire x1="111.4425" y1="85.09" x2="109.855" y2="89.2175" width="0.4064" layer="16"/>
-<wire x1="109.855" y1="89.2175" x2="109.855" y2="91.7575" width="0.4064" layer="16"/>
-<wire x1="109.855" y1="91.7575" x2="111.4425" y2="92.3925" width="0.4064" layer="16"/>
+<wire x1="114.8875" y1="85.09" x2="112.0775" y2="85.09" width="0.4064" layer="16"/>
+<wire x1="112.0775" y1="85.09" x2="109.5375" y2="88.5825" width="0.4064" layer="16"/>
+<wire x1="109.5375" y1="88.5825" x2="109.5375" y2="91.7575" width="0.4064" layer="16"/>
+<wire x1="109.5375" y1="91.7575" x2="111.4425" y2="92.3925" width="0.4064" layer="16"/>
 <wire x1="141.2875" y1="113.665" x2="141.2875" y2="109.22" width="0.6096" layer="16"/>
 <wire x1="155.8925" y1="111.76" x2="150.495" y2="111.76" width="0.6096" layer="16"/>
@@
 <wire x1="127.169346875" y1="87.028978125" x2="125.73" y2="86.6775" width="0.3048" layer="16"/>
 <wire x1="125.73" y1="86.6775" x2="125.5627" y2="88.24055625" width="0.3048" layer="16"/>
+<wire x1="146.415" y1="93.345" x2="148.2725" y2="93.345" width="0.6096" layer="16"/>
+<wire x1="147.9075" y1="90.17" x2="148.2725" y2="93.345" width="0.6096" layer="16"/>
 <wire x1="118.745" y1="123.825" x2="119.65" y2="123.825" width="0" layer="19" extent="16-16"/>
 <wire x1="119.0625" y1="122.3675" x2="118.745" y2="123.825" width="0" layer="19" extent="16-16"/>
 <wire x1="113.3475" y1="113.665" x2="119.0625" y2="120.0675" width="0" layer="19" extent="16-16"/>
-<wire x1="148.2725" y1="92.71" x2="148.225" y2="93.98" width="0" layer="19" extent="16-16"/>
 <wire x1="147.32" y1="73.5965" x2="150.8125" y2="74.6125" width="0" layer="19" extent="16-16"/>
 <wire x1="145.0975" y1="74.565" x2="147.32" y2="73.5965" width="0" layer="19" extent="16-16"/>
@@
 <wire x1="113.7125" y1="48.26" x2="133.985" y2="70.8025" width="0" layer="19" extent="1-1"/>
 <wire x1="108.165" y1="49.2125" x2="113.7125" y2="48.26" width="0" layer="19" extent="1-1"/>
+<wire x1="149.8125" y1="96.52" x2="148.2725" y2="93.345" width="0.6096" layer="16"/>
+<wire x1="150.495" y1="94.2975" x2="148.2725" y2="93.345" width="0.6096" layer="16"/>
 </signal>
 <signal name="ZENER">
@@
 <wire x1="163.9955" y1="91.7575" x2="163.9955" y2="89.535" width="0.8128" layer="16"/>
 <wire x1="144.085" y1="97.79" x2="146.0025" y2="97.79" width="0.4064" layer="16"/>
-<wire x1="146.0025" y1="97.79" x2="146.0025" y2="94.615" width="0.4064" layer="16"/>
 <wire x1="138.43" y1="91.7575" x2="142.24" y2="89.2175" width="0.6096" layer="16"/>
 <wire x1="139.065" y1="100.178" x2="141.2875" y2="100.178" width="0.6096" layer="16"/>
@@
 <wire x1="139.065" y1="100.178" x2="115.57" y2="101.815" width="0" layer="19" extent="16-16"/>
 <wire x1="76.835" y1="101.9175" x2="115.57" y2="101.815" width="0" layer="19" extent="16-16"/>
+<wire x1="146.0025" y1="97.79" x2="146.0025" y2="96.155" width="0.4064" layer="16"/>
+<wire x1="146.0025" y1="96.155" x2="144.415" y2="94.5675" width="0.4064" layer="16"/>
+<wire x1="144.415" y1="94.5675" x2="144.415" y2="93.345" width="0.4064" layer="16"/>
 </signal>
 <signal name="N$8">
@@
 <contactref element="5R3" pad="2"/>
 <contactref element="DA3" pad="5"/>
-<wire x1="140.6525" y1="92.71" x2="144.085" y2="96.52" width="0.4064" layer="16"/>
-<wire x1="140.6525" y1="92.71" x2="144.2475" y2="90.4875" width="0" layer="19" extent="16-16"/>
+<wire x1="140.6525" y1="93.345" x2="144.085" y2="96.52" width="0.4064" layer="16"/>
+<wire x1="144.2475" y1="90.4875" x2="140.6525" y2="93.345" width="0.6096" layer="16"/>
 </signal>
 <signal name="N$17">
@@
 <wire x1="120.015" y1="92.71" x2="120.65" y2="92.075" width="0.4064" layer="16"/>
 <wire x1="120.65" y1="92.075" x2="120.94533125" y2="90.69650625" width="0.4064" layer="16"/>
-<wire x1="120.015" y1="92.71" x2="116.84" y2="93.56" width="0" layer="19" extent="16-16"/>
+<wire x1="120.015" y1="92.71" x2="118.96" y2="92.71" width="0" layer="19" extent="16-16"/>
 </signal>
 <signal name="N$60">

Commit message: .
Parts:
- moved D5 49.0 mm to (144.8, 55.6)
- moved D7 42.8 mm to (141.0, 57.8)
- moved XA1 16.9 mm to (136.5, 81.3)
- moved PAGEL 16.9 mm to (134.0, 81.3)
- moved D2 16.5 mm to (123.8, 78.7)
- moved D1 15.2 mm to (126.4, 78.7)
- moved D0 11.5 mm to (128.9, 78.7)
- moved BS2 8.91 mm to (171.4, 47.3)
- moved D4 4.76 mm to (171.1, 43.2)
- moved 1Z2 2.71 mm to (134.0, 86.0), turned to 200 degrees
- moved XA0 2.54 mm to (134.0, 94.0)
- moved 1C13 2.48 mm to (114.3, 81.3), turned to 90 degrees
- moved 1R9 2.25 mm to (134.3, 78.7)
- moved 1R19 1.93 mm to (128.3, 75.2)
- moved 1R20 1.93 mm to (126.4, 75.2)
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Routing:
- net PD6: track 0.00 -> 14.1 mm
- net PD7: track 0.00 -> 11.3 mm
- net PD3: track 30.5 -> 20.9 mm
- net PD2: track 20.9 -> 14.3 mm
- net PD1: track 21.5 -> 16.1 mm
- net PD5: track 26.7 -> 22.5 mm, vias 1 -> 0
- net AVCC: track 2.24 -> 6.33 mm
- net PB0: track 6.67 -> 10.1 mm
- net PB1: track 5.22 -> 8.27 mm
- net SCK: track 20.4 -> 23.0 mm
- net PB2: track 4.37 -> 6.88 mm
- net T3: track 28.9 -> 31.1 mm
- net T1: track 23.9 -> 25.9 mm
- net MISO: track 15.9 -> 17.9 mm
- net RESET: track 29.6 -> 31.6 mm
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