File: HW_EAGLE/b333.brd (EAGLE design)
At the start: 80 x 50.5 mm, 173 parts, among them Q1 2N4126, Q2 2N4126, X1 USB MICRO

Commit message: .
Parts:
- moved D7 9.97 mm to (148.9, 51.8)
- moved D5 4.85 mm to (140.7, 58.1)
- moved 1R10 4.14 mm to (111.4, 100.6)
- moved 1R9 3.59 mm to (136.8, 76.2), turned to 0 degrees
- moved 3C1 3.24 mm to (142.9, 84.8)
- moved 1R25 2.56 mm to (115.6, 94.9)
- moved D8 2.56 mm to (117.8, 100.3)
- moved OE 2.54 mm to (126.4, 96.5)
- moved 1R17 2.42 mm to (117.8, 96.8)
- moved 5R3 2.22 mm to (146.7, 93.3)
- moved 1R23 1.91 mm to (117.2, 75.6)
- moved 1C7 1.62 mm to (128.9, 91.1)
- moved 5C1 1.27 mm to (146.7, 93.3)
- moved 1R24 1.27 mm to (115.3, 75.6)
- moved 1C13 1.14 mm to (113.7, 82.2), turned to 0 degrees
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Connections:
- net PD4: no longer BS1.1
- net PD4MC: now also BS1.1
Routing:
- net PC3: track 34.9 -> 70.0 mm, vias 1 -> 2
- net T2: track 27.5 -> 46.3 mm, vias 2 -> 1
- net MOSI: track 20.6 -> 37.2 mm, vias 0 -> 1
- net T1: track 25.9 -> 40.9 mm, vias 2 -> 1
- net RESET: track 31.6 -> 42.8 mm
- net T3: track 31.1 -> 41.8 mm, vias 2 -> 1
- net PD2: track 14.3 -> 21.2 mm
- net PC5: track 0.00 -> 5.70 mm
- net PD0: track 14.5 -> 20.0 mm
- net PD3: track 20.9 -> 25.9 mm
- net SCK: track 23.0 -> 27.0 mm, vias 0 -> 1
- net MISO: track 17.9 -> 21.7 mm, vias 0 -> 1
- net PD4MC: track 5.55 -> 9.20 mm
- net PD1: track 16.1 -> 19.1 mm
- net +5V: track 42.0 -> 39.2 mm
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
Commit message: .
Parts:
- moved 1R10 8.04 mm to (119.4, 99.4)
- moved D5 5.24 mm to (141.9, 53.0)
- moved D8 4.02 mm to (114.0, 99.1), turned to 180 degrees
- moved D7 3.13 mm to (147.6, 54.6)
- moved 1Z2 2.93 mm to (131.1, 85.4), turned to 20 degrees
- moved 1C9 2.86 mm to (135.6, 86.7)
- moved PAGEL 2.54 mm to (131.4, 81.3)
- moved ISP 2.54 mm to (132.7, 76.2)
- moved XA1 2.54 mm to (134.0, 81.3)
- moved XTAL1 2.54 mm to (131.4, 91.4)
- moved 1R9 1.71 mm to (136.2, 77.8), turned to 90 degrees
- moved 1C8 1.14 mm to (132.7, 88.9), turned to 0 degrees
- moved J_PD4 0.45 mm to (131.1, 94.3)
- moved 1C7 0.32 mm to (128.9, 91.4)
- turned 3C1 to 0 degrees
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- renumbered T4 to T3, T5 to T2, T6 to T1
Connections:
- net T1: now also 1R23.2, 1R24.2, 4Y3.O, DD1.25, T1.1, TEST.P$1; no longer 1R19.2, 1R20.2, 4R6.1, 4R7.1, DD1.23, T3.1, TEST.P$5
- net T3: now also 1R19.2, 1R20.2, 4R6.1, 4R7.1, DD1.23, T3.1, TEST.P$5; no longer 1R23.2, 1R24.2, 4Y3.O, DD1.25, T1.1, TEST.P$1
Routing:
- net PD4: track 9.40 -> 36.0 mm, vias 0 -> 2
- net +5V: track 39.2 -> 33.5 mm
- net N$69: track 13.2 -> 9.45 mm
- net PD6: track 13.7 -> 10.1 mm
- net PD7: track 11.0 -> 7.97 mm
- net PC4: track 12.2 -> 14.4 mm
- net T2: track 46.3 -> 44.6 mm
- net RESET: track 42.8 -> 44.5 mm
- net PB6: track 11.6 -> 13.1 mm
- net V+: track 87.1 -> 88.2 mm
- net MOSI: track 37.2 -> 36.3 mm
- net T3: track 41.8 -> 40.9 mm
- net MISO: track 21.7 -> 22.3 mm
- net PD5: track 23.2 -> 22.6 mm

Commit message: .
Parts:
- removed C10: 100n, resistor:C0805
- added 1C1: 100n, resistor:C0805K
- added JGND1: (no value), rcl:R1206W
- 1L2: device rcl:IRF24 -> rcl:IRF36
- moved S1 32.8 mm to (74.0, 66.0)
- moved D7 10.4 mm to (138.1, 50.5)
- moved J_NO_LI 9.55 mm to (115.6, 120.3), turned to 180 degrees
- moved DA4A 8.55 mm to (115.9, 123.2), turned to 270 degrees
- moved 5C7 6.16 mm to (122.6, 120.3), turned to 180 degrees
- moved J_PD4 4.82 mm to (132.6, 98.9)
- moved 5C8 3.72 mm to (119.4, 120.3), turned to 180 degrees
- moved DA4 2.93 mm to (121.0, 123.2), turned to 0 degrees
- moved XTAL1 2.54 mm to (134.0, 91.4)
- moved XA0 2.54 mm to (134.0, 96.5)
- moved 1C6 2.31 mm to (112.7, 83.8)
- moved D5 2.25 mm to (141.6, 50.8)
- moved 1C8 1.91 mm to (134.6, 89.1)
- moved 1C7 1.80 mm to (130.2, 92.7), turned to 70 degrees
- moved J_ONE5V 1.80 mm to (133.0, 117.8), turned to 180 degrees
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Connections:
- net +5V: now also 1C1.1; no longer C10.1
- net GND: now also 1C1.2, JGND1.1; no longer 1C7.2, 1C8.1, 1C9.1, C10.2, DD1.3
- net GND1: now also 1C7.2, 1C8.1, 1C9.1, DD1.3, JGND1.2
Routing:
- net PD5: track 22.6 -> 58.2 mm, vias 0 -> 2
- net +5V: track 33.5 -> 64.4 mm
- net GND1: track 0.00 -> 17.1 mm
- net GND: track 342.3 -> 330.8 mm
- net RESET: track 44.5 -> 48.2 mm
- net N$77: track 30.9 -> 27.5 mm
- net PD4: track 36.0 -> 32.9 mm
- net MOSI: track 36.3 -> 33.8 mm
- net PD4MC: track 9.35 -> 11.7 mm
- net AREF: track 2.75 -> 5.03 mm
- net T1: track 40.9 -> 42.8 mm
- net PC5: track 5.92 -> 7.68 mm
- net V+: track 88.2 -> 86.5 mm
- net T2: track 44.6 -> 46.2 mm
- net T3: track 40.9 -> 42.5 mm
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